File: Soccerbot/soccerbotsqr.brd (EAGLE design)
At the start: 127 x 113 mm, 37 parts, among them X1 NXT-SOCKET, X2 NXT-SOCKET, X3 NXT-SOCKET, X4 NXT-SOCKET, X5 NXT-SOCKET, X6 NXT-SOCKET, X7 NXT-SOCKET, X8 NXT-SOCKET

Commit message: dfg
dfg
Connections:
- removed net A4: B1.A4
- removed net A5: B1.A5
- net SCL: now also B1.A5
- net SDA: now also B1.A4
Routing:
- net SDA: track 316.1 -> 392.4 mm, vias 0 -> 1
- net SCL: track 303.3 -> 342.8 mm, vias 1 -> 2
Changed lines of the file:
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@@
 <?xml version="1.0" encoding="utf-8"?>
 <!DOCTYPE eagle SYSTEM "eagle.dtd">
-<eagle version="8.2.2">
+<eagle version="8.3.0">
 <drawing>
 <settings>
 <setting alwaysvectorfont="no"/>
+<setting keepoldvectorfont="yes"/>
 <setting verticaltext="up"/>
 </settings>
@@
 <contactref element="B1" pad="A3"/>
 </signal>
-<signal name="A4">
-<contactref element="B1" pad="A4"/>
-</signal>
 <signal name="+3V3">
 <contactref element="JP5" pad="3"/>
@@
 </signal>
 <signal name="SDA">
-<contactref element="B1" pad="20"/>
 <contactref element="X1" pad="6"/>
 <contactref element="X2" pad="6"/>
@@
 <wire x1="74.93" y1="14.605" x2="74.93" y2="15" width="0.254" layer="16"/>
 <wire x1="90.17" y1="15.24" x2="90.17" y2="15" width="0.254" layer="16"/>
-<wire x1="159.385" y1="20.955" x2="156.21" y2="24.13" width="0.254" layer="16"/>
 <wire x1="159.385" y1="8.255" x2="159.385" y2="20.955" width="0.254" layer="16"/>
 <wire x1="96.52" y1="8.255" x2="159.385" y2="8.255" width="0.254" layer="16"/>
@@
 <wire x1="74.93" y1="15.24" x2="74.93" y2="15" width="0.254" layer="16"/>
 <wire x1="59.69" y1="14.605" x2="59.69" y2="15" width="0.254" layer="16"/>
+<contactref element="B1" pad="A4"/>
+<contactref element="B1" pad="20"/>
+<wire x1="159.385" y1="20.955" x2="156.21" y2="24.13" width="0.254" layer="16"/>
+<wire x1="156.21" y1="24.13" x2="158.75" y2="24.13" width="0.254" layer="1"/>
+<wire x1="158.75" y1="24.13" x2="161.2138" y2="26.5938" width="0.254" layer="1"/>
+<wire x1="161.2138" y1="26.5938" x2="161.2138" y2="39.4462" width="0.254" layer="1"/>
+<wire x1="161.2138" y1="39.4462" x2="158.75" y2="41.91" width="0.254" layer="1"/>
+<wire x1="142.10619375" y1="44.653" x2="142.037" y2="44.653" width="0.254" layer="1"/>
+<wire x1="142.037" y1="44.653" x2="138.43" y2="48.26" width="0.254" layer="1"/>
+<wire x1="158.75" y1="41.91" x2="144.84919375" y2="41.91" width="0.254" layer="1"/>
+<wire x1="144.84919375" y1="41.91" x2="142.10619375" y2="44.653" width="0.254" layer="1"/>
+<wire x1="138.43" y1="48.26" x2="133.35" y2="48.26" width="0.254" layer="1"/>
+<via x="133.35" y="48.26" extent="1-16" drill="1"/>
+<wire x1="133.35" y1="48.26" x2="109.22" y2="48.26" width="0.254" layer="16"/>
+<wire x1="109.22" y1="48.26" x2="107.95" y2="46.99" width="0.254" layer="16"/>
 </signal>
 <signal name="SCL">
@@
 <wire x1="45.085" y1="17.78" x2="45.45" y2="17.54" width="0.254" layer="16"/>
 <wire x1="154.94" y1="20.32" x2="156.21" y2="21.59" width="0.254" layer="16"/>
-<wire x1="93.98" y1="20.32" x2="154.94" y2="20.32" width="0.254" layer="16"/>
+<wire x1="93.98" y1="20.32" x2="113.03" y2="20.32" width="0.254" layer="16"/>
+<wire x1="113.03" y1="20.32" x2="154.94" y2="20.32" width="0.254" layer="16"/>
 <wire x1="91.44" y1="17.78" x2="93.98" y2="20.32" width="0.254" layer="16"/>
 <wire x1="91.44" y1="17.78" x2="91.17" y2="17.54" width="0.254" layer="16"/>
@@
 <wire x1="52.07" y1="45.72" x2="44.45" y2="45.72" width="0.254" layer="16"/>
 <via x="57.785" y="99.06" extent="1-16" drill="0.6096"/>
+<contactref element="B1" pad="A5"/>
+<wire x1="113.03" y1="20.32" x2="113.03" y2="34.29" width="0.254" layer="16"/>
+<wire x1="113.03" y1="34.29" x2="118.11" y2="34.29" width="0.254" layer="16"/>
+<via x="118.11" y="34.29" extent="1-16" drill="1"/>
+<wire x1="118.11" y1="34.29" x2="118.11" y2="44.45" width="0.254" layer="1"/>
+<wire x1="118.11" y1="44.45" x2="114.36919375" y2="44.45" width="0.254" layer="1"/>
+<wire x1="114.36919375" y1="44.45" x2="114.16619375" y2="44.653" width="0.254" layer="1"/>
+<wire x1="114.16619375" y1="44.653" x2="111.89380625" y2="44.653" width="0.254" layer="1"/>
+<wire x1="111.89380625" y1="44.653" x2="111.69080625" y2="44.45" width="0.254" layer="1"/>
+<wire x1="111.69080625" y1="44.45" x2="107.95" y2="44.45" width="0.254" layer="1"/>
 </signal>
 <signal name="D22">
@@
 <via x="58.42" y="68.58" extent="1-16" drill="0.6096"/>
 </signal>
-<signal name="A5">
-<contactref element="B1" pad="A5"/>
-</signal>
 <signal name="D44">
