File: Soccerbot/soccerbotsqr.brd (EAGLE design)
At the start: 127 x 113 mm, 37 parts, among them X1 NXT-SOCKET, X2 NXT-SOCKET, X3 NXT-SOCKET, X4 NXT-SOCKET, X5 NXT-SOCKET, X6 NXT-SOCKET, X7 NXT-SOCKET, X8 NXT-SOCKET

Commit message: sad
sd
Routing:
- net 5.5V: track 79.0 -> 78.2 mm
Changed lines of the file:
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@@
 <contactref element="B1" pad="5V@0"/>
 <contactref element="B1" pad="5V@1"/>
-<wire x1="156.21" y1="13.335" x2="156.21" y2="11.43" width="0.254" layer="1"/>
-<wire x1="153.035" y1="24.765" x2="107.95" y2="69.85" width="0.254" layer="1"/>
-<wire x1="153.035" y1="16.51" x2="153.035" y2="24.765" width="0.254" layer="1"/>
-<wire x1="156.21" y1="13.335" x2="153.035" y2="16.51" width="0.254" layer="1"/>
-<wire x1="156.21" y1="13.335" x2="156.21" y2="13.97" width="0.254" layer="1"/>
+<wire x1="156.21" y1="13.97" x2="156.21" y2="11.43" width="0.254" layer="1"/>
+<wire x1="141.605" y1="22.225" x2="107.95" y2="69.85" width="0.254" layer="1"/>
+<wire x1="153.035" y1="17.78" x2="141.605" y2="22.225" width="0.254" layer="1"/>
+<wire x1="156.21" y1="14.605" x2="153.035" y2="17.78" width="0.254" layer="1"/>
+<wire x1="156.21" y1="14.605" x2="156.21" y2="13.97" width="0.254" layer="1"/>
 </signal>
 <signal name="INT">

Commit message: And
And
Routing:
- net BAT+: track 285.2 -> 181.5 mm, vias 0 -> 5
- net D2: track 114.9 -> 190.4 mm, vias 0 -> 1
- net 3.3V: track 217.6 -> 275.8 mm
- net VIN: track 367.5 -> 320.9 mm
- net BAT-: track 251.2 -> 219.5 mm, vias 1 -> 0
- net SCL: track 342.8 -> 319.9 mm, vias 2 -> 4
- net 5.5V: track 78.2 -> 94.0 mm
- net GND: track 476.1 -> 464.7 mm
- net D7: track 123.6 -> 113.9 mm
- net D4: track 83.9 -> 90.9 mm
- net D5: track 75.5 -> 69.6 mm
- net D6: track 94.6 -> 90.1 mm, vias 1 -> 0
- net N$5: track 8.63 -> 9.90 mm
- net D3: track 96.6 -> 97.7 mm, vias 1 -> 0
- net N$3: track 6.25 -> 6.78 mm
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