File: Soccerbot/Nsoccerbots.sch (EAGLE design)
At the start: 37 parts, among them X1 NXT-SOCKET, X2 NXT-SOCKET, X3 NXT-SOCKET, X4 NXT-SOCKET, X5 NXT-SOCKET, X6 NXT-SOCKET, X7 NXT-SOCKET, X8 NXT-SOCKET

Commit message: j
J
Parts:
- removed D1: BLUE, SparkFun-LED:LED-BLUE1206
- removed D2: GREEN, SparkFun-LED:LED-GREEN0603
- removed D3: RED, SparkFun-LED:LED-RED0603
- removed F1, F2, F3: 72V/0.25A, SparkFun-Fuses:PPTC_PTH
- removed JP5: (no value), microbuilder:HEADER-1X770MIL
- removed X1, X2, X3, X4, X5, X6, X7, X8: NXT-SOCKET, NXT Compatible (female) Sockets - Mindsensors:NXT-SOCKET
- added COLORSENSOR2: (no value), microbuilder:HEADER-1X770MIL
- added IMU2: (no value), microbuilder:HEADER-1X876MIL
- added IR1, IR2, IR3, IR4, IR5, IR6: (no value), adafruit:PINHD-1X3
Connections:
- removed net N$3: D1.C, D2.A
- removed net N$5: D2.C, D3.A
- removed net N$6: D1.A, F1.1, S1.O
- new net DRDY: IMU2.5
- new net INT1: IMU2.4
- new net INT2: IMU2.3
- net +3V3: now also COLORSENSOR2.3, IMU2.8; no longer JP5.3
- net 3.3V: no longer X1.4, X2.4, X3.4, X4.4, X5.4, X6.4, X7.4, X8.4
- net 5.5V: now also IR1.3, IR2.3, IR3.3, IR4.3, IR5.3, IR6.3
- net BAT+: now also S1.O; no longer D3.C, F1.2
- net BAT-: no longer F2.2, F3.1, F3.2
- net D10: now also IR3.1
- net D11: now also IR4.1
- net D12: now also IR5.1
- net D13: now also IR6.1
- net D8: now also IR1.1
- net D9: now also IR2.1
- net GND: now also COLORSENSOR2.2, IMU2.6, IR1.2, IR2.2, IR3.2, IR4.2, IR5.2, IR6.2; no longer F2.1, JP5.2, X1.2, X1.3, X2.2, X2.3, X3.2, X3.3, X4.2, X4.3, X5.2, X5.3, X6.2, X6.3, X7.2, X7.3, X8.2, X8.3
- net INT: now also COLORSENSOR2.6; no longer JP5.6
- net SCL: now also COLORSENSOR2.4, IMU2.1; no longer JP5.4, X1.5, X2.5, X3.5, X4.5, X5.5, X6.5, X7.5, X8.5
- net SDA: now also COLORSENSOR2.5, IMU2.2; no longer JP5.5, X1.6, X2.6, X3.6, X4.6, X5.6, X6.6, X7.6, X8.6
- net VIN: now also COLORSENSOR2.1, COLORSENSOR2.7, IMU2.7; no longer JP5.1, JP5.7, X1.1, X2.1, X3.1, X4.1, X5.1, X6.1, X7.1, X8.1
Other:
- note added: "IMU"
- note added: "Pins 8-13 are dedicated to IR D13=IR1 D12=IR2 D11=IR3 D10=IR4 D9=IR5 D8=IR6"
- note removed: "NXT PORTS"

Commit message: And
Sad
Parts:
- added X1, X2: NXT-SOCKET, NXT Compatible (female) Sockets - Mindsensors:NXT-SOCKET
Connections:
- net 3.3V: now also X1.4, X2.4
- net GND: now also X1.2, X1.3, X2.2, X2.3
- net SCL: now also X1.5, X2.5
- net SDA: now also X1.6, X2.6
- net VIN: now also X1.1, X2.1
Changed lines of the file:
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@@
 <part name="IR5" library="adafruit" library_urn="urn:adsk.eagle:library:420" deviceset="PINHD-1X3" device=""/>
 <part name="IR6" library="adafruit" library_urn="urn:adsk.eagle:library:420" deviceset="PINHD-1X3" device=""/>
+<part name="X1" library="NXT Compatible (female) Sockets - Mindsensors" deviceset="NXT-SOCKET" device=""/>
+<part name="X2" library="NXT Compatible (female) Sockets - Mindsensors" deviceset="NXT-SOCKET" device=""/>
 </parts>
 <sheets>
@@
 <instance part="IR5" gate="A" x="116.84" y="15.24"/>
 <instance part="IR6" gate="A" x="106.68" y="15.24"/>
+<instance part="X1" gate="G$1" x="70.82469375" y="17.1958125"/>
+<instance part="X2" gate="G$1" x="70.82469375" y="-3.1241875"/>
 </instances>
 <busses>
@@
 <label x="99.06" y="15.24" size="1.778" layer="95"/>
 </segment>
+<segment>
+<pinref part="X1" gate="G$1" pin="2"/>
+<wire x1="78.44469375" y1="19.7358125" x2="81.28" y2="19.7358125" width="0.1524" layer="91"/>
+<wire x1="81.28" y1="19.7358125" x2="81.28" y2="20.32" width="0.1524" layer="91"/>
+<label x="81.28" y="20.32" size="1.778" layer="95"/>
+</segment>
+<segment>
+<pinref part="X1" gate="G$1" pin="3"/>
+<wire x1="78.44469375" y1="17.1958125" x2="81.28" y2="17.1958125" width="0.1524" layer="91"/>
+<wire x1="81.28" y1="17.1958125" x2="81.28" y2="17.78" width="0.1524" layer="91"/>
+<label x="81.28" y="17.78" size="1.778" layer="95"/>
+</segment>
+<segment>
+<pinref part="X2" gate="G$1" pin="2"/>
+<wire x1="78.44469375" y1="-0.5841875" x2="81.28" y2="-0.5841875" width="0.1524" layer="91"/>
+<wire x1="81.28" y1="-0.5841875" x2="81.28" y2="0" width="0.1524" layer="91"/>
+<label x="81.28" y="0" size="1.778" layer="95"/>
+</segment>
+<segment>
+<pinref part="X2" gate="G$1" pin="3"/>
+<wire x1="78.44469375" y1="-3.1241875" x2="81.28" y2="-3.1241875" width="0.1524" layer="91"/>
+<wire x1="81.28" y1="-3.1241875" x2="81.28" y2="-2.54" width="0.1524" layer="91"/>
+<label x="81.28" y="-2.54" size="1.778" layer="95"/>
+</segment>
 </net>
 <net name="D11" class="0">
@@
 </segment>
 </net>
+<net name="VIN" class="0">
+<segment>
+<pinref part="X1" gate="G$1" pin="1"/>
+<wire x1="78.44469375" y1="22.2758125" x2="81.28" y2="22.2758125" width="0.1524" layer="91"/>
+<wire x1="81.28" y1="22.2758125" x2="81.28" y2="22.86" width="0.1524" layer="91"/>
+<label x="81.28" y="22.86" size="1.778" layer="95"/>
+</segment>
+<segment>
+<pinref part="X2" gate="G$1" pin="1"/>
+<wire x1="78.44469375" y1="1.9558125" x2="81.28" y2="1.9558125" width="0.1524" layer="91"/>
+<wire x1="81.28" y1="1.9558125" x2="81.28" y2="2.54" width="0.1524" layer="91"/>
+<label x="81.28" y="2.54" size="1.778" layer="95"/>
+</segment>
+</net>
+<net name="3.3V" class="0">
+<segment>
+<pinref part="X1" gate="G$1" pin="4"/>
+<wire x1="78.44469375" y1="14.6558125" x2="81.28" y2="14.6558125" width="0.1524" layer="91"/>
+<wire x1="81.28" y1="14.6558125" x2="81.28" y2="15.24" width="0.1524" layer="91"/>
+<label x="81.28" y="15.24" size="1.778" layer="95"/>
+</segment>
+<segment>
+<pinref part="X2" gate="G$1" pin="4"/>
+<wire x1="78.44469375" y1="-5.6641875" x2="81.28" y2="-5.6641875" width="0.1524" layer="91"/>
+<wire x1="81.28" y1="-5.6641875" x2="81.28" y2="-5.08" width="0.1524" layer="91"/>
+<label x="81.28" y="-5.08" size="1.778" layer="95"/>
+</segment>
+</net>
+<net name="SCL" class="0">
+<segment>
+<pinref part="X1" gate="G$1" pin="5"/>
+<wire x1="78.44469375" y1="12.1158125" x2="81.28" y2="12.1158125" width="0.1524" layer="91"/>
+<wire x1="81.28" y1="12.1158125" x2="81.28" y2="12.7" width="0.1524" layer="91"/>
+<label x="81.28" y="12.7" size="1.778" layer="95"/>
+</segment>
+<segment>
+<pinref part="X2" gate="G$1" pin="5"/>
+<wire x1="78.44469375" y1="-8.2041875" x2="81.28" y2="-8.2041875" width="0.1524" layer="91"/>
+<wire x1="81.28" y1="-8.2041875" x2="81.28" y2="-7.62" width="0.1524" layer="91"/>
+<label x="81.28" y="-7.62" size="1.778" layer="95"/>
+</segment>
+</net>
+<net name="SDA" class="0">
+<segment>
+<pinref part="X1" gate="G$1" pin="6"/>
+<wire x1="78.44469375" y1="9.5758125" x2="81.28" y2="9.5758125" width="0.1524" layer="91"/>
+<wire x1="81.28" y1="9.5758125" x2="81.28" y2="10.16" width="0.1524" layer="91"/>
+<label x="81.28" y="10.16" size="1.778" layer="95"/>
+</segment>
+<segment>
+<pinref part="X2" gate="G$1" pin="6"/>
+<wire x1="78.44469375" y1="-10.7441875" x2="81.28" y2="-10.7441875" width="0.1524" layer="91"/>
+<wire x1="81.28" y1="-10.7441875" x2="81.28" y2="-10.16" width="0.1524" layer="91"/>
+<label x="81.28" y="-10.16" size="1.778" layer="95"/>
+</segment>
+</net>

Commit message: S
S
Parts:
- added JP1, JP2: (no value), adafruit:PINHD-1X3
Changed lines of the file:
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@@
 <part name="X1" library="NXT Compatible (female) Sockets - Mindsensors" deviceset="NXT-SOCKET" device=""/>
 <part name="X2" library="NXT Compatible (female) Sockets - Mindsensors" deviceset="NXT-SOCKET" device=""/>
+<part name="JP1" library="adafruit" library_urn="urn:adsk.eagle:library:420" deviceset="PINHD-1X3" device=""/>
+<part name="JP2" library="adafruit" library_urn="urn:adsk.eagle:library:420" deviceset="PINHD-1X3" device=""/>
 </parts>
 <sheets>
@@
 <attribute name="MPN" x="-187.96" y="76.2" size="1.778" layer="96" display="off"/>
 </instance>
+<instance part="JP1" gate="A" x="-203.2" y="129.54"/>
+<instance part="JP2" gate="A" x="-203.2" y="116.84"/>
 </instances>
 <busses>

Commit message: z
Z
Parts:
- removed ESC1+, ESC1-, ESC2+, ESC2-, ESC3+, ESC3-, ESC4+, ESC4-, ESC5+, ESC5-, ESC6+, ESC6-, PSU+(1-12V), PSU-(1-12V): (no value), wirepad:SMD5
- added BATERY, ESC1P, ESC2P, ESC3P, ESC4P, ESC5P, ESC6P, MOTOR, MOTOR1, MOTOR2, MOTOR3, MOTOR4, MOTOR5: (no value), con-wago-500:W237-102
- added DIOD1, DIOD2, DIOD3, DIOD4, DIOD5, DIOD6: 1N4004, adafruit:1N4004
- added RESITOR+1, RESITOR+2, RESITOR+3, RESITOR+4, RESITOR+5, RESITOR+6, RESITOR-1, RESITOR-2, RESITOR-3, RESITOR-4, RESITOR-5, RESITOR-6: (no value), adafruit:PINHD-1X1
- added TRANSISTOR1, TRANSISTOR2, TRANSISTOR3, TRANSISTOR4, TRANSISTOR5, TRANSISTOR6: 2N2907, adafruit:2N2907
- added X3, X4: NXT-SOCKET, NXT Compatible (female) Sockets - Mindsensors:NXT-SOCKET
Connections:
- new net N$1: RESITOR-1.1, TRANSISTOR1.B
- new net N$10: DIOD5.A, TRANSISTOR5.C
- new net N$11: DIOD4.A, TRANSISTOR4.C
- new net N$12: RESITOR-6.1, TRANSISTOR6.B
- new net N$13: DIOD6.A, TRANSISTOR6.C
- new net N$2: DIOD1.A, TRANSISTOR1.C
- new net N$3: RESITOR-4.1, TRANSISTOR4.B
- new net N$5: RESITOR-2.1, TRANSISTOR2.B
- new net N$6: DIOD2.A, TRANSISTOR2.C
- new net N$7: RESITOR-3.1, TRANSISTOR3.B
- new net N$8: DIOD3.A, TRANSISTOR3.C
- new net N$9: RESITOR-5.1, TRANSISTOR5.B
- net 3.3V: now also X3.4, X4.4
- net 5.5V: now also DIOD1.C, DIOD2.C, DIOD3.C, DIOD4.C, DIOD5.C, DIOD6.C, MOTOR-1.KL, MOTOR1-1.KL, MOTOR2-1.KL, MOTOR3-1.KL, MOTOR4-1.KL, MOTOR5-1.KL
- net BAT+: now also ESC1P-2.KL, ESC2P-2.KL, ESC3P-2.KL, ESC4P-2.KL, ESC5P-2.KL, ESC6P-2.KL; no longer ESC1+.P, ESC2+.P, ESC3+.P, ESC4+.P, ESC5+.P, ESC6+.P
- net BAT-: now also BATERY-2.KL, ESC1P-1.KL, ESC2P-1.KL, ESC3P-1.KL, ESC4P-1.KL, ESC5P-1.KL, ESC6P-1.KL; no longer ESC1-.P, ESC2-.P, ESC3-.P, ESC4-.P, ESC5-.P, ESC6-.P, PSU-(1-12V).P
- net D2: now also RESITOR+4.1
- net D3: now also RESITOR+1.1
- net D4: now also RESITOR+2.1
- net D5: now also RESITOR+3.1
- net D6: now also RESITOR+5.1
- net D7: now also RESITOR+6.1
- net GND: now also MOTOR-2.KL, MOTOR1-2.KL, MOTOR2-2.KL, MOTOR3-2.KL, MOTOR4-2.KL, MOTOR5-2.KL, TRANSISTOR1.E, TRANSISTOR2.E, TRANSISTOR3.E, TRANSISTOR4.E, TRANSISTOR5.E, TRANSISTOR6.E, X3.2, X3.3, X4.2, X4.3
- net N$4: now also BATERY-1.KL; no longer PSU+(1-12V).P
- net SCL: now also X3.5, X4.5
- net SDA: now also X3.6, X4.6
- net VIN: now also X3.1, X4.1

Commit message: Z
z
Parts:
- removed RESITOR+1, RESITOR+2, RESITOR+3, RESITOR+4, RESITOR+5, RESITOR+6, RESITOR-1, RESITOR-2, RESITOR-3, RESITOR-4, RESITOR-5, RESITOR-6: (no value), adafruit:PINHD-1X1
- added R1, R2, R3, R4, R5, R6: (no value), BaseApp:RESISTOR
- B1: MPN (none) -> A000067; OC_NEWARK unknown -> 45W6205
- BATERY, ESC1P, ESC2P, ESC3P, ESC4P, ESC5P, ESC6P, MOTOR, MOTOR1, MOTOR2, MOTOR3, MOTOR4, MOTOR5: MPN (none) -> MA522-500M02; OC_NEWARK (none) -> 04R6830
- DIOD1, DIOD2, DIOD3, DIOD4, DIOD5, DIOD6: MPN (none) -> 1N4004-T; OC_NEWARK (none) -> 12T2303
- IMU2, IR1, IR2, IR3, IR4, IR5, IR6, JP1, JP2: OC_NEWARK (none) -> unknown
- TRANSISTOR1, TRANSISTOR2, TRANSISTOR3, TRANSISTOR4, TRANSISTOR5, TRANSISTOR6: MPN (none) -> PN2222ATF; OC_NEWARK (none) -> 29X6831
- X1, X2, X3, X4: MPN (none) -> RJE01-660-01; OC_NEWARK (none) -> 01M6133
Connections:
- net D2: now also R3.1; no longer RESITOR+4.1
- net D3: now also R4.1; no longer RESITOR+1.1
- net D4: now also R5.1; no longer RESITOR+2.1
- net D5: now also R6.1; no longer RESITOR+3.1
- net D6: now also R1.1; no longer RESITOR+5.1
- net D7: now also R2.1; no longer RESITOR+6.1
- net N$1: now also R4.2; no longer RESITOR-1.1
- net N$12: now also R2.2; no longer RESITOR-6.1
- net N$3: now also R3.2; no longer RESITOR-4.1
- net N$5: now also R5.2; no longer RESITOR-2.1
- net N$7: now also R6.2; no longer RESITOR-3.1
- net N$9: now also R1.2; no longer RESITOR-5.1
