File: Soccerbot/Nsoccerbots.brd (EAGLE design)
At the start: 127 x 113 mm, 30 parts

Commit message: j
J
Parts:
- removed COLORSENSOR: (no value), microbuilder:1X07_ROUND_70
- removed IMU: (no value), microbuilder:1X08_ROUND_76
- added COLORSENSOR2: (no value), microbuilder:1X07_ROUND_70
- added IMU2: (no value), microbuilder:1X08_ROUND_76
- moved IR3 330.6 mm to (152.4, 94.0)
- moved IR2 325.3 mm to (19.1, 96.5), turned to 180 degrees
- moved IR1 293.7 mm to (16.5, 49.5), turned to 90 degrees
- moved IR4 276.0 mm to (154.9, 48.3), turned to 270 degrees
- moved IR5 223.7 mm to (153.7, 3.81)
- moved IR6 173.1 mm to (19.1, 5.08)
- moved ESC6+ 108.6 mm to (146.1, 47.0), turned to 0 degrees
- moved ESC6- 105.1 mm to (151.1, 47.0), turned to 0 degrees
- moved ESC6 101.6 mm to (146.1, 52.1)
- moved ESC3- 72.2 mm to (119.4, 91.4), turned to 0 degrees
- moved ESC3+ 67.8 mm to (114.3, 91.4), turned to 0 degrees
- moved ESC5- 65.6 mm to (29.2, 47.0), turned to 0 degrees
- moved PSU+(1-12V) 63.8 mm to (39.4, 8.89), turned to 180 degrees
- moved ESC5+ 62.9 mm to (24.1, 47.0), turned to 0 degrees
- moved PSU-(1-12V) 60.2 mm to (34.3, 8.89), turned to 180 degrees
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Connections:
- net +3V3: now also COLORSENSOR2.3, IMU2.8; no longer COLORSENSOR.3, IMU.8
- net D10: now also IR3.1; no longer IR4.1
- net D11: now also IR4.1; no longer IR3.1
- net D12: now also IR5.1; no longer IR2.1
- net D13: now also IR6.1; no longer IR1.1
- net D8: now also IR1.1; no longer IR6.1
- net D9: now also IR2.1; no longer IR5.1
- net DRDY: now also IMU2.5; no longer IMU.5
- net GND: now also COLORSENSOR2.2, IMU2.6; no longer COLORSENSOR.2, IMU.6
- net INT: now also COLORSENSOR2.6; no longer COLORSENSOR.6
- net INT1: now also IMU2.4; no longer IMU.4
- net INT2: now also IMU2.3; no longer IMU.3
- net SCL: now also COLORSENSOR2.4, IMU2.1; no longer COLORSENSOR.4, IMU.1
- net SDA: now also COLORSENSOR2.5, IMU2.2; no longer COLORSENSOR.5, IMU.2
- net VIN: now also COLORSENSOR2.1, COLORSENSOR2.7, IMU2.7; no longer COLORSENSOR.1, COLORSENSOR.7, IMU.7
Routing:
- net 5.5V: track 94.0 -> 416.8 mm, vias 0 -> 2
- net GND: track 320.9 -> 525.0 mm, vias 0 -> 1
- net D12: track 0.00 -> 164.0 mm, vias 0 -> 1
- net BAT+: track 198.0 -> 344.4 mm, vias 5 -> 0
- net +3V3: track 0.00 -> 138.0 mm
- net D11: track 0.00 -> 123.6 mm, vias 0 -> 1
- net BAT-: track 204.9 -> 313.5 mm, vias 0 -> 4
- net D2: track 190.4 -> 84.9 mm
- net D8: track 0.00 -> 103.1 mm, vias 0 -> 1
- net D10: track 0.00 -> 90.0 mm, vias 0 -> 1
- net D13: track 0.00 -> 88.9 mm, vias 0 -> 1
- net 3.3V: track 84.3 -> 0.00 mm
- net VIN: track 253.9 -> 329.9 mm, vias 0 -> 2
- net SCL: track 247.7 -> 183.9 mm, vias 4 -> 2
- net D9: track 0.00 -> 60.0 mm, vias 0 -> 1
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Other:
- board size 127 x 113 mm -> 144.8 x 100 mm
- board text removed: "+"
- board text removed: "-"
- board text removed: "3V3"
- board text removed: "D2"
- board text removed: "D3"
- board text removed: "D4"
- board text removed: "D5"
- board text removed: "D6"
- board text removed: "D7"
- board text removed: "FUSES"
- board text removed: "GND"
- board text removed: "INT"
- board text removed: "M4"
- board text removed: "ON/OFF"
- board text removed: "PWM"
- board text removed: "Power"
- board text removed: "SCL"
- board text removed: "SDA"
- board text removed: "VIN"
- board text removed: "color sensor"

Commit message: And
Sad
Parts:
- added X1, X2: NXT-SOCKET, NXT Compatible (female) Sockets - Mindsensors:NXT-SOCKET
Connections:
- net 3.3V: now also X1.4, X2.4
- net GND: now also X1.2, X1.3, X2.2, X2.3
- net SCL: now also X1.5, X2.5
- net SDA: now also X1.6, X2.6
- net VIN: now also X1.1, X2.1
Routing:
- net 3.3V: track 0.00 -> 174.6 mm
- net SDA: track 193.6 -> 278.3 mm, vias 1 -> 0
- net SCL: track 183.9 -> 262.1 mm, vias 2 -> 0
- net VIN: track 329.9 -> 384.7 mm
- net BAT+: track 344.4 -> 378.8 mm
- net D12: track 164.0 -> 139.5 mm
- net D8: track 103.1 -> 81.9 mm, vias 1 -> 2
- net D11: track 123.6 -> 144.7 mm, vias 1 -> 2
- net D3: track 77.3 -> 95.4 mm, vias 0 -> 1
- net D5: track 34.1 -> 52.1 mm
- net BAT-: track 313.5 -> 327.2 mm
- net D6: track 72.9 -> 62.2 mm, vias 1 -> 0
- net D7: track 104.7 -> 114.1 mm, vias 1 -> 2
- net D2: track 84.9 -> 76.8 mm
- net D13: track 88.9 -> 96.7 mm
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Other:
- board size 144.8 x 100 mm -> 146 x 100 mm
- board text added: "GND"
- board text added: "SIGNAL"
- board text added: "VIN"

Commit message: And
And
Routing:
- net SDA: track 278.3 -> 284.9 mm
- net SCL: track 262.1 -> 262.9 mm
Changed lines of the file:
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@@
 <wire x1="158.73" y1="100" x2="12.7" y2="100" width="0" layer="20"/>
 <wire x1="12.7" y1="100" x2="12.7" y2="0" width="0" layer="20"/>
-<wire x1="95.25" y1="55.88" x2="95.25" y2="48.26" width="0.635" layer="45"/>
-<wire x1="95.25" y1="48.26" x2="100.33" y2="48.26" width="0.635" layer="45"/>
-<wire x1="100.33" y1="48.26" x2="100.33" y2="55.88" width="0.635" layer="45"/>
-<wire x1="100.33" y1="55.88" x2="95.25" y2="55.88" width="0.635" layer="45"/>
 <text x="16.51" y="8.89" size="0.6096" layer="25" rot="R90">SIGNAL</text>
 <text x="66.04" y="15.24" size="0.6096" layer="25" rot="R90">SIGNAL</text>
@@
 <text x="22.86" y="50.8" size="0.6096" layer="25" rot="R90">GND</text>
 <text x="31.75" y="50.8" size="0.6096" layer="25" rot="R90">SIGNAL</text>
+<dimension x1="12.7" y1="0" x2="158.75" y2="0" x3="85.725" y3="-2.54" textsize="0.6096" layer="25"/>
+<dimension x1="12.7" y1="100" x2="12.7" y2="0" x3="8.89" y3="50" textsize="0.6096" layer="25"/>
+<wire x1="95.25" y1="55.88" x2="101.6" y2="55.88" width="0.1524" layer="45"/>
+<wire x1="101.6" y1="55.88" x2="101.6" y2="48.26" width="0.1524" layer="45"/>
+<wire x1="101.6" y1="48.26" x2="95.25" y2="48.26" width="0.1524" layer="45"/>
+<wire x1="95.25" y1="48.26" x2="95.25" y2="55.88" width="0.1524" layer="45"/>
 </plain>
 <attributes>
@@
 <wire x1="78.74" y1="42.545" x2="78.74" y2="26.67" width="0.635" layer="16"/>
 <wire x1="26.67" y1="42.545" x2="78.74" y2="42.545" width="0.635" layer="16"/>
-<wire x1="78.74" y1="13.335" x2="78.74" y2="10.795" width="0.635" layer="16"/>
-<wire x1="78.74" y1="26.67" x2="78.74" y2="13.335" width="0.635" layer="1"/>
+<wire x1="78.74" y1="12.065" x2="78.74" y2="10.795" width="0.635" layer="16"/>
+<wire x1="78.74" y1="26.67" x2="78.74" y2="12.065" width="0.635" layer="1"/>
 <wire x1="142.24" y1="41.91" x2="142.24" y2="25.4" width="0.635" layer="16"/>
 <wire x1="139.7" y1="41.91" x2="142.24" y2="41.91" width="0.635" layer="16"/>
@@
 <wire x1="116.84" y1="12.7" x2="116.84" y2="12.573" width="0.635" layer="1"/>
 <via x="26.67" y="42.545" extent="1-16" drill="0.35"/>
-<via x="78.74" y="13.335" extent="1-16" drill="0.35"/>
+<via x="78.74" y="12.065" extent="1-16" drill="0.35"/>
 </signal>
 <signal name="D2">
@@
 <wire x1="24.765" y1="48.895" x2="20.955" y2="48.895" width="0.635" layer="16"/>
 <wire x1="25.4" y1="48.26" x2="24.765" y2="48.895" width="0.635" layer="16"/>
-<wire x1="93.345" y1="48.26" x2="25.4" y2="48.26" width="0.635" layer="16"/>
-<wire x1="119.38" y1="74.295" x2="93.345" y2="48.26" width="0.635" layer="16"/>
-<wire x1="119.38" y1="74.93" x2="119.38" y2="74.295" width="0.635" layer="16"/>
-<wire x1="95.885" y1="27.305" x2="96.52" y2="26.67" width="0.635" layer="1"/>
-<wire x1="95.885" y1="50.165" x2="95.885" y2="27.305" width="0.635" layer="1"/>
-<wire x1="119.38" y1="73.66" x2="95.885" y2="50.165" width="0.635" layer="1"/>
-<wire x1="119.38" y1="74.93" x2="119.38" y2="73.66" width="0.635" layer="1"/>
+<wire x1="119.38" y1="74.295" x2="119.38" y2="74.93" width="0.635" layer="16"/>
 <wire x1="130.81" y1="83.185" x2="140.335" y2="73.66" width="0.635" layer="1"/>
 <wire x1="119.38" y1="83.185" x2="130.81" y2="83.185" width="0.635" layer="1"/>
 <wire x1="119.38" y1="74.93" x2="119.38" y2="83.185" width="0.635" layer="1"/>
+<wire x1="96.52" y1="26.67" x2="96.52" y2="30.1414" width="0.635" layer="1"/>
+<wire x1="96.52" y1="30.1414" x2="96.1265" y2="30.5349" width="0.635" layer="1"/>
+<wire x1="96.1265" y1="30.5349" x2="96.1265" y2="35.1665" width="0.635" layer="1"/>
+<wire x1="96.1265" y1="35.1665" x2="116.84" y2="55.88" width="0.635" layer="1"/>
+<wire x1="118.7323" y1="74.2823" x2="119.38" y2="74.93" width="0.635" layer="1"/>
+<wire x1="116.84" y1="55.88" x2="116.84" y2="71.22894375" width="0.635" layer="1"/>
+<wire x1="116.84" y1="71.22894375" x2="118.7323" y2="73.12124375" width="0.635" layer="1"/>
+<wire x1="118.7323" y1="73.12124375" x2="118.7323" y2="74.2823" width="0.635" layer="1"/>
+<wire x1="119.38" y1="74.93" x2="119.38" y2="73.66" width="0.635" layer="16"/>
+<wire x1="119.38" y1="73.66" x2="106.68" y2="60.96" width="0.635" layer="16"/>
+<wire x1="106.68" y1="60.96" x2="104.4786" y2="60.96" width="0.635" layer="16"/>
+<wire x1="94.8565" y1="56.7565" x2="93.98" y2="55.88" width="0.635" layer="16"/>
+<wire x1="104.4786" y1="60.96" x2="100.2751" y2="56.7565" width="0.635" layer="16"/>
+<wire x1="100.2751" y1="56.7565" x2="94.8565" y2="56.7565" width="0.635" layer="16"/>
+<wire x1="93.98" y1="55.88" x2="92.60105625" y2="55.88" width="0.635" layer="16"/>
+<wire x1="92.60105625" y1="55.88" x2="84.98105625" y2="48.26" width="0.635" layer="16"/>
+<wire x1="84.98105625" y1="48.26" x2="25.4" y2="48.26" width="0.635" layer="16"/>
 </signal>
 <signal name="D22">
@@
 <wire x1="116.84" y1="74.93" x2="116.84" y2="75.565" width="0.635" layer="16"/>
 <wire x1="144.78" y1="74.295" x2="145.02" y2="74.93" width="0.635" layer="16"/>
-<wire x1="94.615" y1="27.305" x2="93.98" y2="26.67" width="0.635" layer="1"/>
-<wire x1="94.615" y1="50.8" x2="94.615" y2="27.305" width="0.635" layer="1"/>
-<wire x1="116.84" y1="73.025" x2="94.615" y2="50.8" width="0.635" layer="1"/>
-<wire x1="116.84" y1="74.93" x2="116.84" y2="73.025" width="0.635" layer="1"/>
+<wire x1="116.1923" y1="74.14618125" x2="115.08381875" y2="73.0377" width="0.635" layer="1"/>
+<wire x1="107.3277" y1="73.0377" x2="91.44" y2="57.15" width="0.635" layer="1"/>
+<wire x1="116.84" y1="74.93" x2="116.1923" y2="74.2823" width="0.635" layer="1"/>
+<wire x1="116.1923" y1="74.2823" x2="116.1923" y2="74.14618125" width="0.635" layer="1"/>
+<wire x1="115.08381875" y1="73.0377" x2="107.3277" y2="73.0377" width="0.635" layer="1"/>
+<wire x1="93.3323" y1="27.45381875" x2="93.3323" y2="27.3177" width="0.635" layer="1"/>
+<wire x1="93.3323" y1="27.3177" x2="93.98" y2="26.67" width="0.635" layer="1"/>
+<wire x1="91.44" y1="57.15" x2="91.44" y2="29.34611875" width="0.635" layer="1"/>
+<wire x1="91.44" y1="29.34611875" x2="93.3323" y2="27.45381875" width="0.635" layer="1"/>
 </signal>
 <signal name="BAT+">

Commit message: S
S
Parts:
- added JP1, JP2: (no value), adafruit:1X03
Other:
- board text added: "Designed By, David Bershadsky"
- board text added: "The ESC Connections are D2=ESC1 D3=ESC2 D4=ESC3 D5=ESC4 D6=ESC5 D7=ESC6"
- board text added: "The IR Sesnor Connections are D13=IR1 D12=IR2 D11=IR3 D10=IR4 D9=IR5 D8=IR6"
Changed lines of the file:
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@@
 <dimension x1="12.7" y1="0" x2="158.75" y2="0" x3="85.725" y3="-2.54" textsize="0.6096" layer="25"/>
 <dimension x1="12.7" y1="100" x2="12.7" y2="0" x3="8.89" y3="50" textsize="0.6096" layer="25"/>
-<wire x1="95.25" y1="55.88" x2="101.6" y2="55.88" width="0.1524" layer="45"/>
-<wire x1="101.6" y1="55.88" x2="101.6" y2="48.26" width="0.1524" layer="45"/>
-<wire x1="101.6" y1="48.26" x2="95.25" y2="48.26" width="0.1524" layer="45"/>
-<wire x1="95.25" y1="48.26" x2="95.25" y2="55.88" width="0.1524" layer="45"/>
+<hole x="27.94" y="95.25" drill="0.35"/>
+<hole x="144.78" y="93.98" drill="0.35"/>
+<hole x="138.43" y="11.43" drill="0.35"/>
+<hole x="48.26" y="10.16" drill="0.35"/>
+<hole x="21.59" y="17.78" drill="0.35"/>
+<hole x="20.32" y="74.93" drill="0.35"/>
+<text x="31.75" y="76.2" size="1.778" layer="25">The ESC Connections are
+D2=ESC1
+D3=ESC2
+D4=ESC3
+D5=ESC4
+D6=ESC5
+D7=ESC6
+</text>
+<text x="72.39" y="78.74" size="1.778" layer="25">The IR Sesnor Connections are
+D13=IR1
+D12=IR2
+D11=IR3
+D10=IR4
+D9=IR5
+D8=IR6</text>
+<text x="69.85" y="6.35" size="1.778" layer="25">Designed By,
+David Bershadsky</text>
 </plain>
 <attributes>
@@
 <attribute name="OC_NEWARK" value="unknown" x="147.32" y="77.47" size="1.778" layer="27" rot="R90" display="off"/>
 </element>
+<element name="JP1" library="adafruit" library_urn="urn:adsk.eagle:library:420" package="1X03" value="" x="99.06" y="52.07" rot="R90"/>
+<element name="JP2" library="adafruit" library_urn="urn:adsk.eagle:library:420" package="1X03" value="" x="96.52" y="52.07" rot="R90"/>
 </elements>
 <signals>
@@
 </drawing>
 <compatibility>
+<note version="6.3" minversion="6.2.2" severity="warning">
+Since Version 6.2.2 text objects can contain more than one line,
+which will not be processed correctly with this version.
+</note>
 <note version="8.2" severity="warning">
 Since Version 8.2, Eagle supports online libraries. The ids

Commit message: z
Z
Parts:
- removed ESC1+, ESC1-, ESC2+, ESC2-, ESC3+, ESC3-, ESC4+, ESC4-, ESC5+, ESC5-, ESC6+, ESC6-, PSU+(1-12V), PSU-(1-12V): (no value), wirepad:SMD2,54-5,08
- added BATERY, ESC1P, ESC2P, ESC3P, ESC4P, ESC5P, ESC6P, MOTOR, MOTOR1, MOTOR2, MOTOR3, MOTOR4, MOTOR5: (no value), con-wago-500:W237-102
- added DIOD1, DIOD2, DIOD3, DIOD4, DIOD5, DIOD6: 1N4004, adafruit:DO41-10
- added RESITOR+1, RESITOR+2, RESITOR+3, RESITOR+4, RESITOR+5, RESITOR+6, RESITOR-1, RESITOR-2, RESITOR-3, RESITOR-4, RESITOR-5, RESITOR-6: (no value), adafruit:1X01
- added TRANSISTOR1, TRANSISTOR2, TRANSISTOR3, TRANSISTOR4, TRANSISTOR5, TRANSISTOR6: 2N2907, adafruit:TO92-EBC-OVAL
- added X3, X4: NXT-SOCKET, NXT Compatible (female) Sockets - Mindsensors:NXT-SOCKET
- moved COLORSENSOR2 2.54 mm to (20.3, 47.0)
- moved S1 1.27 mm to (39.4, 19.1)
Connections:
- new net N$1: RESITOR-1.1, TRANSISTOR1.B
- new net N$10: DIOD5.A, TRANSISTOR5.C
- new net N$11: DIOD4.A, TRANSISTOR4.C
- new net N$12: RESITOR-6.1, TRANSISTOR6.B
- new net N$13: DIOD6.A, TRANSISTOR6.C
- new net N$2: DIOD1.A, TRANSISTOR1.C
- new net N$3: RESITOR-4.1, TRANSISTOR4.B
- new net N$5: RESITOR-2.1, TRANSISTOR2.B
- new net N$6: DIOD2.A, TRANSISTOR2.C
- new net N$7: RESITOR-3.1, TRANSISTOR3.B
- new net N$8: DIOD3.A, TRANSISTOR3.C
- new net N$9: RESITOR-5.1, TRANSISTOR5.B
- net 3.3V: now also X3.4, X4.4
- net 5.5V: now also DIOD1.C, DIOD2.C, DIOD3.C, DIOD4.C, DIOD5.C, DIOD6.C, MOTOR.1, MOTOR1.1, MOTOR2.1, MOTOR3.1, MOTOR4.1, MOTOR5.1
- net BAT+: now also ESC1P.2, ESC2P.2, ESC3P.2, ESC4P.2, ESC5P.2, ESC6P.2; no longer ESC1+.1, ESC2+.1, ESC3+.1, ESC4+.1, ESC5+.1, ESC6+.1
- net BAT-: now also BATERY.2, ESC1P.1, ESC2P.1, ESC3P.1, ESC4P.1, ESC5P.1, ESC6P.1; no longer ESC1-.1, ESC2-.1, ESC3-.1, ESC4-.1, ESC5-.1, ESC6-.1, PSU-(1-12V).1
- net D2: now also RESITOR+4.1
- net D3: now also RESITOR+1.1
- net D4: now also RESITOR+2.1
- net D5: now also RESITOR+3.1
- net D6: now also RESITOR+5.1
- net D7: now also RESITOR+6.1
- net GND: now also MOTOR.2, MOTOR1.2, MOTOR2.2, MOTOR3.2, MOTOR4.2, MOTOR5.2, TRANSISTOR1.E, TRANSISTOR2.E, TRANSISTOR3.E, TRANSISTOR4.E, TRANSISTOR5.E, TRANSISTOR6.E, X3.2, X3.3, X4.2, X4.3
- net N$4: now also BATERY.1; no longer PSU+(1-12V).1
- net SCL: now also X3.5, X4.5
- net SDA: now also X3.6, X4.6
- net VIN: now also X3.1, X4.1
Routing:
- net GND: track 526.6 -> 686.1 mm, vias 2 -> 4
- net D4: track 41.8 -> 148.9 mm, vias 0 -> 2
- net 5.5V: track 419.1 -> 500.0 mm, vias 3 -> 1
- net D6: track 62.2 -> 143.0 mm, vias 0 -> 3
- net D5: track 52.1 -> 127.5 mm, vias 0 -> 2
- net D3: track 95.4 -> 154.7 mm, vias 1 -> 2
- net N$7: track 0.00 -> 46.6 mm, vias 0 -> 1
- net BAT-: track 327.2 -> 371.3 mm, vias 4 -> 2
- net N$13: track 0.00 -> 43.6 mm, vias 0 -> 1
- net N$11: track 0.00 -> 43.4 mm
- net D7: track 114.1 -> 155.3 mm, vias 2 -> 0
- net 3.3V: track 174.6 -> 211.2 mm, vias 0 -> 1
- net VIN: track 384.7 -> 418.8 mm, vias 2 -> 5
- net D9: track 60.0 -> 85.1 mm
- net D2: track 76.8 -> 98.2 mm, vias 1 -> 0
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
Commit message: s
S
Parts:
- added IC1: 33035P, motorola-sensor-driver:DIL24S
- added U$1: VNH2SP30, SparkFun-IC-Special-Function:VNH2SP30
Connections:
- new net VC: IC1.18
- new net VCC: IC1.17
- net GND: now also IC1.16
Changed lines of the file:
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@@
 <attribute name="OC_NEWARK" value="70K9898" x="39.37" y="6.35" size="1.778" layer="27" display="off"/>
+</element>
+<element name="U$1" library="SparkFun-IC-Special-Function" package="VNH2SP30" value="VNH2SP30" x="21.59" y="-16.51"/>
+<element name="IC1" library="motorola-sensor-driver" package="DIL24S" value="33035P" x="25.4" y="-39.37">
+<attribute name="MF" value="ON SEMICONDUCTOR" x="25.4" y="-39.37" size="1.778" layer="27" display="off"/>
+<attribute name="MPN" value="MC33035P" x="25.4" y="-39.37" size="1.778" layer="27" display="off"/>
+<attribute name="OC_FARNELL" value="1192056" x="25.4" y="-39.37" size="1.778" layer="27" display="off"/>
+<attribute name="OC_NEWARK" value="07F4698" x="25.4" y="-39.37" size="1.778" layer="27" display="off"/>
 </element>
 </elements>
@@
 <via x="58.42" y="10.16" extent="1-16" drill="0.35"/>
 <via x="93.98" y="10.795" extent="1-16" drill="0.35"/>
+<contactref element="IC1" pad="16"/>
+<wire x1="31.75" y1="-35.56" x2="31.75" y2="6.985" width="0" layer="19" extent="16-16"/>
 </signal>
 <signal name="D3">
@@
 <wire x1="37.465" y1="5.08" x2="36.87" y2="5.08" width="0.635" layer="1"/>
 </signal>
+<signal name="VCC">
+<contactref element="IC1" pad="17"/>
+</signal>
+<signal name="VC">
+<contactref element="IC1" pad="18"/>
+</signal>
 </signals>

Commit message: M
Mm
Parts:
- removed IC1: 33035P, motorola-sensor-driver:DIL24S
- removed U$1: VNH2SP30, SparkFun-IC-Special-Function:VNH2SP30
Connections:
- removed net VC: IC1.18
- removed net VCC: IC1.17
- net GND: no longer IC1.16
Changed lines of the file:
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@@
 <attribute name="OC_NEWARK" value="70K9898" x="39.37" y="6.35" size="1.778" layer="27" display="off"/>
-</element>
-<element name="U$1" library="SparkFun-IC-Special-Function" package="VNH2SP30" value="VNH2SP30" x="21.59" y="-16.51"/>
-<element name="IC1" library="motorola-sensor-driver" package="DIL24S" value="33035P" x="25.4" y="-39.37">
-<attribute name="MF" value="ON SEMICONDUCTOR" x="25.4" y="-39.37" size="1.778" layer="27" display="off"/>
-<attribute name="MPN" value="MC33035P" x="25.4" y="-39.37" size="1.778" layer="27" display="off"/>
-<attribute name="OC_FARNELL" value="1192056" x="25.4" y="-39.37" size="1.778" layer="27" display="off"/>
-<attribute name="OC_NEWARK" value="07F4698" x="25.4" y="-39.37" size="1.778" layer="27" display="off"/>
 </element>
 </elements>
@@
 <via x="58.42" y="10.16" extent="1-16" drill="0.35"/>
 <via x="93.98" y="10.795" extent="1-16" drill="0.35"/>
-<contactref element="IC1" pad="16"/>
-<wire x1="31.75" y1="-35.56" x2="31.75" y2="6.985" width="0" layer="19" extent="16-16"/>
 </signal>
 <signal name="D3">
@@
 <wire x1="37.465" y1="5.08" x2="36.87" y2="5.08" width="0.635" layer="1"/>
 </signal>
-<signal name="VCC">
-<contactref element="IC1" pad="17"/>
-</signal>
-<signal name="VC">
-<contactref element="IC1" pad="18"/>
-</signal>
 </signals>

Commit message: Z
z
Parts:
- removed RESITOR+1, RESITOR+2, RESITOR+3, RESITOR+4, RESITOR+5, RESITOR+6, RESITOR-1, RESITOR-2, RESITOR-3, RESITOR-4, RESITOR-5, RESITOR-6: (no value), adafruit:1X01
- added R1, R2, R3, R4, R5, R6: (no value), BaseApp:R0603
Connections:
- net D2: now also R3.1; no longer RESITOR+4.1
- net D3: now also R4.1; no longer RESITOR+1.1
- net D4: now also R5.1; no longer RESITOR+2.1
- net D5: now also R6.1; no longer RESITOR+3.1
- net D6: now also R1.1; no longer RESITOR+5.1
- net D7: now also R2.1; no longer RESITOR+6.1
- net N$1: now also R4.2; no longer RESITOR-1.1
- net N$12: now also R2.2; no longer RESITOR-6.1
- net N$3: now also R3.2; no longer RESITOR-4.1
- net N$5: now also R5.2; no longer RESITOR-2.1
- net N$7: now also R6.2; no longer RESITOR-3.1
- net N$9: now also R1.2; no longer RESITOR-5.1
Routing:
- net 5.5V: track 500.0 -> 547.7 mm
- net N$7: track 46.6 -> 4.66 mm, vias 1 -> 0
- net BAT+: track 367.5 -> 327.9 mm, vias 1 -> 2
- net SCL: track 283.5 -> 318.9 mm
- net D6: track 143.0 -> 110.7 mm
- net 3.3V: track 211.2 -> 242.0 mm, vias 1 -> 2
- net D5: track 127.5 -> 100.8 mm
- net D9: track 85.1 -> 62.6 mm, vias 0 -> 1
- net D11: track 147.9 -> 169.8 mm, vias 1 -> 2
- net GND: track 686.1 -> 664.2 mm, vias 4 -> 1
- net D13: track 116.5 -> 95.6 mm
- net N$9: track 20.3 -> 4.81 mm
- net D2: track 98.2 -> 113.5 mm
- net SDA: track 299.8 -> 285.8 mm, vias 2 -> 1
- net D7: track 155.3 -> 143.3 mm, vias 0 -> 2
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