File: Soccerbot/Nsoccerbots.brd (EAGLE design)
At the start: 146 x 100 mm, 53 parts, among them X1 NXT-SOCKET, X2 NXT-SOCKET, X3 NXT-SOCKET, X4 NXT-SOCKET

Commit message: k
J
Parts:
- turned IR1 to 270 degrees
- turned IR3 to 180 degrees
- turned IR4 to 90 degrees
Routing:
- net D4: track 139.4 -> 309.2 mm, vias 2 -> 6
- net BAT+: track 327.9 -> 482.4 mm, vias 2 -> 0
- net N$11: track 44.4 -> 194.1 mm, vias 1 -> 4
- net BAT-: track 368.5 -> 502.9 mm, vias 1 -> 0
- net D2: track 113.5 -> 185.3 mm, vias 0 -> 2
- net D6: track 110.7 -> 173.7 mm, vias 3 -> 5
- net VIN: track 411.8 -> 468.2 mm, vias 3 -> 12
- net 3.3V: track 242.0 -> 197.5 mm, vias 2 -> 5
- net SDA: track 285.8 -> 314.9 mm, vias 1 -> 5
- net 5.5V: track 547.7 -> 572.3 mm, vias 1 -> 4
- net D12: track 130.6 -> 151.5 mm, vias 3 -> 5
- net GND: track 664.2 -> 682.5 mm, vias 1 -> 6
- net D9: track 62.6 -> 76.3 mm, vias 1 -> 3
- net N$13: track 40.8 -> 53.3 mm, vias 2 -> 3
- net D11: track 169.8 -> 157.6 mm, vias 2 -> 3
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Other:
- board text added: "3v3"
- board text added: "SCL"
- board text added: "SDA"
- board text added: "___ 3v3"
