File: GYRO/ASD2421.sch (EAGLE design)
At the start: 11 parts, among them J2 DF12-32-DS

Commit message: nk
kk
Parts:
- removed C1, C2, C3: 0.1uF, tinycircuits:AS-ITM-00008
- removed J2: DF12-32-DS, tinycircuits:AS-ITM-00012
- removed U$2, U$3: AS-ITM-00133, tinycircuits:AS-ITM-00133
- removed U$4: AS-ITM-00134, tinycircuits:AS-ITM-00134
- removed U$5, U$6, U$7, U$8: AS-ITM-00135, tinycircuits:AS-ITM-00135
Connections:
- removed net +3V3: J2.6
- removed net +5V: J2.8
- removed net AD0: J2.11
- removed net AD1: J2.9
- removed net AD2: J2.7
- removed net AD3: J2.5
- removed net AD4/SDA: J2.3, U$4.SDA
- removed net AD5/SCL: J2.1, U$4.SCL
- removed net AREF: J2.13
- removed net GND: C1.2, C2.2, C3.2, J2.12, J2.14, U$4.GND, U$4.GND2, U$4.GND3, U$4.GND4, U$4.GNDPAD
- removed net GPIO0: U$2.A, U$6.6
- removed net GPIO1: U$2.B, U$6.8
- removed net GPIO10: U$3.C, U$5.2
- removed net GPIO11: U$3.D, U$5.4
- removed net GPIO12: U$3.E, U$5.6
- removed net GPIO13: U$3.F, U$5.8
- removed net GPIO14: U$3.G, U$6.2
- removed net GPIO15: U$3.DP, U$6.4
- removed net GPIO2: U$2.C, U$8.7
- removed net GPIO3: U$2.D, U$8.5
- removed net GPIO4: U$2.E, U$8.3
- removed net GPIO5: U$2.F, U$8.1
- removed net GPIO6: U$2.G, U$7.7
- removed net GPIO7: U$2.DP, U$7.5
- removed net GPIO8: U$3.A, U$7.3
- removed net GPIO9: U$3.B, U$7.1
- removed net IO0: J2.24
- removed net IO1: J2.26
- removed net IO2: J2.28
- removed net IO3: J2.30
- removed net IO4: J2.32
- removed net IO5: J2.31
- removed net IO6: J2.29
- removed net IO7: J2.27
- removed net IO8: J2.25
- removed net IO9: J2.23
- removed net MISO: J2.17
- removed net MOSI: J2.19
- removed net N$1: U$4.IO9, U$7.2
- removed net N$10: U$4.IO2, U$8.8
- removed net N$19: U$4.IO10, U$5.1
- removed net N$2: U$4.IO8, U$7.4
- removed net N$20: U$4.IO11, U$5.3
- removed net N$21: U$4.IO12, U$5.5
- removed net N$22: U$4.IO13, U$5.7
- removed net N$23: U$4.IO14, U$6.1
- removed net N$24: U$4.IO15, U$6.3
- removed net N$25: U$4.IO0, U$6.5
- removed net N$26: U$4.IO1, U$6.7
- removed net N$3: U$4.IO7, U$7.6
- removed net N$4: U$4.IO6, U$7.8
- removed net N$6: U$4.IO5, U$8.2
- removed net N$7: U$4.IO4, U$8.4
- removed net N$9: U$4.IO3, U$8.6
- removed net RESET: J2.22
- removed net RSV0: J2.20
- removed net RSV1: J2.18
- removed net RSV2: J2.16
- removed net SCK: J2.15
- removed net SS: J2.21
- removed net VBATT: J2.4
- removed net VCC: C1.1, C2.1, C3.1, J2.2, U$2.VCC, U$2.VCC1, U$3.VCC, U$3.VCC1, U$4.NINT, U$4.NRESET, U$4.VCC1, U$4.VCC2, U$4.VDDM
- removed net VIN: J2.10
Other:
- note removed: "1"
- note removed: "7 Segment Display Board"
- note removed: "AS-SCH-ASD2421"
- note removed: "IOREF"
- note removed: "LilyPad Arduino Design by Leah Buechley and Sparkfun Electronics"
- note removed: "Original Arduino Uno Design by Team Arduino"
- note removed: "Released under the Creative Commons Attribution Share-Alike 3.0 License"
- note removed: "TinyDuino, TinyLily and TinyShield Designs by TinyCircuits"
- note removed: "TinyShield Expansion - Bottom"
- note removed: "http://creativecommons.org/licenses/by-sa/3.0"
