File: GYRO/COMP.sch (EAGLE design)
At the start: 115 parts, among them J1 3013, J10 PIN_1X.1"1, J11 DF12-32-DS, J12 DF12-32-DP, J13 DF12-32-DS, J14 47346-0001, J15 47346-0001, J16 DF12-32-DS, J17 DF12-32-DS, J2 DF12-32-DP, J3 961102, J4 SM02B-SRSS-TB(LF)(SN), J5 DF12-32-DP, J6 DF12-32-DS, J7 PIN_1X.1"1, J8 PIN_1X.1"1, J9 PIN_1X.1"1, Q1 DMP2035U, Q2 DMP2035U, SW1 PCM12SMTR, U1 ATMEGA328P, U10 LSM9DS1, U11 BMP280, U12 FT231XQ-R, U2 MCP73831, U3 TX0102, U4 XC6217A33, U5 BMA250, U6 HMC5883L, U7 L3G4200D, U8 SI7020-A10-GM1, U9 TSL2572, Y1 8.00MHZ

Commit message: nk
kk
Parts:
- removed C10: .22uF, tinycircuits:AS-ITM-00087
- removed C11, C12, C20, C22, C26: 10uF, tinycircuits:AS-ITM-00002
- removed C13, C14, C15, C16, C17, C18, C19, C21, C23, C24, C25, C27, C28, C29, C32, C33, C34, C35, C36, C37, C6, C7: 0.1uF, tinycircuits:AS-ITM-00008
- removed C30, C31: 47pF, tinycircuits:AS-ITM-00241
- removed C8: 10nF, tinycircuits:AS-ITM-00084
- removed C9: 4.7uF, tinycircuits:AS-ITM-00242
- removed D5, D6: AMBER, tinycircuits:AS-ITM-00026
- removed J10, J7, J8, J9: PIN_1X.1"1, tinycircuits:PIN_1X.1"1
- removed J11, J13, J16, J17, J6: DF12-32-DS, tinycircuits:AS-ITM-00012
- removed J12, J5: DF12-32-DP, tinycircuits:AS-ITM-00015
- removed J14, J15: 47346-0001, tinycircuits:AS-ITM-00021
- removed Q1: DMP2035U, tinycircuits:AS-ITM-00024
- removed R10, R11: 0.0, tinycircuits:AS-ITM-00076
- removed R12: 0.0, tinycircuits:AS-ITM-000760402_SHORT
- removed R13, R14, R15, R16: 27.0, tinycircuits:AS-ITM-00240
- removed R17, R18, R7, R8, R9: 1.00K, tinycircuits:AS-ITM-00003
- removed U$1, U$15, U$16, U$2, U$3, U$9: AS-ITM-00133, tinycircuits:AS-ITM-00133
- removed U$10, U$17, U$4: AS-ITM-00134, tinycircuits:AS-ITM-00134
- removed U$11, U$12, U$13, U$14, U$18, U$19, U$20, U$21, U$5, U$6, U$7, U$8: AS-ITM-00135, tinycircuits:AS-ITM-00135
- removed U10: LSM9DS1, tinycircuits:AS-ITM-00265
- removed U11: BMP280, tinycircuits:AS-ITM-00264
- removed U12: FT231XQ-R, tinycircuits:AS-ITM-00223
- removed U3: TX0102, tinycircuits:AS-ITM-00073
- removed U4: XC6217A33, tinycircuits:AS-ITM-00249
- removed U5: BMA250, tinycircuits:AS-ITM-00070
- removed U6: HMC5883L, tinycircuits:AS-ITM-00086
- removed U7: L3G4200D, tinycircuits:AS-ITM-00089
- removed U8: SI7020-A10-GM1, tinycircuits:AS-ITM-00218
- removed U9: TSL2572, tinycircuits:AS-ITM-00116
- C2, C4: value 0.1uF -> .1uF
Connections:
- removed net 3V3OUT: C28.1, R11.1, R7.2, R8.2, U12.3V3OUT, U12.RESET, U12.VCCIO
- removed net DTR: C29.1, U12.DTR
- removed net GPIO0: U$1.A, U$12.6, U$15.A, U$19.6, U$2.A, U$6.6
- removed net GPIO1: U$1.B, U$12.8, U$15.B, U$19.8, U$2.B, U$6.8
- removed net GPIO10: U$11.2, U$16.C, U$18.2, U$3.C, U$5.2, U$9.C
- removed net GPIO11: U$11.4, U$16.D, U$18.4, U$3.D, U$5.4, U$9.D
- removed net GPIO12: U$11.6, U$16.E, U$18.6, U$3.E, U$5.6, U$9.E
- removed net GPIO13: U$11.8, U$16.F, U$18.8, U$3.F, U$5.8, U$9.F
- removed net GPIO14: U$12.2, U$16.G, U$19.2, U$3.G, U$6.2, U$9.G
- removed net GPIO15: U$12.4, U$16.DP, U$19.4, U$3.DP, U$6.4, U$9.DP
- removed net GPIO2: U$1.C, U$14.7, U$15.C, U$2.C, U$21.7, U$8.7
- removed net GPIO3: U$1.D, U$14.5, U$15.D, U$2.D, U$21.5, U$8.5
- removed net GPIO4: U$1.E, U$14.3, U$15.E, U$2.E, U$21.3, U$8.3
- removed net GPIO5: U$1.F, U$14.1, U$15.F, U$2.F, U$21.1, U$8.1
- removed net GPIO6: U$1.G, U$13.7, U$15.G, U$2.G, U$20.7, U$7.7
- removed net GPIO7: U$1.DP, U$13.5, U$15.DP, U$2.DP, U$20.5, U$7.5
- removed net GPIO8: U$13.3, U$16.A, U$20.3, U$3.A, U$7.3, U$9.A
- removed net GPIO9: U$13.1, U$16.B, U$20.1, U$3.B, U$7.1, U$9.B
- removed net N$10: C10.1, U6.SETP
- removed net N$11: C18.1, U7.PLLFILT
- removed net N$12: C8.1, U10.CAP
- removed net N$13: C7.1, U10.C1
- removed net N$14: U9.INT
- removed net N$15: U5.INT1
- removed net N$16: U5.INT2
- removed net N$17: U7.INT2
- removed net N$18: U7.INT1
- removed net N$19: U10.DRDY_M
- removed net N$20: U10.INT_M
- removed net N$21: U10.INT1_AG
- removed net N$22: U10.INT2_AG
- removed net N$23: U$4.IO9, U$7.2
- removed net N$24: U$4.IO8, U$7.4
- removed net N$25: U$4.IO7, U$7.6
- removed net N$26: U$4.IO6, U$7.8
- removed net N$27: U$4.IO5, U$8.2
- removed net N$28: U$4.IO4, U$8.4
- removed net N$29: U$4.IO3, U$8.6
- removed net N$30: U$4.IO2, U$8.8
- removed net N$31: U$4.IO10, U$5.1
- removed net N$32: U$4.IO11, U$5.3
- removed net N$33: U$4.IO12, U$5.5
- removed net N$34: U$4.IO13, U$5.7
- removed net N$35: U$4.IO14, U$6.1
- removed net N$36: U$4.IO15, U$6.3
- removed net N$37: U$4.IO0, U$6.5
- removed net N$38: U$4.IO1, U$6.7
- removed net N$39: D5.C, U12.CBUS1
- removed net N$40: D6.C, U12.CBUS2
- removed net N$41: D5.A, R7.1
- removed net N$42: D6.A, R8.1
- removed net N$43: Q1.D, R10.2, R11.2
- removed net N$44: J14.2, R13.1
- removed net N$45: J14.3, R14.1
- removed net N$46: J15.2, R15.1
- removed net N$47: J15.3, R16.1
- removed net N$48: R17.2, U12.RXD
- removed net N$49: R18.2, U12.TXD
- removed net N$50: U$10.IO9, U$13.2
- removed net N$51: U$10.IO8, U$13.4
- removed net N$52: U$10.IO7, U$13.6
- removed net N$53: U$10.IO6, U$13.8
- removed net N$54: U$10.IO5, U$14.2
- removed net N$55: U$10.IO4, U$14.4
- removed net N$56: U$10.IO3, U$14.6
- removed net N$57: U$10.IO2, U$14.8
- removed net N$58: U$10.IO10, U$11.1
- removed net N$59: U$10.IO11, U$11.3
- removed net N$60: U$10.IO12, U$11.5
- removed net N$61: U$10.IO13, U$11.7
- removed net N$62: U$10.IO14, U$12.1
- removed net N$63: U$10.IO15, U$12.3
- removed net N$64: U$10.IO0, U$12.5
- removed net N$65: U$10.IO1, U$12.7
- removed net N$66: U$17.IO9, U$20.2
- removed net N$67: U$17.IO8, U$20.4
- removed net N$68: U$17.IO7, U$20.6
- removed net N$69: U$17.IO6, U$20.8
- removed net N$70: U$17.IO5, U$21.2
- removed net N$71: U$17.IO4, U$21.4
- removed net N$72: U$17.IO3, U$21.6
- removed net N$73: U$17.IO2, U$21.8
- removed net N$74: U$17.IO10, U$18.1
- removed net N$75: U$17.IO11, U$18.3
- removed net N$76: U$17.IO12, U$18.5
- removed net N$77: U$17.IO13, U$18.7
- removed net N$78: U$17.IO14, U$19.1
- removed net N$79: U$17.IO15, U$19.3
- removed net N$8: C9.1, U6.C1
- removed net N$80: U$17.IO0, U$19.5
- removed net N$81: U$17.IO1, U$19.7
- removed net N$9: C10.2, U6.SETC
- removed net RTS: R12.1, U12.RTS
- removed net SCL_3V3: U10.SCL/SPC, U11.SCK, U3.A1, U5.SCX, U6.SCL, U7.SCL, U8.SCL, U9.SCL
- removed net SDA_3V3: U10.SDA/SDI, U11.SDI, U3.A2, U5.SDX, U6.SDA, U7.SDA, U8.SDA, U9.SDA
- removed net USBDM: C30.1, R13.2, R15.2, U12.USBDM
- removed net USBDP: C31.1, R14.2, R16.2, U12.USBDP
- removed net USBVCC: C26.1, C27.1, J14.1, J15.1, R10.1, U12.VCC
- removed net VCC_3V3: C12.1, C13.1, C14.1, C15.1, C16.1, C17.1, C19.1, C20.1, C21.1, C22.1, U10.CS_AG, U10.CS_M, U10.VDD, U10.VDDIO, U11.CSB, U11.SDO, U11.VDD, U11.VDDIO, U3.OE, U3.VCCA, U4.VOUT, U5.PS, U5.VDD, U5.VDDIO, U6.S1, U6.VDD, U6.VDDIO, U7.CS, U7.RESV_VDD, U7.SA0, U7.VDD, U7.VDD_IO, U8.VCC, U9.VDD
- net +3V3: no longer J11.6, J12.6, J13.6, J16.6, J17.6, J5.6, J6.6
- net +5V: no longer J11.8, J12.8, J13.8, J16.8, J17.8, J5.8, J6.8, Q1.S
- net AD0: no longer J11.11, J12.11, J13.11, J16.11, J17.11, J5.11, J6.11
- net AD1: no longer J11.9, J12.9, J13.9, J16.9, J17.9, J5.9, J6.9
- net AD2: no longer J11.7, J12.7, J13.7, J16.7, J17.7, J5.7, J6.7
- net AD3: no longer J11.5, J12.5, J13.5, J16.5, J17.5, J5.5, J6.5
- net AD4/SDA: no longer J11.3, J12.3, J13.3, J16.3, J17.3, J5.3, J6.3, J8.1, U$10.SDA, U$17.SDA, U$4.SDA, U3.B2
- net AD5/SCL: no longer J11.1, J12.1, J13.1, J16.1, J17.1, J5.1, J6.1, J9.1, U$10.SCL, U$17.SCL, U$4.SCL, U3.B1
- net AREF: no longer J11.13, J12.13, J13.13, J16.13, J17.13, J5.13, J6.13
- net GND: no longer C11.2, C12.2, C13.2, C14.2, C15.2, C16.2, C17.2, C18.2, C19.2, C20.2, C21.2, C22.2, C23.2, C24.2, C25.2, C26.2, C27.2, C28.2, C30.2, C31.2, C32.2, C33.2, C34.2, C35.2, C36.2, C37.2, C6.2, C7.2, C8.2, C9.2, J10.1, J11.12, J11.14, J12.12, J12.14, J13.12, J13.14, J14.5, J14.P1, J14.P2, J14.P3, J14.P4, J14.P5, J14.P6, J15.5, J15.P1, J15.P2, J15.P3, J15.P4, J15.P5, J15.P6, J16.12, J16.14, J17.12, J17.14, J5.12, J5.14, J6.12, J6.14, R9.1, U$10.GND, U$10.GND2, U$10.GND3, U$10.GND4, U$10.GNDPAD, U$17.GND, U$17.GND2, U$17.GND3, U$17.GND4, U$17.GNDPAD, U$4.GND, U$4.GND2, U$4.GND3, U$4.GND4, U$4.GNDPAD, U10.DEN_AG, U10.GND, U10.SDO_AG, U10.SDO_M, U11.GND, U12.GND0, U12.GND1, U12.GND2, U3.GND, U4.NC/GO, U4.VSS, U5.GND, U5.GNDIO, U5.SDO, U6.GND, U6.GND1, U7.GND, U7.GND1, U7.GND2, U7.GND3, U7.GND4, U7.GND5, U8.GND, U9.GND
- net IO0: no longer J11.24, J12.24, J13.24, J16.24, J17.24, J5.24, J6.24, R18.1
- net IO1: no longer J11.26, J12.26, J13.26, J16.26, J17.26, J5.26, J6.26, R17.1
- net IO2: no longer J11.28, J12.28, J13.28, J16.28, J17.28, J5.28, J6.28
- net IO3: no longer J11.30, J12.30, J13.30, J16.30, J17.30, J5.30, J6.30
- net IO4: no longer J11.32, J12.32, J13.32, J16.32, J17.32, J5.32, J6.32
- net IO5: no longer J11.31, J12.31, J13.31, J16.31, J17.31, J5.31, J6.31
- net IO6: no longer J11.29, J12.29, J13.29, J16.29, J17.29, J5.29, J6.29
- net IO7: no longer J11.27, J12.27, J13.27, J16.27, J17.27, J5.27, J6.27
- net IO8: no longer J11.25, J12.25, J13.25, J16.25, J17.25, J5.25, J6.25
- net IO9: no longer J11.23, J12.23, J13.23, J16.23, J17.23, J5.23, J6.23
- net MISO: no longer J11.17, J12.17, J13.17, J16.17, J17.17, J5.17, J6.17
- net MOSI: no longer J11.19, J12.19, J13.19, J16.19, J17.19, J5.19, J6.19
- net RESET: no longer C29.2, J11.22, J12.22, J13.22, J16.22, J17.22, J5.22, J6.22
- net RSV0: no longer J11.20, J12.20, J13.20, J16.20, J17.20, J5.20, J6.20
- net RSV1: no longer J11.18, J12.18, J13.18, J16.18, J17.18, J5.18, J6.18
- net RSV2: no longer J11.16, J12.16, J13.16, J16.16, J17.16, J5.16, J6.16, R12.2
- net SCK: no longer J11.15, J12.15, J13.15, J16.15, J17.15, J5.15, J6.15
- net SS: no longer J11.21, J12.21, J13.21, J16.21, J17.21, J5.21, J6.21
- net VBATT: no longer J11.4, J12.4, J13.4, J16.4, J17.4, J5.4, J6.4
- net VCC: no longer C11.1, C23.1, C24.1, C25.1, C32.1, C33.1, C34.1, C35.1, C36.1, C37.1, C6.1, J11.2, J12.2, J13.2, J16.2, J17.2, J5.2, J6.2, J7.1, U$1.VCC, U$1.VCC1, U$10.NINT, U$10.NRESET, U$10.VCC1, U$10.VCC2, U$10.VDDM, U$15.VCC, U$15.VCC1, U$16.VCC, U$16.VCC1, U$17.NINT, U$17.NRESET, U$17.VCC1, U$17.VCC2, U$17.VDDM, U$2.VCC, U$2.VCC1, U$3.VCC, U$3.VCC1, U$4.NINT, U$4.NRESET, U$4.VCC1, U$4.VCC2, U$4.VDDM, U$9.VCC, U$9.VCC1, U3.VCCB, U4.CE, U4.VIN
- net VIN: no longer J11.10, J12.10, J13.10, J16.10, J17.10, J5.10, J6.10, Q1.G, R9.2
Other:
- note removed: "1"
- note removed: "3.3V Out: Pop R5 (50mA Max)"
- note removed: "3.3V Power Supply"
- note removed: "5"
- note removed: "5V Out: Pop R4 (Default)"
- note removed: "6"
- note removed: "7 Segment Display Board"
- note removed: "9 Axis"
- note removed: "AS-SCH-ASD2101"
- note removed: "AS-SCH-ASD2421"
- note removed: "AS-SCH-ASD2511"
- note removed: "Accelerometer"
- note removed: "Ambient Light"
- note removed: "External Connections"
- note removed: "Gyro"
- note removed: "I2C Level Shifter"
- note removed: "Magnetometer"
- note removed: "Micro USB"
- note removed: "Pressure"
- note removed: "Temp and Humidity"
- note removed: "TinyShield - Sensor Board"
- note removed: "TinyShield - USB & ICP"
- note removed: "TinyShield Expansion - Bottom"
- note removed: "USB Power Option:"
