File: GYRO/COMP.sch (EAGLE design)
At the start: 59 parts, among them J10 SM02B-SRSS-TB(LF)(SN), J11 47346-0001, J12 EVP-ANDA1A, J13 EVP-ANDA1A, J14 EVP-ANDA1A, J15 EVP-ANDA1A, J3 PIN_1X.1", J4 PIN_1X.1", J5 PIN_1X.1", J6 PIN_1X.1", J7 PIN_1X.1", J8 PIN_1X.1", Q1 DMP2035U, SW1 PCM12SMTR, U1 XC6210B33, U2 TX0102, U3 MCP73831, U4 L3G4200D, U5 ATSAMD21G18A, U6 XC6210B33, U7 UG-9664HDDAG01, U8 FAN5340, Y1 32.7680

Commit message: as
as
Parts:
- C1, C3, C4: MPN (none) -> GRM155R61A104JA01D; OC_NEWARK (none) -> 03AC2559
- C10: MF (none) -> BC COMPONENTS; MPN (none) -> VJ0402V103ZXACW1BC; OC_NEWARK (none) -> 57J7497
- C11, C12, C14, C17, C18: MPN (none) -> GRM155R61C104KA88D; OC_NEWARK (none) -> 03AC2568
- C13: MPN (none) -> C0603X5R0J474K030BC; OC_NEWARK (none) -> 78Y9870
- C15, C16: MF (none) -> KEMET; MPN (none) -> C0402C220C5GACTU; OC_NEWARK (none) -> 01E9918
- C19, C2, C20, C5: MF (none) -> Taiyo Yuden (U.S.A.), Inc.; MPN (none) -> LMK212BJ106KG-T; OC_NEWARK (none) -> 18J2720
- C21: MPN (none) -> TAJA475K020RNJ; OC_NEWARK (none) -> 60R5858
- C22: MPN (none) -> C0402C475M9PACTU; OC_NEWARK (none) -> 23AC3655
- C6, C7, C8: MPN (none) -> C0603X5R1A104K030BC; OC_NEWARK (none) -> 04X3188
- C9: MPN (none) -> GRM155R60J474KE19D; OC_NEWARK (none) -> 03AC2556
- D1: MPN (none) -> MBR120LSFT1G; OC_NEWARK (none) -> 10N9423
- D2: MPN (none) -> LNJ426W83RA1; OC_NEWARK (none) -> 43W4882
- D3: MF (none) -> BOURNS, INC.; MPN (none) -> CD0603-S01575; OC_NEWARK (none) -> 02J1227
- J10: MPN (none) -> SM02B-SRSS-TB (LF)(SN); OC_NEWARK (none) -> 33P8179
- J11: MPN (none) -> 47346-0001; OC_NEWARK (none) -> 47M0505
- J12, J13, J14, J15: MPN (none) -> EVP-ANDA1A; OC_NEWARK (none) -> 52W2464
- J3, J4, J5, J6, J7, J8, L1, R2, R5, SW1, U1, U2, U3, U4, U5, U6, U7, U8, Y1: OC_NEWARK (none) -> unknown
- Q1: MPN (none) -> DMP2035U; OC_NEWARK (none) -> 65T8230
- R1: MF (none) -> VISHAY/DALE; MPN (none) -> CRCW120610K0FKTA; OC_NEWARK (none) -> 05F1568
- R10: MPN (none) -> 373-4.7K; OC_NEWARK (none) -> 82T4833
- R3: MPN (none) -> CRG0402J100K/10; OC_NEWARK (none) -> 20R1174
- R4: MF (none) -> VISHAY/DALE; MPN (none) -> CRCW04021K00FKTD; OC_NEWARK (none) -> 07J7497
- R6: MPN (none) -> CPF0402B115KE1; OC_NEWARK (none) -> 05AC7931
- R7, R8, R9: MPN (none) -> TNPW040210K0BEED; OC_NEWARK (none) -> 11R2753
