File: GYRO/ASD2614.sch (EAGLE design)
At the start: 26 parts, among them J1 47346-0001, J2 DF12-32-DS, J3 47346-0001, J4 DF12-32-DP, Q1 DMP2035U, U2 FT231XQ-R

Commit message: asdsa
asd
Parts:
- removed D1, D2: AMBER, tinycircuits:AS-ITM-00026
- removed Q1: DMP2035U, tinycircuits:AS-ITM-00024
- removed R10, R7, R8, R9: 27.0, tinycircuits:AS-ITM-00240
- removed R11, R12, R2, R3: 1.00K, tinycircuits:AS-ITM-00003
- removed R4, R5: 0.0, tinycircuits:AS-ITM-00076
- removed R6: 0.0, tinycircuits:AS-ITM-000760402_SHORT
- added C10: 10nF, tinycircuits:AS-ITM-00084
- added C9: 0.47uF, tinycircuits:AS-ITM-00090
- added J5, J6, J7, J8: PIN_1X.1", tinycircuits:PIN_1X.1"
- added U1: XC6210B33, tinycircuits:AS-ITM-00046
- added U4: L3G4200D, tinycircuits:AS-ITM-00089
- C2: value 0.1uF -> 10uF; device tinycircuits:AS-ITM-00008 -> tinycircuits:AS-ITM-00045; PARTNO (none) -> AS-ITM-00045; VALUE (none) -> 10uF
- C3: value 10uF -> 0.1uF; device tinycircuits:AS-ITM-00002 -> tinycircuits:AS-ITM-00008; PARTNO (none) -> AS-ITM-00008; VALUE (none) -> 0.1uF
- C4: PARTNO AS-ITM-00008 -> (none); VALUE 0.1uF -> (none)
- C5: value 47pF -> 10uF; device tinycircuits:AS-ITM-00241 -> tinycircuits:AS-ITM-00045; PARTNO AS-ITM-00241 -> (none); VALUE 47pF -> (none)
- C6: value 47pF -> 10uF; device tinycircuits:AS-ITM-00241 -> tinycircuits:AS-ITM-00002; PARTNO AS-ITM-00241 -> (none); VALUE 47pF -> (none)
- J1: value 47346-0001 -> DF12-32-DP; device tinycircuits:AS-ITM-00021 -> tinycircuits:AS-ITM-00015; PARTNO AS-ITM-00021 -> AS-ITM-00015; VALUE (none) -> DF12-32-DP
- J3: value 47346-0001 -> PIN_1X.1"; device tinycircuits:AS-ITM-00021 -> tinycircuits:PIN_1X.1"; PARTNO AS-ITM-00021 -> (none)
- J4: value DF12-32-DP -> PIN_1X.1"; device tinycircuits:AS-ITM-00015 -> tinycircuits:PIN_1X.1"; PARTNO AS-ITM-00015 -> (none); VALUE DF12-32-DP -> (none)
- R1: value 1.00K -> 10.0K; device tinycircuits:AS-ITM-00003 -> tinycircuits:AS-ITM-00032
- U2: value FT231XQ-R -> TX0102; device tinycircuits:AS-ITM-00223 -> tinycircuits:AS-ITM-00073
Connections:
- removed net 3V3OUT: C4.1, R1.2, R2.2, R5.1, U2.3V3OUT, U2.RESET, U2.VCCIO
- removed net DTR: C1.1, U2.DTR
- removed net N$10: R12.2, U2.TXD
- removed net N$16: D1.C, U2.CBUS1
- removed net N$3: J1.3, R10.1
- removed net N$4: Q1.D, R4.2, R5.2
- removed net N$5: D2.C, U2.CBUS2
- removed net N$6: D1.A, R1.1
- removed net N$7: D2.A, R2.1
- removed net N$8: J3.3, R8.1
- removed net N$9: R11.2, U2.RXD
- removed net RTS: R6.1, U2.RTS
- removed net USBDM: C5.1, R7.2, R9.2, U2.USBDM
- removed net USBDP: C6.1, R10.2, R8.2, U2.USBDP
- removed net USBVCC: C2.1, C3.1, J1.1, J3.1, R4.1, U2.VCC
- new net INT1: J7.1, U4.INT1
- new net INT2: J8.1, U4.INT2
- new net SCL_3V3: U2.A1, U4.SCL
- new net SDA_3V3: U2.A2, U4.SDA
- new net VCC_3V3: C2.1, C3.1, C4.1, C6.1, U1.VOUT, U2.OE, U2.VCCA, U4.CS, U4.RESV_VDD, U4.VDD, U4.VDD_IO
- net +3V3: now also J1.6; no longer J4.6
- net +5V: now also J1.8; no longer J4.8, Q1.S
- net AD0: now also J1.11; no longer J4.11
- net AD1: now also J1.9; no longer J4.9
- net AD2: now also J1.7; no longer J4.7
- net AD3: now also J1.5; no longer J4.5
- net AD4/SDA: now also J1.3, J4.1, U2.B2; no longer J4.3
- net AD5/SCL: now also J1.1, J5.1, U2.B1; no longer J4.1
- net AREF: now also J1.13; no longer J4.13
- net GND: now also C1.2, C10.2, J1.12, J1.14, J6.1, R1.2, U1.VSS, U2.GND, U4.GND, U4.GND1, U4.GND2, U4.GND3, U4.GND4, U4.GND5; no longer J1.5, J1.P1, J1.P2, J1.P3, J1.P4, J1.P5, J1.P6, J3.5, J3.P1, J3.P2, J3.P3, J3.P4, J3.P5, J3.P6, J4.12, J4.14, R3.1, U2.GND0, U2.GND1, U2.GND2
- net IO0: now also J1.24; no longer J4.24, R12.1
- net IO1: now also J1.26; no longer J4.26, R11.1
- net IO2: now also J1.28; no longer J4.28
- net IO3: now also J1.30; no longer J4.30
- net IO4: now also J1.32; no longer J4.32
- net IO5: now also J1.31; no longer J4.31
- net IO6: now also J1.29; no longer J4.29
- net IO7: now also J1.27; no longer J4.27
- net IO8: now also J1.25; no longer J4.25
- net IO9: now also J1.23; no longer J4.23
- net MISO: now also J1.17; no longer J4.17
- net MOSI: now also J1.19; no longer J4.19
- net N$1: now also C9.2, R1.1; no longer J3.2, R7.1
- net N$2: now also C10.1, C9.1, U4.PLLFILT; no longer J1.2, R9.1
- net RESET: now also J1.22; no longer C1.2, J4.22
- net RSV0: now also J1.20; no longer J4.20
- net RSV1: now also J1.18; no longer J4.18
- net RSV2: now also J1.16; no longer J4.16, R6.2
- net SCK: now also J1.15; no longer J4.15
- net SS: now also J1.21; no longer J4.21
- net VBATT: now also J1.4; no longer J4.4
- net VCC: now also C1.1, C5.1, J1.2, J3.1, U1.CE, U1.VIN, U2.VCCB; no longer J4.2
- net VIN: now also J1.10; no longer J4.10, Q1.G, R3.2
Other:
- note added: "1"
- note added: "3.3V Power Supply"
- note added: "AS-SCH-ASD2614"
- note added: "External Connections"
- note added: "I2C Level Shifter"
- note added: "STmicro L3G4200D"
- note added: "TinyShield - 3-Axis Gyro"
- note removed: "3.3V Out: Pop R5 (50mA Max)"
- note removed: "5V Out: Pop R4 (Default)"
- note removed: "6"
- note removed: "AS-SCH-ASD2101"
- note removed: "Micro USB"
- note removed: "TinyShield - USB & ICP"
- note removed: "USB Power Option:"
- moved on the sheet: C1, C2, C3, C4, C5, C6, J2, R1
