File: GYRO/ASM2022.sch (EAGLE design)
At the start: 59 parts, among them J10 SM02B-SRSS-TB(LF)(SN), J11 47346-0001, J12 EVP-ANDA1A, J13 EVP-ANDA1A, J14 EVP-ANDA1A, J15 EVP-ANDA1A, J3 PIN_1X.1", J4 PIN_1X.1", J5 PIN_1X.1", J6 PIN_1X.1", J7 PIN_1X.1", J8 PIN_1X.1", Q1 DMP2035U, SW1 PCM12SMTR, U1 XC6210B33, U2 TX0102, U3 MCP73831, U4 L3G4200D, U5 ATSAMD21G18A, U6 XC6210B33, U7 UG-9664HDDAG01, U8 FAN5340, Y1 32.7680

Commit message: asdsa
asd
Parts:
- removed C15, C16: 22pF, tinycircuits:AS-ITM-00211
- removed C17, C18: .1uF, tinycircuits:AS-ITM-00008
- removed C19, C20: 10uF, tinycircuits:AS-ITM-00045
- removed C21: 4.7uF, tinycircuits:AS-ITM-00232
- removed C22: 4.7uF, tinycircuits:AS-ITM-00242
- removed J10: SM02B-SRSS-TB(LF)(SN), tinycircuits:AS-ITM-00231
- removed J11: 47346-0001, tinycircuits:AS-ITM-00021
- removed J12, J13, J14, J15: EVP-ANDA1A, tinycircuits:AS-ITM-00236
- removed J8: PIN_1X.1", tinycircuits:PIN_1X.1"
- removed R10: 4.7k, tinycircuits:AS-ITM-00167
- removed U6: XC6210B33, tinycircuits:AS-ITM-00046
- removed U7: UG-9664HDDAG01, tinycircuits:AS-ITM-00158
- removed U8: FAN5340, tinycircuits:AS-ITM-00277
- added J1: SM02B-SRSS-TB(LF)(SN), tinycircuits:AS-ITM-00231
- added J2: 47346-0001, tinycircuits:AS-ITM-00021
- C1: value 0.1uF -> 4.7uF; device tinycircuits:AS-ITM-00008 -> tinycircuits:AS-ITM-00088; PARTNO AS-ITM-00008 -> AS-ITM-00088; VALUE 0.1uF -> 4.7uF
- C10: value 10nF -> 10uF; device tinycircuits:AS-ITM-00084 -> tinycircuits:AS-ITM-00045; PARTNO (none) -> AS-ITM-00045; VALUE (none) -> 10uF
- C13: value 4.7uF -> .1uF; device tinycircuits:AS-ITM-00088 -> tinycircuits:AS-ITM-00008; PARTNO AS-ITM-00088 -> AS-ITM-00008; VALUE 4.7uF -> 0.1uF
- C2: VALUE 10uF -> (none)
- C3: value 0.1uF -> 10uF; device tinycircuits:AS-ITM-00008 -> tinycircuits:AS-ITM-00002; PARTNO AS-ITM-00008 -> AS-ITM-00002; VALUE 0.1uF -> 10uF
- C4: value 0.1uF -> 10uF; device tinycircuits:AS-ITM-00008 -> tinycircuits:AS-ITM-00002; PARTNO (none) -> AS-ITM-00002
- C5: value 10uF -> 22pF; device tinycircuits:AS-ITM-00045 -> tinycircuits:AS-ITM-00211; PARTNO (none) -> AS-ITM-00211; VALUE (none) -> 22pF
- C6: value 10uF -> 4.7uF; device tinycircuits:AS-ITM-00002 -> tinycircuits:AS-ITM-00232; PARTNO (none) -> AS-ITM-00232; VALUE (none) -> F931D475MAA
- C7: value 10uF -> 22pF; device tinycircuits:AS-ITM-00002 -> tinycircuits:AS-ITM-00211; PARTNO AS-ITM-00002 -> AS-ITM-00211; VALUE (none) -> 22pF
- C8: value 10uF -> 4.7uF; device tinycircuits:AS-ITM-00002 -> tinycircuits:AS-ITM-00242; PARTNO AS-ITM-00002 -> (none); VALUE 10uF -> (none)
- C9: value 0.47uF -> .1uF; device tinycircuits:AS-ITM-00090 -> tinycircuits:AS-ITM-00008; PARTNO (none) -> AS-ITM-00008; VALUE (none) -> 0.1uF
- J3, J4, J5, J7: value PIN_1X.1" -> EVP-ANDA1A; device tinycircuits:PIN_1X.1" -> tinycircuits:AS-ITM-00236; PARTNO (none) -> AS-ITM-00236; VALUE (none) -> PTS840 GKP
- J6: value PIN_1X.1" -> DF12-32-DP; device tinycircuits:PIN_1X.1" -> tinycircuits:AS-ITM-00015; PARTNO (none) -> AS-ITM-00015; VALUE (none) -> DF12-32-DP
- R1: value 10.0K -> 5K; device tinycircuits:AS-ITM-00032 -> tinycircuits:AS-ITM-00289
- R2: value 5K -> 1k; device tinycircuits:AS-ITM-00289 -> tinycircuits:AS-ITM-00003; PARTNO (none) -> AS-ITM-00003; VALUE (none) -> 1.00K
- R4: value 1k -> 1.2M; device tinycircuits:AS-ITM-00003 -> tinycircuits:AS-ITM-00280; PARTNO AS-ITM-00003 -> AS-ITM-00280; VALUE 1.00K -> 1.2M
- R5: value 1.2M -> 115k; device tinycircuits:AS-ITM-00280 -> tinycircuits:AS-ITM-00179; PARTNO AS-ITM-00280 -> (none); VALUE 1.2M -> 115K
- R6: value 115k -> 4.7k; device tinycircuits:AS-ITM-00179 -> tinycircuits:AS-ITM-00167; PARTNO (none) -> AS-ITM-00167; VALUE 115K -> 4.7K
- U2: value TX0102 -> MCP73831; device tinycircuits:AS-ITM-00073 -> tinycircuits:AS-ITM-00136
- U3: value MCP73831 -> UG-9664HDDAG01; device tinycircuits:AS-ITM-00136 -> tinycircuits:AS-ITM-00158
- U4: value L3G4200D -> FAN5340; device tinycircuits:AS-ITM-00089 -> tinycircuits:AS-ITM-00277
Connections:
- removed net INT1: J7.1, U4.INT1
- removed net INT2: J8.1, U4.INT2
- removed net N$10: L1.2, U8.SW
- removed net N$2 (its old number): C10.1, C9.1, U4.PLLFILT
- removed net N$4: C15.1, U5.PA00, Y1.1
- removed net SCL_3V3: U2.A1, U4.SCL
- removed net SDA_3V3: U2.A2, U4.SDA
- removed net VCC_3V3: C2.1, C3.1, C4.1, C6.1, U1.VOUT, U2.OE, U2.VCCA, U4.CS, U4.RESV_VDD, U4.VDD, U4.VDD_IO
- new net +3V3: J6.6
- new net N$3: C7.1, U5.PA01, Y1.2
- new net RSV2: J6.16
- new net VIN: J6.10
- net +12V: now also C10.1, U3.VCC, U4.VOUT; no longer C20.1, U7.VCC, U8.VOUT
- net +5V: now also C3.1, J2.1, J6.8, U2.VDD; no longer C8.1, J11.1, U3.VDD
- net AD0: now also J6.11
- net AD1: now also J6.9
- net AD2: now also J6.7
- net AD3: now also J6.5
- net AD4/SDA: now also J6.3; no longer J4.1, U2.B2
- net AD5: now also J3.1; no longer J12.1
- net AD5/SCL: now also J6.1; no longer J5.1, U2.B1
- net AREF: now also J6.13
- net ATN/IO38: now also U3.CS#; no longer U7.CS#
- net DBG_RXD: now also J7.1; no longer J14.1
- net DBG_TXD: now also J5.1; no longer J15.1
- net GND: now also C9.2, J1.2, J2.5, J2.P1, J2.P2, J2.P3, J2.P4, J2.P5, J2.P6, J3.2, J4.2, J5.2, J6.12, J6.14, J7.2, R4.1, R6.1, U2.VSS, U3.BS1, U3.BS2, U3.D3, U3.D4, U3.D5, U3.D6, U3.D7, U3.E, U3.R/W#, U4.PGND; no longer C15.2, C16.2, C17.2, C18.2, C19.2, C20.2, C21.2, C22.2, J10.2, J11.5, J11.P1, J11.P2, J11.P3, J11.P4, J11.P5, J11.P6, J12.2, J13.2, J14.2, J15.2, J6.1, R10.1, R2.2, R5.1, U2.GND, U4.GND1, U4.GND2, U4.GND3, U4.GND4, U4.GND5, U6.VSS, U7.BS1, U7.BS2, U7.D3, U7.D4, U7.D5, U7.D6, U7.D7, U7.E, U7.R/W#, U7.VSS, U8.GND, U8.PGND
- net IO0: now also J6.24
- net IO1: now also J6.26
- net IO2: now also J6.28
- net IO3: now also J6.30
- net IO4: now also J6.32
- net IO5: now also J6.31
- net IO6: now also J6.29
- net IO7: now also J6.27
- net IO8: now also J6.25
- net IO9: now also J6.23
- net MISO: now also J6.17
- net MISO_ALT: now also U3.D/C#; no longer U7.D/C#
- net MOSI: now also J6.19
- net MOSI_ALT: now also U3.D1; no longer U7.D1
- net N$1: now also C5.1, U5.PA00, Y1.1; no longer C9.2, R1.1
- net N$11: now also R4.2, U3.IREF; no longer R5.2, U7.IREF
- net N$12: now also C6.1, U3.VCOMH; no longer C21.1, U7.VCOMH
- net N$13: now also R5.1, U4.VLED; no longer R6.1, U8.VLED
- net N$15: now also U3.D2; no longer U7.D2
- net N$5: now also R2.1; no longer R4.1
- net N$6: now also R1.1, U2.PROG; no longer R2.1, U3.PROG
- net N$7: now also R2.2, U2.STAT; no longer R4.2, U3.STAT
- net N$8: now also C9.1, U5.VDDCORE; no longer C16.1, U5.PA01, Y1.2
- net N$9: now also L1.2, U4.SW; no longer C14.1, U5.VDDCORE
- net RESET: now also J6.22
- net RX_LED/IO25/AIN11: now also J4.1; no longer J13.1
- net SCK: now also J6.15
- net SCK_ALT: now also U3.D0; no longer U7.D0
- net SS: now also J6.21
- net SWCLK: now also J6.20
- net SWDIO: now also J6.18
- net TX_LED/IO26: now also U3.RES#; no longer U7.RES#
- net USB_HOST_EN/IO27: now also U4.SHDN; no longer U8.SHDN
- net USB_N: now also J2.2; no longer J11.2
- net USB_P: now also J2.3; no longer J11.3
- net VBATT: now also C1.1, J1.1, J6.4, U2.VBAT; no longer C13.1, J10.1, U3.VBAT
- net VCC: now also C13.1, C14.1, C4.1, J6.2, U1.VOUT, U3.VDD, U3.VDDIO; no longer C1.1, C17.1, C18.1, C5.1, C7.1, J3.1, U1.CE, U1.VIN, U2.VCCB, U6.VOUT, U7.VDD, U7.VDDIO
- net VCC_IN: now also C2.1, C8.1, U1.CE, U1.VIN, U4.VIN; no longer C19.1, C22.1, U6.CE, U6.VIN, U8.VIN
- net V_FB: now also R5.2, U4.FB; no longer R10.2, U8.FB
Other:
- note added: "IOREF"
- note added: "TinyShield Expansion - Top"
- note removed: "1"
- note removed: "3.3V Power Supply"
- note removed: "AS-SCH-ASD2614"
- note removed: "External Connections"
- note removed: "I2C Level Shifter"
- note removed: "STmicro L3G4200D"
- note removed: "TinyShield - 3-Axis Gyro"
