File: GYRO/Comp2/COMP2.sch (EAGLE design)
At the start: 15 parts, among them U2 LSM9DS0TR

Commit message: m
m
Parts:
- U$1: OC_NEWARK (none) -> unknown
Changed lines of the file:
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@@
 <attribute name="OC_NEWARK" value="97K1682"/>
 </part>
-<part name="U$1" library="SparkFun" deviceset="AVR_SPI_PRG_6" device="PTH"/>
+<part name="U$1" library="SparkFun" deviceset="AVR_SPI_PRG_6" device="PTH">
+<attribute name="MF" value=""/>
+<attribute name="MPN" value=""/>
+<attribute name="OC_NEWARK" value="unknown"/>
+</part>
 </parts>
 <sheets>
@@
 <attribute name="MPN" x="2.54" y="40.64" size="1.778" layer="96" display="off"/>
 </instance>
-<instance part="U$1" gate="G$1" x="119.38" y="78.74"/>
+<instance part="U$1" gate="G$1" x="119.38" y="78.74">
+<attribute name="OC_NEWARK" x="119.38" y="78.74" size="1.778" layer="96" display="off"/>
+<attribute name="MF" x="119.38" y="78.74" size="1.778" layer="96" display="off"/>
+<attribute name="MPN" x="119.38" y="78.74" size="1.778" layer="96" display="off"/>
+</instance>
 </instances>
 <busses>

Commit message: Z
z
Parts:
- U1: MPN (none) -> ATMEGA8A-MU; OC_NEWARK unknown -> 15AC6102
Changed lines of the file:
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@@
 <part name="U1" library="SparkFun-IC-Microcontroller" deviceset="ATMEGA328P_MLF" device="MLF32">
 <attribute name="MF" value=""/>
-<attribute name="MPN" value=""/>
-<attribute name="OC_NEWARK" value="unknown"/>
+<attribute name="MPN" value="ATMEGA8A-MU"/>
+<attribute name="OC_NEWARK" value="15AC6102"/>
 </part>
 <part name="JP1" library="SparkFun" deviceset="M08" device="LOCK">
