File: Soccerbot/V3/Nsoccerbots.brd (EAGLE design)
At the start: 146 x 100 mm, 65 parts, among them X1 NXT-SOCKET, X2 NXT-SOCKET, X3 NXT-SOCKET, X4 NXT-SOCKET

Commit message: K
M
Routing:
- net GND: track 0.00 -> 730.1 mm, vias 0 -> 6
- net 5.5V: track 0.00 -> 450.0 mm, vias 0 -> 8
- net VIN: track 0.00 -> 445.0 mm, vias 0 -> 10
- net SDA: track 0.00 -> 418.7 mm, vias 0 -> 7
- net BAT-: track 0.00 -> 413.9 mm
- net SCL: track 0.00 -> 396.9 mm, vias 0 -> 8
- net BAT+: track 0.00 -> 376.2 mm
- net 3.3V: track 0.00 -> 178.6 mm, vias 0 -> 4
- net D9: track 0.00 -> 176.7 mm, vias 0 -> 4
- net D23: track 0.00 -> 170.9 mm, vias 0 -> 3
- net D22: track 0.00 -> 165.1 mm, vias 0 -> 6
- net D4: track 0.00 -> 160.6 mm, vias 0 -> 3
- net D3: track 0.00 -> 160.2 mm, vias 0 -> 6
- net +3V3: track 0.00 -> 148.3 mm, vias 0 -> 4
- net D8: track 0.00 -> 141.9 mm, vias 0 -> 2
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Other:
- board size 146 x 100 mm -> 148.6 x 101.3 mm

Commit message: d
d
Routing:
- net D7: track 31.9 -> 187.6 mm, vias 3 -> 10
- net D10: track 5.40 -> 152.9 mm, vias 0 -> 9
- net D26: track 0.00 -> 107.2 mm, vias 0 -> 5
- net D5: track 29.3 -> 113.3 mm, vias 0 -> 6
- net D25: track 0.00 -> 79.6 mm
- net 3.3V: track 178.6 -> 245.4 mm, vias 4 -> 7
- net BAT+: track 376.2 -> 309.6 mm
- net N$18: track 0.00 -> 51.5 mm, vias 0 -> 4
- net GND: track 730.1 -> 771.9 mm, vias 6 -> 9
- net N$11: track 0.00 -> 37.0 mm, vias 0 -> 3
- net D23: track 170.9 -> 176.0 mm
- net N$16: track 0.00 -> 4.20 mm
- net VIN: track 445.0 -> 448.6 mm
- net D24: track 137.5 -> 140.9 mm
- net N$17: track 0.00 -> 3.18 mm
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Other:
- board size 148.6 x 101.3 mm -> 149.8 x 102.5 mm

Commit message: S
S
Parts:
- removed JP1, JP2: (no value), adafruit:1X03
- added ISP1: AVRISP-6, adafruit:AVRISP
Connections:
- new net VCC: ISP1.2
- net GND: now also ISP1.6
Routing:
- net GND: track 771.9 -> 795.2 mm, vias 9 -> 10
- net D3: track 160.2 -> 163.0 mm

Commit message: S
S
Routing:
- net D25: track 79.6 -> 77.5 mm
Other:
- board size 149.8 x 102.5 mm -> 149.8 x 101.3 mm
- board text added: "DATA"
- board text added: "POWER"
Changed lines of the file:
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@@
 <plain>
 <wire x1="10.16" y1="-1.27" x2="160" y2="-1.27" width="0" layer="20"/>
-<wire x1="160" y1="-1.27" x2="160" y2="101.27" width="0" layer="20"/>
-<wire x1="160" y1="101.27" x2="10.16" y2="101.27" width="0" layer="20"/>
-<wire x1="10.16" y1="101.27" x2="10.16" y2="-1.27" width="0" layer="20"/>
+<wire x1="160" y1="-1.27" x2="160" y2="100" width="0" layer="20"/>
+<wire x1="160" y1="100" x2="10.16" y2="100" width="0" layer="20"/>
+<wire x1="10.16" y1="100" x2="10.16" y2="-1.27" width="0" layer="20"/>
 <text x="66.04" y="15.24" size="0.6096" layer="25" rot="R90">SIGNAL</text>
 <text x="119.38" y="15.24" size="0.6096" layer="25" rot="R90">SIGNAL</text>
@@
 <text x="22.86" y="50.8" size="0.6096" layer="25" rot="R90">GND</text>
 <text x="31.75" y="50.8" size="0.6096" layer="25" rot="R90">SIGNAL</text>
-<dimension x1="12.7" y1="0" x2="158.75" y2="0" x3="85.725" y3="-2.54" textsize="0.6096" layer="25"/>
-<dimension x1="12.7" y1="100" x2="12.7" y2="0" x3="8.89" y3="50" textsize="0.6096" layer="25"/>
 <hole x="27.94" y="95.25" drill="0.35"/>
 <hole x="144.78" y="93.98" drill="0.35"/>
@@
 <text x="138.43" y="55.88" size="0.508" layer="25" rot="R90">SCL</text>
 <text x="68.58" y="27.94" size="1.016" layer="25" rot="R90">___ 3v3</text>
+<dimension x1="10.16" y1="-1.27" x2="160" y2="-1.27" x3="85.08" y3="-5.08" textsize="1.778" layer="20"/>
+<dimension x1="10.16" y1="100" x2="10.16" y2="-1.27" x3="6.35" y3="49.365" textsize="1.778" layer="20"/>
+<text x="19.05" y="96.52" size="0.508" layer="20" rot="R90">POWER</text>
+<text x="149.86" y="96.52" size="0.508" layer="20" rot="R90">POWER</text>
+<text x="158.75" y="50.8" size="0.508" layer="20" rot="R180">POWER</text>
+<text x="154.94" y="3.81" size="0.508" layer="20" rot="R270">POWER</text>
+<text x="24.13" y="2.54" size="0.508" layer="20" rot="R270">POWER</text>
+<text x="11.43" y="44.45" size="0.508" layer="20">POWER</text>
+<text x="11.43" y="49.53" size="0.508" layer="20">DATA</text>
+<text x="24.13" y="97.79" size="0.508" layer="20" rot="R90">DATA</text>
+<text x="154.94" y="97.79" size="0.508" layer="20" rot="R90">DATA</text>
+<text x="158.75" y="44.45" size="0.508" layer="20" rot="R180">DATA</text>
+<text x="149.86" y="3.81" size="0.508" layer="20" rot="R270">DATA</text>
+<text x="19.05" y="2.54" size="0.508" layer="20" rot="R270">DATA</text>
+<text x="11.43" y="46.99" size="0.508" layer="20">GND</text>
+<text x="21.59" y="97.79" size="0.508" layer="20" rot="R90">GND</text>
+<text x="152.4" y="97.79" size="0.508" layer="20" rot="R90">GND</text>
+<text x="158.75" y="46.99" size="0.508" layer="20" rot="R180">GND</text>
+<text x="152.4" y="3.81" size="0.508" layer="20" rot="R270">GND</text>
+<text x="21.59" y="2.54" size="0.508" layer="20" rot="R270">GND</text>
 </plain>
 <attributes>
@@
 <wire x1="157.14133125" y1="87.7135" x2="157.3965" y2="90.2535" width="0.635" layer="1"/>
 <wire x1="155.55933125" y1="87.4015" x2="157.14133125" y2="87.7135" width="0.635" layer="1"/>
-<wire x1="157.3965" y1="90.2535" x2="157.3965" y2="99.9365" width="0.635" layer="1"/>
-<wire x1="157.3965" y1="99.9365" x2="141.8465" y2="99.9365" width="0.635" layer="1"/>
-<wire x1="141.8465" y1="99.9365" x2="140.97" y2="99.06" width="0.635" layer="1"/>
-<wire x1="140.97" y1="99.06" x2="140.97" y2="81.28" width="0.635" layer="1"/>
+<wire x1="157.3965" y1="98.6665" x2="157.3965" y2="90.2535" width="0.635" layer="1"/>
+<wire x1="140.97" y1="81.28" x2="140.97" y2="97.79" width="0.635" layer="1"/>
 <wire x1="140.97" y1="81.28" x2="129.54" y2="69.85" width="0.635" layer="1"/>
 <wire x1="149.86" y1="92.71" x2="149.86" y2="91.94" width="0.635" layer="1"/>
+<wire x1="140.97" y1="97.79" x2="144.4463125" y2="97.79" width="0.635" layer="1"/>
+<wire x1="144.4463125" y1="97.79" x2="145.8433125" y2="99.187" width="0.635" layer="1"/>
+<wire x1="145.8433125" y1="99.187" x2="151.96530625" y2="99.187" width="0.635" layer="1"/>
+<wire x1="151.96530625" y1="99.187" x2="152.48580625" y2="98.6665" width="0.635" layer="1"/>
+<wire x1="152.48580625" y1="98.6665" x2="157.3965" y2="98.6665" width="0.635" layer="1"/>
 </signal>
 <signal name="D26">
