File: Soccerbot/V3/Nsoccerbots.sch (EAGLE design)
At the start: 65 parts, among them X1 NXT-SOCKET, X2 NXT-SOCKET, X3 NXT-SOCKET, X4 NXT-SOCKET

Commit message: S
S
Parts:
- removed JP1, JP2: (no value), adafruit:PINHD-1X3
- added ISP1: AVRISP-6, adafruit:AVRISP-6
- B1: MPN A000067 -> (none); OC_NEWARK 45W6205 -> unknown
- IR1, IR2, IR3, IR4, IR5, IR6: MF (none) -> VISHAY/TELEFUNKEN; MPN (none) -> TSOP32256; OC_NEWARK unknown -> 09J7370
- LED1, LED2, LED3, LED4, LED5, LED6: MPN (none) -> VLMB1500-GS08; OC_NEWARK (none) -> 12X9113
- R10, R11, R12, R7, R8, R9: MF (none) -> VISHAY/DALE; MPN (none) -> CRCW080510K0FKTA; OC_NEWARK (none) -> 05F1511

Commit message: S
s
Parts:
- removed DIOD1, DIOD2, DIOD3, DIOD4, DIOD5, DIOD6: 1N4004, adafruit:1N4004
- removed LED1, LED3, LED4, LED5, LED6: (no value), adafruit:LED
- removed MOTOR, MOTOR1, MOTOR2, MOTOR3, MOTOR4, MOTOR5: (no value), con-wago-500:W237-102
- removed R10, R11, R12, R7, R8, R9: (no value), adafruit:R-US_M0805
- removed TRANSISTOR1, TRANSISTOR2, TRANSISTOR3, TRANSISTOR4, TRANSISTOR5, TRANSISTOR6: 2N2907, adafruit:2N2907
- added A5, A6, A7, A8, A9: (no value), microbuilder:SOLDERJUMPERREFLOW_NOPASTE
- added C11, C7, C8: 0.1uF, microbuilder:CAP_CERAMIC0805-NOOUTLINE
- added C12: 47uF/16v, microbuilder:CAP_ELECTROLYTICPANASONIC_C
- added C13: 47uF+/16v, microbuilder:CAP_ELECTROLYTICPANASONIC_C
- added C14: 10\0uF 6.3V, adafruit:CPOL-USC
- added C15, C16: 10uF, microbuilder:CAP_CERAMIC0805-NOOUTLINE
- added CN2: 1X4-CLEANBIG, adafruit:1X4-CLEANBIG
- added D0-1, JP6: (no value), adafruit:PINHD-1X8CLEANBIG
- added IC2, IC4: TB6612FNG, adafruit:TB6612FNG
- added J3, J4: 1X5, adafruit:1X5
- added JP5: (no value), microbuilder:HEADER-1X476MIL
- added JP7: (no value), microbuilder:HEADER-1X1070MIL
- added JP8: (no value), microbuilder:HEADER-1X2ROUND
- added MPOWER1, SERPWR1: 1X2-3.5MM, adafruit:1X2-3.5MM
- added PWR1: (no value), jumper:JP1E
- added Q2: AOD417, transistor-power:IRFR5305
- added R15, R16, R17, R19, R20: 10k, microbuilder:RESISTOR0805_NOOUTLINE
- added R18: 1K, microbuilder:RESISTOR0805_NOOUTLINE
- added R21, R22: 10K, microbuilder:RESISTOR0805_NOOUTLINE
- added SERVO3, SERVO4: (no value), adafruit:PINHD-1X3
- added SJ2: (no value), microbuilder:SOLDERJUMPER_2WAY
- added SW2: SPST_TACT-EVQQ2, adafruit:SPST_TACT-EVQQ2
- added TP10, TP6, TP7, TP8, TP9: (no value), microbuilder:TESTPOINTROUND2MM
- added U$12, U$13, U$15: FIDUCIAL, adafruit:FIDUCIAL
- added U1: PCA9685, microbuilder:PCA9685
- IR1, IR2, IR3, IR4, IR5, IR6: device adafruit:PINHD-1X3 -> led:LED5MM; MF VISHAY/TELEFUNKEN -> (none); MPN TSOP32256 -> (none); OC_NEWARK 09J7370 -> (none)
- LED2: value (none) -> Green; device adafruit:LED -> microbuilder:LED0805_NOOUTLINE; MPN VLMB1500-GS08 -> (none); OC_NEWARK 12X9113 -> (none)
- R1, R2, R3, R4, R5, R6: device BaseApp:RESISTOR -> adafruit:R-US_R0603; MF BOURNS, INC. -> (none); MPN CR0603-FX-2700GLF -> (none); OC_NEWARK 32K2331 -> (none)
Connections:
- removed net N$10: DIOD5.A, TRANSISTOR5.C
- removed net N$11: DIOD4.A, TRANSISTOR4.C
- removed net N$12: R2.2, TRANSISTOR6.B
- removed net N$13: DIOD6.A, TRANSISTOR6.C
- removed net N$14: LED1.C, R8.1
- removed net N$15: LED2.C, R7.1
- removed net N$16: LED3.C, R9.1
- removed net N$17: LED4.C, R10.1
- removed net N$18: LED5.C, R11.1
- removed net N$19: LED6.C, R12.1
- removed net N$2: DIOD1.A, TRANSISTOR1.C
- removed net N$5: R5.2, TRANSISTOR2.B
- removed net N$6: DIOD2.A, TRANSISTOR2.C
- removed net N$7: R6.2, TRANSISTOR3.B
- removed net N$8: DIOD3.A, TRANSISTOR3.C
- removed net N$9: R1.2, TRANSISTOR5.B
- new net +12V: C12.+, C13.+, IC2.VM1, IC2.VM2, IC2.VM3, IC4.VM1, IC4.VM2, IC4.VM3, LED2.A, PWR1.1, Q2.S
- new net +5V: C14.+, SERPWR1.1, SERVO3.2, SERVO4.2, SJ2.1
- new net 18: A5.1, A6.1, A7.1, A8.2, A9.2, C11.1, C15.1, C16.1, C7.1, C8.1, IC2.STBY, IC2.VCC, IC4.STBY, IC4.VCC, R21.2, R22.2, SJ2.2, U1.A5, U1.VDD
- new net 19: PWR1.2
- new net A4: A9.1, R20.2, TP6.P$1, U1.A4
- new net GND1: IR5.A
- new net GND2: IR4.A
- new net GND3: IR1.A
- new net GND4: IR2.A
- new net GND5: IR3.A
- new net IOREF1: JP6.7
- new net M1A1: IC2.AO1, IC2.AO1', J3.5
- new net M1B1: IC2.AO2, IC2.AO2', J3.4
- new net M2A1: IC2.BO1, IC2.BO1', J3.1
- new net M2B1: IC2.BO2, IC2.BO2', J3.2
- new net M3A1: IC4.AO1, IC4.AO1', J4.1
- new net M3B1: IC4.AO2, IC4.AO2', J4.2
- new net M4A1: IC4.BO1, IC4.BO1', J4.5
- new net M4B1: IC4.BO2, IC4.BO2', J4.4
- new net PWM0: JP5.1, U1.PWM0
- new net PWM1: JP5.2, U1.PWM1
- new net PWM10: IC2.AIN1, U1.PWM10
- new net PWM11: IC2.BIN1, U1.PWM11
- new net PWM12: IC2.BIN2, U1.PWM12
- new net PWM13: IC2.PWMB, U1.PWM13
- new net PWM14: JP5.3, U1.PWM14
- new net PWM15: JP5.4, U1.PWM15
- new net PWM2: IC4.PWMA, U1.PWM2
- new net PWM3: IC4.AIN2, U1.PWM3
- new net PWM4: IC4.AIN1, U1.PWM4
- new net PWM5: IC4.BIN1, U1.PWM5
- new net PWM6: IC4.BIN2, U1.PWM6
- new net PWM7: IC4.PWMB, U1.PWM7
- new net PWM8: IC2.PWMA, U1.PWM8
- new net PWM9: IC2.AIN2, U1.PWM9
- new net VMOTOR1: MPOWER1.2, Q2.D
- net 3.3V: now also JP6.5, SJ2.3
- net 5.5V: now also JP6.4, R1.1, R2.1, R3.1, R4.1, R5.1, R6.1; no longer DIOD1.C, DIOD2.C, DIOD3.C, DIOD4.C, DIOD5.C, DIOD6.C, MOTOR-1.KL, MOTOR1-1.KL, MOTOR2-1.KL, MOTOR3-1.KL, MOTOR4-1.KL, MOTOR5-1.KL
- net A0: now also A5.2, CN2.4, R15.2, TP10.P$1, U1.A0
- net A1: now also A6.2, CN2.3, R16.2, TP9.P$1, U1.A1
- net A10: now also IR6.C, R1.2
- net A11: now also IR5.C, R2.2
- net A12: now also IR4.C, R3.2
- net A13: now also IR3.C, R6.2
- net A14: now also IR2.C, R5.2
- net A15: now also IR1.C, R4.2
- net A2: now also A7.2, CN2.2, R17.2, TP8.P$1, U1.A2
- net A3: now also A8.1, CN2.1, R19.2, TP7.P$1, U1.A3
- net AREF: now also JP7.3
- net D0: now also D0-1.1
- net D1: now also D0-1.2
- net D10: now also JP7.8, SERVO3.3; no longer IR4.1, R10.2
- net D11: now also JP7.7; no longer IR3.1, R9.2
- net D12: now also JP7.6; no longer IR2.1, R7.2
- net D13: now also JP7.5; no longer IR1.1, R8.2
- net D2: now also D0-1.3; no longer R3.1
- net D22: no longer IR1.3, LED1.A
- net D23: no longer IR2.3, LED2.A
- net D24: no longer IR3.3, LED3.A
- net D25: no longer IR4.3, LED4.A
- net D26: no longer IR5.3, LED5.A
- net D27: no longer IR6.3, LED6.A
- net D3: now also D0-1.4; no longer R4.1
- net D4: now also D0-1.5; no longer R5.1
- net D5: now also D0-1.6; no longer R6.1
- net D6: now also D0-1.7; no longer R1.1
- net D7: now also D0-1.8; no longer R2.1
- net D8: now also JP7.10; no longer IR6.1, R12.2
- net D9: now also JP7.9, SERVO4.3; no longer IR5.1, R11.2
- net GND: now also C11.2, C12.-, C13.-, C14.-, C15.2, C16.2, C7.2, C8.2, IC2.GND, IC2.PGND1, IC2.PGND1', IC2.PGND2, IC2.PGND2', IC4.GND, IC4.PGND1, IC4.PGND1', IC4.PGND2, IC4.PGND2', IR6.A, J3.3, J4.3, JP6.2, JP6.3, JP7.4, MPOWER1.1, Q2.G, R15.1, R16.1, R17.1, R18.1, R19.1, R20.1, SERPWR1.2, SERVO3.1, SERVO4.1, SW2.P, SW2.P1, U1.#OE, U1.EXTCLK, U1.GND; no longer IR1.2, IR2.2, IR3.2, IR4.2, IR5.2, IR6.2, MOTOR-2.KL, MOTOR1-2.KL, MOTOR2-2.KL, MOTOR3-2.KL, MOTOR4-2.KL, MOTOR5-2.KL, TRANSISTOR1.E, TRANSISTOR2.E, TRANSISTOR3.E, TRANSISTOR4.E, TRANSISTOR5.E, TRANSISTOR6.E
- net N$1: now also LED2.C, R18.2; no longer R4.2, TRANSISTOR1.B
- net N$3: now also JP6.8; no longer R3.2, TRANSISTOR4.B
- net RESET: now also JP6.6, SW2.S, SW2.S1
- net SCL: now also JP7.1, JP8.1, R22.1, U1.SCL
- net SDA: now also JP7.2, JP8.2, R21.1, U1.SDA
- net VIN: now also JP6.1
Other:
- note added: "5v"
- note added: "IR1"
- note added: "IR2"
- note added: "IR3"
- note added: "IR4"
- note added: "IR5"
- note added: "IR6"
- note added: "Pins 8-13 are dedicated to IR A15=IR1 A14=IR2 A13=IR3 A12=IR4 A11=IR5 A10=IR6"
- note added: "gnd"
- note removed: "Pins 8-13 are dedicated to IR D13=IR1 D12=IR2 D11=IR3 D10=IR4 D9=IR5 D8=IR6"

Commit message: S
S
Parts:
- added SJ1: (no value), microbuilder:SOLDERJUMPER_CLOSEDPERM
- A5, A6, A7, A8, A9, CN2, D0-1, IC2, IC4, IR1, IR2, IR3, IR4, IR5, IR6, J3, J4, JP5, JP6, JP7, JP8, MPOWER1, PWR1, R1, R15, R16, R17, R19, R2, R20, R21, R22, R3, R4, R5, R6, SERPWR1, SERVO3, SERVO4, SW2, TP10, TP6, TP7, TP8, TP9, U$12, U$13, U$15: OC_NEWARK (none) -> unknown
- C11, C7, C8: MPN (none) -> 0603YC104K4Z2A; OC_NEWARK (none) -> 26M5119
- C12, C13: MPN (none) -> EEEHB1C470P; OC_NEWARK (none) -> 17AC6791
- C14: MPN (none) -> EEFCX0J101R; OC_NEWARK (none) -> 17AC6838
- C15, C16: MPN (none) -> GRM21BC80J106KE19L; OC_NEWARK (none) -> 03AC2709
- LED2: MPN (none) -> MCL-S270GC; OC_NEWARK (none) -> 14N9356
- Q2: MPN (none) -> AUIRFR540ZTRL; OC_NEWARK (none) -> 91Y4154
- R18: MF (none) -> VISHAY/DALE; MPN (none) -> CRCW12061K00FKTA; OC_NEWARK (none) -> 05F1545
- S1: MPN 5636A9 -> (none); OC_NEWARK 13M4539 -> unknown
- SJ2: MPN (none) -> 2211S-02G; OC_NEWARK (none) -> 08N6744
- U1: MPN (none) -> 6EDL04N02PRXUMA1; OC_NEWARK (none) -> 18AC0914
Connections:
- net BAT-: no longer BATERY-2.KL
- net GND: now also BATERY-2.KL, SJ1.1, SJ1.2

Commit message: S
S
Parts:
- IR1, IR2, IR3, IR4, IR5, IR6: MPN (none) -> OP993; OC_NEWARK unknown -> 42AC0040
- R1, R2, R3, R4, R5, R6: MPN (none) -> CR0603-JW-103GLF; OC_NEWARK unknown -> 12AC0507
- R15, R16, R17, R19, R20, R21, R22: MF (none) -> VISHAY/DALE; MPN (none) -> CRCW080510K0FKTA; OC_NEWARK unknown -> 05F1511
- SW2: MPN (none) -> EVQ-Q2P03W; OC_NEWARK unknown -> 01X1669
Changed lines of the file:
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@@
 <part name="IR6" library="led" library_urn="urn:adsk.eagle:library:259" deviceset="LED" device="5MM" package3d_urn="urn:adsk.eagle:package:15799/1">
 <attribute name="MF" value=""/>
-<attribute name="MPN" value=""/>
-<attribute name="OC_NEWARK" value="unknown"/>
+<attribute name="MPN" value="OP993"/>
+<attribute name="OC_NEWARK" value="42AC0040"/>
 </part>
 <part name="R1" library="adafruit" library_urn="urn:adsk.eagle:library:420" deviceset="R-US_" device="R0603">
 <attribute name="MF" value=""/>
-<attribute name="MPN" value=""/>
-<attribute name="OC_NEWARK" value="unknown"/>
+<attribute name="MPN" value="CR0603-JW-103GLF"/>
+<attribute name="OC_NEWARK" value="12AC0507"/>
 </part>
 <part name="IR5" library="led" library_urn="urn:adsk.eagle:library:259" deviceset="LED" device="5MM" package3d_urn="urn:adsk.eagle:package:15799/1">
 <attribute name="MF" value=""/>
-<attribute name="MPN" value=""/>
-<attribute name="OC_NEWARK" value="unknown"/>
+<attribute name="MPN" value="OP993"/>
+<attribute name="OC_NEWARK" value="42AC0040"/>
 </part>
 <part name="R2" library="adafruit" library_urn="urn:adsk.eagle:library:420" deviceset="R-US_" device="R0603">
 <attribute name="MF" value=""/>
-<attribute name="MPN" value=""/>
-<attribute name="OC_NEWARK" value="unknown"/>
+<attribute name="MPN" value="CR0603-JW-103GLF"/>
+<attribute name="OC_NEWARK" value="12AC0507"/>
 </part>
 <part name="IR4" library="led" library_urn="urn:adsk.eagle:library:259" deviceset="LED" device="5MM" package3d_urn="urn:adsk.eagle:package:15799/1">
 <attribute name="MF" value=""/>
-<attribute name="MPN" value=""/>
-<attribute name="OC_NEWARK" value="unknown"/>
+<attribute name="MPN" value="OP993"/>
+<attribute name="OC_NEWARK" value="42AC0040"/>
 </part>
 <part name="R3" library="adafruit" library_urn="urn:adsk.eagle:library:420" deviceset="R-US_" device="R0603">
 <attribute name="MF" value=""/>
-<attribute name="MPN" value=""/>
-<attribute name="OC_NEWARK" value="unknown"/>
+<attribute name="MPN" value="CR0603-JW-103GLF"/>
+<attribute name="OC_NEWARK" value="12AC0507"/>
 </part>
 <part name="IR1" library="led" library_urn="urn:adsk.eagle:library:259" deviceset="LED" device="5MM" package3d_urn="urn:adsk.eagle:package:15799/1">
 <attribute name="MF" value=""/>
-<attribute name="MPN" value=""/>
-<attribute name="OC_NEWARK" value="unknown"/>
+<attribute name="MPN" value="OP993"/>
+<attribute name="OC_NEWARK" value="42AC0040"/>
 </part>
 <part name="R4" library="adafruit" library_urn="urn:adsk.eagle:library:420" deviceset="R-US_" device="R0603">
 <attribute name="MF" value=""/>
-<attribute name="MPN" value=""/>
-<attribute name="OC_NEWARK" value="unknown"/>
+<attribute name="MPN" value="CR0603-JW-103GLF"/>
+<attribute name="OC_NEWARK" value="12AC0507"/>
 </part>
 <part name="IR2" library="led" library_urn="urn:adsk.eagle:library:259" deviceset="LED" device="5MM" package3d_urn="urn:adsk.eagle:package:15799/1">
 <attribute name="MF" value=""/>
-<attribute name="MPN" value=""/>
-<attribute name="OC_NEWARK" value="unknown"/>
+<attribute name="MPN" value="OP993"/>
+<attribute name="OC_NEWARK" value="42AC0040"/>
 </part>
 <part name="R5" library="adafruit" library_urn="urn:adsk.eagle:library:420" deviceset="R-US_" device="R0603">
 <attribute name="MF" value=""/>
-<attribute name="MPN" value=""/>
-<attribute name="OC_NEWARK" value="unknown"/>
+<attribute name="MPN" value="CR0603-JW-103GLF"/>
+<attribute name="OC_NEWARK" value="12AC0507"/>
 </part>
 <part name="IR3" library="led" library_urn="urn:adsk.eagle:library:259" deviceset="LED" device="5MM" package3d_urn="urn:adsk.eagle:package:15799/1">
 <attribute name="MF" value=""/>
-<attribute name="MPN" value=""/>
-<attribute name="OC_NEWARK" value="unknown"/>
+<attribute name="MPN" value="OP993"/>
+<attribute name="OC_NEWARK" value="42AC0040"/>
 </part>
 <part name="R6" library="adafruit" library_urn="urn:adsk.eagle:library:420" deviceset="R-US_" device="R0603">
 <attribute name="MF" value=""/>
-<attribute name="MPN" value=""/>
-<attribute name="OC_NEWARK" value="unknown"/>
+<attribute name="MPN" value="CR0603-JW-103GLF"/>
+<attribute name="OC_NEWARK" value="12AC0507"/>
 </part>
 <part name="IC2" library="adafruit" deviceset="TB6612FNG" device="">
@@
 <part name="GND31" library="supply1" deviceset="GND" device=""/>
 <part name="R15" library="microbuilder" deviceset="RESISTOR" device="0805_NOOUTLINE" value="10k">
-<attribute name="MF" value=""/>
-<attribute name="MPN" value=""/>
-<attribute name="OC_NEWARK" value="unknown"/>
+<attribute name="MF" value="VISHAY/DALE"/>
+<attribute name="MPN" value="CRCW080510K0FKTA"/>
+<attribute name="OC_NEWARK" value="05F1511"/>
 </part>
 <part name="R16" library="microbuilder" deviceset="RESISTOR" device="0805_NOOUTLINE" value="10k">
-<attribute name="MF" value=""/>
-<attribute name="MPN" value=""/>
-<attribute name="OC_NEWARK" value="unknown"/>
+<attribute name="MF" value="VISHAY/DALE"/>
+<attribute name="MPN" value="CRCW080510K0FKTA"/>
+<attribute name="OC_NEWARK" value="05F1511"/>
 </part>
 <part name="R17" library="microbuilder" deviceset="RESISTOR" device="0805_NOOUTLINE" value="10k">
-<attribute name="MF" value=""/>
-<attribute name="MPN" value=""/>
-<attribute name="OC_NEWARK" value="unknown"/>
+<attribute name="MF" value="VISHAY/DALE"/>
+<attribute name="MPN" value="CRCW080510K0FKTA"/>
+<attribute name="OC_NEWARK" value="05F1511"/>
 </part>
 <part name="P+26" library="supply1" deviceset="VCC" device=""/>
@@
 <part name="P+34" library="supply1" deviceset="VCC" device=""/>
 <part name="R19" library="microbuilder" deviceset="RESISTOR" device="0805_NOOUTLINE" value="10k">
-<attribute name="MF" value=""/>
-<attribute name="MPN" value=""/>
-<attribute name="OC_NEWARK" value="unknown"/>
+<attribute name="MF" value="VISHAY/DALE"/>
+<attribute name="MPN" value="CRCW080510K0FKTA"/>
+<attribute name="OC_NEWARK" value="05F1511"/>
 </part>
 <part name="R20" library="microbuilder" deviceset="RESISTOR" device="0805_NOOUTLINE" value="10k">
-<attribute name="MF" value=""/>
-<attribute name="MPN" value=""/>
-<attribute name="OC_NEWARK" value="unknown"/>
+<attribute name="MF" value="VISHAY/DALE"/>
+<attribute name="MPN" value="CRCW080510K0FKTA"/>
+<attribute name="OC_NEWARK" value="05F1511"/>
 </part>
 <part name="TP6" library="microbuilder" deviceset="TESTPOINT" device="ROUND2MM">
@@
 </part>
 <part name="R21" library="microbuilder" deviceset="RESISTOR" device="0805_NOOUTLINE" value="10K">
-<attribute name="MF" value=""/>
-<attribute name="MPN" value=""/>
-<attribute name="OC_NEWARK" value="unknown"/>
+<attribute name="MF" value="VISHAY/DALE"/>
+<attribute name="MPN" value="CRCW080510K0FKTA"/>
+<attribute name="OC_NEWARK" value="05F1511"/>
 </part>
 <part name="R22" library="microbuilder" deviceset="RESISTOR" device="0805_NOOUTLINE" value="10K">
-<attribute name="MF" value=""/>
-<attribute name="MPN" value=""/>
-<attribute name="OC_NEWARK" value="unknown"/>
+<attribute name="MF" value="VISHAY/DALE"/>
+<attribute name="MPN" value="CRCW080510K0FKTA"/>
+<attribute name="OC_NEWARK" value="05F1511"/>
 </part>
 <part name="P+35" library="supply1" deviceset="VCC" device=""/>
@@
 <part name="SW2" library="adafruit" deviceset="SPST_TACT" device="-EVQQ2">
 <attribute name="MF" value=""/>
-<attribute name="MPN" value=""/>
-<attribute name="OC_NEWARK" value="unknown"/>
+<attribute name="MPN" value="EVQ-Q2P03W"/>
+<attribute name="OC_NEWARK" value="01X1669"/>
 </part>
 <part name="GND45" library="supply1" deviceset="GND" device=""/>

Commit message: S
S
Parts:
- removed SJ1: (no value), microbuilder:SOLDERJUMPER_CLOSEDPERM
- added JP1: JUMPER-SMT_2_NC_TRACE_NO-SILK, SparkFun-Jumpers:JUMPER-SMT_2_NC_TRACE_NO-SILK
Connections:
- removed net +3V3: COLORSENSOR2.3, IMU2.8
- removed net +5V: C14.+, SERPWR1.1, SERVO3.2, SERVO4.2, SJ2.1
- removed net BAT-: ESC1P-1.KL, ESC2P-1.KL, ESC3P-1.KL, ESC4P-1.KL, ESC5P-1.KL, ESC6P-1.KL
- removed net DRDY: IMU2.5
- removed net INT: COLORSENSOR2.6
- removed net INT1: IMU2.4
- removed net INT2: IMU2.3
- net 5.5V: now also C14.+, COLORSENSOR2.1, ESC1.2, ESC2.2, ESC3.2, ESC4.2, ESC5.2, ESC6.2, IMU2.7, SERPWR1.1, SERVO3.2, SERVO4.2, SJ2.1
- net BAT+: now also B1.VIN, JP1.1, X1.1, X2.1, X3.1, X4.1
- net GND: now also ESC1P-1.KL, ESC2P-1.KL, ESC3P-1.KL, ESC4P-1.KL, ESC5P-1.KL, ESC6P-1.KL; no longer SJ1.1, SJ1.2
- net VIN: now also JP1.2; no longer B1.VIN, COLORSENSOR2.1, COLORSENSOR2.7, ESC1.2, ESC2.2, ESC3.2, ESC4.2, ESC5.2, ESC6.2, IMU2.7, X1.1, X2.1, X3.1, X4.1

Commit message: Changes detailed in email
Parts:
- removed A5, A6, A7, A8, A9: (no value), microbuilder:SOLDERJUMPERREFLOW_NOPASTE
- removed JP1: JUMPER-SMT_2_NC_TRACE_NO-SILK, SparkFun-Jumpers:JUMPER-SMT_2_NC_TRACE_NO-SILK
- removed MPOWER1, SERPWR1: 1X2-3.5MM, adafruit:1X2-3.5MM
- removed PWR1: (no value), jumper:JP1E
- removed Q2: AOD417, transistor-power:IRFR5305
- removed SJ2: (no value), microbuilder:SOLDERJUMPER_2WAY
- removed TP10, TP6, TP7, TP8, TP9: (no value), microbuilder:TESTPOINTROUND2MM
- removed U$12, U$13, U$15: FIDUCIAL, adafruit:FIDUCIAL
- added IC1: LM340S-05, linear:LM340S-05
- added Q1: AOD417, transistor-power:IRFR5305
Connections:
- removed net +12V: C12.+, C13.+, IC2.VM1, IC2.VM2, IC2.VM3, IC4.VM1, IC4.VM2, IC4.VM3, LED2.A, PWR1.1, Q2.S
- removed net 18: A5.1, A6.1, A7.1, A8.2, A9.2, C11.1, C15.1, C16.1, C7.1, C8.1, IC2.STBY, IC2.VCC, IC4.STBY, IC4.VCC, R21.2, R22.2, SJ2.2, U1.A5, U1.VDD
- removed net 19: PWR1.2
- removed net VIN: JP1.2, JP6.1
- removed net VMOTOR1: MPOWER1.2, Q2.D
- new net N$5: Q1.D, S1.O
- new net SERVO5V: IC1.GND, SERVO3.2, SERVO4.2
- net 3.3V: no longer SJ2.3
- net 5.5V: now also C11.1, C15.1, C16.1, C7.1, C8.1, IC2.STBY, IC2.VCC, IC4.STBY, IC4.VCC, R21.2, R22.2, U1.A5, U1.VDD; no longer SERPWR1.1, SERVO3.2, SERVO4.2, SJ2.1
- net A0: no longer A5.2, TP10.P$1
- net A1: no longer A6.2, TP9.P$1
- net A2: no longer A7.2, TP8.P$1
- net A3: no longer A8.1, TP7.P$1
- net A4: no longer A9.1, TP6.P$1
- net BAT+: now also C12.+, C13.+, IC1.VO, IC2.VM1, IC2.VM2, IC2.VM3, IC4.VM1, IC4.VM2, IC4.VM3, JP6.1, LED2.A, Q1.S; no longer JP1.1, S1.O
- net GND: now also IC1.VI, ISP1.GND, Q1.G; no longer MPOWER1.1, Q2.G, SERPWR1.2
Other:
- note added: "SERVO 5V Regulator"
