File: Soccerbot/V3/Nsoccerbots.sch (EAGLE design)
At the start: 91 parts, among them CN2 1X4-CLEANBIG, IC1 LM340S-05, IC2 TB6612FNG, IC4 TB6612FNG, J3 1X5, J4 1X5, Q1 AOD417, SW2 SPST_TACT-EVQQ2, U1 PCA9685, U2 LM358DT, U3 LM358DT, U4 LM358DT, U5 LM358DT, X1 NXT-SOCKET, X2 NXT-SOCKET, X3 NXT-SOCKET, X4 NXT-SOCKET

Commit message: Misc Changes
Parts:
- removed S1: (no value), switch:320-916
- added U$2: TOGGLESWITCH, toggleswitch:TOGGLESWITCH
- R7: value 300ohm -> 150ohm
Connections:
- net N$4: now also U$2.IN; no longer S1.P
- net N$5: now also U$2.OUT; no longer S1.O
Changed lines of the file:
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@@
 <?xml version="1.0" encoding="utf-8"?>
 <!DOCTYPE eagle SYSTEM "eagle.dtd">
-<eagle version="8.4.1">
+<eagle version="8.4.3">
 <drawing>
 <settings>
@@
 <attribute name="OC_NEWARK" value="unknown"/>
 </part>
-<part name="S1" library="switch" deviceset="320-916" device="">
-<attribute name="MF" value=""/>
-<attribute name="MPN" value=""/>
-<attribute name="OC_NEWARK" value="unknown"/>
-</part>
 <part name="ESC1" library="SparkFun" deviceset="M03" device="LOCK">
 <attribute name="MF" value="MOLEX"/>
@@
 <attribute name="OC_NEWARK" value="01AC5221"/>
 </part>
-<part name="R7" library="rcl" library_urn="urn:adsk.eagle:library:334" deviceset="R-US_" device="R0603" package3d_urn="urn:adsk.eagle:package:23555/2" value="300ohm">
+<part name="R7" library="rcl" library_urn="urn:adsk.eagle:library:334" deviceset="R-US_" device="R0603" package3d_urn="urn:adsk.eagle:package:23555/2" value="150ohm">
 <attribute name="MF" value=""/>
 <attribute name="MPN" value=""/>
@@
 <attribute name="OC_NEWARK" value="68R2991"/>
 </part>
+<part name="U$2" library="toggleswitch" deviceset="TOGGLESWITCH" device=""/>
 </parts>
 <sheets>
@@
 <attribute name="MPN" x="-137.16" y="73.66" size="1.778" layer="96" display="off"/>
 </instance>
-<instance part="S1" gate="1" x="-187.96" y="76.2">
-<attribute name="OC_NEWARK" x="-187.96" y="76.2" size="1.778" layer="96" display="off"/>
-<attribute name="MF" x="-187.96" y="76.2" size="1.778" layer="96" display="off"/>
-<attribute name="MPN" x="-187.96" y="76.2" size="1.778" layer="96" display="off"/>
-</instance>
 <instance part="BATERY" gate="-1" x="-228.6" y="66.04"/>
 <instance part="BATERY" gate="-2" x="-228.6" y="60.96"/>
@@
 <attribute name="MPN" x="-205.74" y="45.72" size="1.778" layer="96" display="off"/>
 </instance>
+<instance part="U$2" gate="G$1" x="-185.42" y="76.2" rot="R90"/>
 </instances>
 <busses>
@@
 <net name="N$4" class="1">
 <segment>
-<pinref part="S1" gate="1" pin="P"/>
 <pinref part="BATERY" gate="-1" pin="KL"/>
-<wire x1="-185.42" y1="71.12" x2="-223.52" y2="71.12" width="0.1524" layer="91"/>
+<wire x1="-195.58" y1="71.12" x2="-223.52" y2="71.12" width="0.1524" layer="91"/>
 <wire x1="-223.52" y1="71.12" x2="-223.52" y2="66.04" width="0.1524" layer="91"/>
-</segment>
-</net>
-<net name="N$5" class="1">
-<segment>
-<pinref part="S1" gate="1" pin="O"/>
-<wire x1="-187.96" y1="81.28" x2="-187.96" y2="93.98" width="0.1524" layer="91"/>
-<wire x1="-187.96" y1="93.98" x2="-200.66" y2="93.98" width="0.1524" layer="91"/>
-<wire x1="-200.66" y1="93.98" x2="-200.66" y2="99.06" width="0.1524" layer="91"/>
-<pinref part="Q1" gate="G$1" pin="D"/>
-<wire x1="-200.66" y1="99.06" x2="-213.36" y2="99.06" width="0.1524" layer="91"/>
-<wire x1="-213.36" y1="99.06" x2="-213.36" y2="96.52" width="0.1524" layer="91"/>
+<wire x1="-195.58" y1="71.12" x2="-195.58" y2="78.74" width="0.1524" layer="91"/>
+<pinref part="U$2" gate="G$1" pin="IN"/>
+<wire x1="-195.58" y1="78.74" x2="-187.96" y2="71.12" width="0.1524" layer="91"/>
 </segment>
 </net>
@@
 </segment>
 </net>
+<net name="N$5" class="1">
+<segment>
+<pinref part="Q1" gate="G$1" pin="D"/>
+<wire x1="-213.36" y1="96.52" x2="-185.42" y2="96.52" width="0.1524" layer="91"/>
+<wire x1="-185.42" y1="96.52" x2="-185.42" y2="83.82" width="0.1524" layer="91"/>
+<wire x1="-185.42" y1="83.82" x2="-180.34" y2="83.82" width="0.1524" layer="91"/>
+<pinref part="U$2" gate="G$1" pin="OUT"/>
+<wire x1="-180.34" y1="83.82" x2="-180.34" y2="71.12" width="0.1524" layer="91"/>
+<wire x1="-180.34" y1="71.12" x2="-182.88" y2="71.12" width="0.1524" layer="91"/>
+</segment>
+</net>
