File: Soccerbot/V3/Nsoccerbots.sch (EAGLE design)
At the start: 91 parts, among them CN2 1X4-CLEANBIG, IC1 LM340S-05, IC2 TB6612FNG, IC4 TB6612FNG, J3 1X5, J4 1X5, Q1 AOD417, SW2 SPST_TACT-EVQQ2, U1 PCA9685, U2 LM358DT, U3 LM358DT, U4 LM358DT, U5 LM358DT, X1 NXT-SOCKET, X2 NXT-SOCKET, X3 NXT-SOCKET, X4 NXT-SOCKET

Commit message: Changes
Parts:
- removed C14: 10\0uF 6.3V, adafruit:CPOL-USC
- removed IRP1, IRP2, IRP3, IRP4, IRP5, IRP6, IRP7, IRP8: TRIMPOT, trimPot:TRIMPOT
- removed R10, R11, R12, R13, R14, R18, R23, R24: 330ohms, resistor:R-US_R0603
- removed U2, U3, U4, U5: LM358DT, LM358DT:LM358DT
- added C1: (no value), rcl:C-USC0805
- R1, R2, R3, R4, R5, R6, R8, R9: value 10k -> 49.9k
Connections:
- removed net IR1O+: IR1.A, R4.1, U5.2IN+
- removed net IR2O+: IR2.A, R5.1, U5.1IN+
- removed net IR3O+: IR3.A, R6.1, U4.2IN+
- removed net IR4O+: IR4.A, R3.1, U4.1IN+
- removed net IR5O+: IR5.A, R2.1, U2.2IN+
- removed net IR6O+: IR6.A, R1.1, U2.1IN+
- removed net IR7O+: IR7.A, R9.1, U3.1IN+
- removed net IR8O+: IR8.A, R8.1, U3.2IN+
- removed net N$10: R14.1, U5.2OUT
- removed net N$11: IRP6.OUT, U2.1IN-
- removed net N$12: R18.2, U5.1OUT
- removed net N$13: R23.2, U3.1OUT
- removed net N$14: IRP5.OUT, U2.2IN-
- removed net N$15: R24.1, U3.2OUT
- removed net N$17: IRP8.OUT, U3.2IN-
- removed net N$18: IRP3.OUT, U4.2IN-
- removed net N$2: R10.1, U2.2OUT
- removed net N$21: IRP4.OUT, U4.1IN-
- removed net N$24: IRP2.OUT, U5.1IN-
- removed net N$27: IRP1.OUT, U5.2IN-
- removed net N$6: IRP7.OUT, U3.1IN-
- removed net N$7: R11.2, U2.1OUT
- removed net N$8: R12.2, U4.1OUT
- removed net N$9: R13.1, U4.2OUT
- net 5.5V: no longer IRP1.VCC, IRP2.VCC, IRP3.VCC, IRP4.VCC, IRP5.VCC, IRP6.VCC, IRP7.VCC, IRP8.VCC, U2.VCC, U3.VCC, U4.VCC, U5.VCC
- net A10: now also IR6.A, R1.1; no longer R11.1
- net A11: now also IR5.A, R2.1; no longer R10.2
- net A12: now also IR4.A, R3.1; no longer R12.1
- net A13: now also IR3.A, R6.1; no longer R13.2
- net A14: now also IR2.A, R5.1; no longer R18.1
- net A15: now also IR1.A, R4.1; no longer R14.2
- net A6: now also IR7.A, R9.1; no longer R23.1
- net A7: now also IR8.A, R8.1; no longer R24.2
- net BAT+: now also Q1.D; no longer Q1.S
- net GND: now also C1.2; no longer C14.-, IRP1.GND, IRP2.GND, IRP3.GND, IRP4.GND, IRP5.GND, IRP6.GND, IRP7.GND, IRP8.GND, U2.GND, U3.GND, U4.GND, U5.GND
- net N$5: now also Q1.S; no longer Q1.D
- net SERVO5V: now also C1.1; no longer C14.+
