File: Soccerbot/V3/NsoccerbotsAuto.sch (EAGLE design)
At the start: 83 parts, among them CN2 1X4-CLEANBIG, IC2 TB6612FNG, IC4 TB6612FNG, J3 1X5, J4 1X5, Q2 AOD417, SW2 SPST_TACT-EVQQ2, U1 PCA9685, X1 NXT-SOCKET, X2 NXT-SOCKET, X3 NXT-SOCKET, X4 NXT-SOCKET

Commit message: S
S
Parts:
- removed A5, A6, A7, A8, A9: (no value), microbuilder:SOLDERJUMPERREFLOW_NOPASTE
- removed MPOWER1, SERPWR1: 1X2-3.5MM, adafruit:1X2-3.5MM
- removed PWR1: (no value), jumper:JP1E
- removed Q2: AOD417, transistor-power:IRFR5305
- removed SJ2: (no value), microbuilder:SOLDERJUMPER_2WAY
- removed TP10, TP6, TP7, TP8, TP9: (no value), microbuilder:TESTPOINTROUND2MM
- removed U$12, U$13, U$15: FIDUCIAL, adafruit:FIDUCIAL
- added IC1: LM340S-05, linear:LM340S-05
- added Q1: AOD417, transistor-power:IRFR5305
Connections:
- removed net +12V: C12.+, C13.+, IC2.VM1, IC2.VM2, IC2.VM3, IC4.VM1, IC4.VM2, IC4.VM3, LED2.A, PWR1.1, Q2.S
- removed net 18: A5.1, A6.1, A7.1, A8.2, A9.2, C11.1, C15.1, C16.1, C7.1, C8.1, IC2.STBY, IC2.VCC, IC4.STBY, IC4.VCC, R21.2, R22.2, SJ2.2, U1.A5, U1.VDD
- removed net 19: PWR1.2
- removed net VIN: JP6.1
- removed net VMOTOR1: MPOWER1.2, Q2.D
- new net A0A: B1.A0(RX0), CN2.4
- new net A1A: B1.A1(TX0), CN2.3
- new net A2A: B1.A2, CN2.2
- new net A3A: B1.A3, CN2.1
- new net N$5: Q1.D, S1.O
- new net SERVO5V: C14.+, IC1.GND, SERVO3.2, SERVO4.2
- net 3.3V: no longer SJ2.3
- net 5.5V: now also C11.1, C15.1, C16.1, C7.1, C8.1, IC2.STBY, IC2.VCC, IC4.STBY, IC4.VCC, R21.2, R22.2, U1.A5, U1.VDD; no longer C14.+, SERPWR1.1, SERVO3.2, SERVO4.2, SJ2.1
- net A0: no longer A5.2, B1.A0(RX0), CN2.4, TP10.P$1
- net A1: no longer A6.2, B1.A1(TX0), CN2.3, TP9.P$1
- net A2: no longer A7.2, B1.A2, CN2.2, TP8.P$1
- net A3: no longer A8.1, B1.A3, CN2.1, TP7.P$1
- net A4: no longer A9.1, TP6.P$1
- net BAT+: now also C12.+, C13.+, IC1.VO, IC2.VM1, IC2.VM2, IC2.VM3, IC4.VM1, IC4.VM2, IC4.VM3, JP6.1, LED2.A, Q1.S; no longer S1.O
- net GND: now also IC1.VI, ISP1.GND, Q1.G; no longer MPOWER1.1, Q2.G, SERPWR1.2
Other:
- note added: "SERVO 5V Regulator"
