File: GYRO/Comp3/COMP3.brd (EAGLE design)
At the start: 16.5 x 42.8 mm, 21 parts, among them U2 LSM9DS1

Commit message: S
S
Connections:
- new net RSTS: JP1.2
Other:
- board text added: "Designed By David Bershadsky"
Changed lines of the file:
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@@
 <dimension x1="0" y1="44.12" x2="0" y2="1.27" x3="-2.54" y3="22.695" textsize="1.778" layer="1"/>
 <dimension x1="0" y1="1.27" x2="16.49" y2="1.27" x3="8.245" y3="-2.54" textsize="1.778" layer="1"/>
+<text x="2.54" y="17.78" size="0.508" layer="25">Designed By
+David Bershadsky</text>
 </plain>
 <attributes>
@@
 <wire x1="8.89" y1="35.56" x2="8.89" y2="35.433" width="0.254" layer="1"/>
 </signal>
+<signal name="RSTS">
+<contactref element="JP1" pad="2"/>
+</signal>
 </signals>
 </board>
 </drawing>
+<compatibility>
+<note version="6.3" minversion="6.2.2" severity="warning">
+Since Version 6.2.2 text objects can contain more than one line,
+which will not be processed correctly with this version.
+</note>
+</compatibility>
 </eagle>
