File: GYRO/Comp3/COMP3.sch (EAGLE design)
At the start: 21 parts, among them U2 LSM9DS1

Commit message: S
S
Connections:
- new net RSTS: JP1.2
Changed lines of the file:
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@@
+</segment>
+</net>
+<net name="RSTS" class="0">
+<segment>
+<pinref part="JP1" gate="G$1" pin="2"/>
+<wire x1="63.5" y1="63.5" x2="66.04" y2="63.5" width="0.1524" layer="91"/>
+<label x="66.04" y="63.5" size="1.778" layer="95"/>
 </segment>
 </net>
