File: Soccerbot/V4/soccerbot.brd (EAGLE design)
At the start: 149.8 x 101.3 mm, 73 parts, among them CN2 1X4-CLEANBIG, IC1 LM340S-05, IC2 TB6612FNG, IC4 TB6612FNG, J3 1X5, J4 1X5, Q1 AOD417, SW2 SPST_TACT-EVQQ2, U1 PCA9685, X1 NXT-SOCKET, X2 NXT-SOCKET, X3 NXT-SOCKET, X4 NXT-SOCKET

Commit message: k
Parts:
- removed JP8: (no value), microbuilder:1X02_ROUND
- removed U$17: (no value), microbuilder:ADAFRUIT_TEXT_30MM
- removed U$18: (no value), microbuilder:ADAFRUIT_3.5MM
- IC2, IC4: value TB6612FNG -> (none)
- R15, R16, R17, R19, R20: value 10k -> (none)
- R4: value 49.9k -> (none)
- moved R4 1.76 mm to (3.49, 41.3)
Connections:
- net SCL: no longer JP8.1
- net SDA: no longer JP8.2
Routing:
- net 5.5V: track 799.0 -> 0.00 mm, vias 4 -> 0
- net BAT+: track 503.2 -> 0.00 mm, vias 13 -> 0
- net SDA: track 359.2 -> 0.00 mm, vias 7 -> 0
- net A6: track 343.2 -> 0.00 mm, vias 4 -> 0
- net SCL: track 338.6 -> 0.00 mm, vias 6 -> 0
- net A15: track 265.6 -> 0.00 mm, vias 1 -> 0
- net 3.3V: track 179.8 -> 0.00 mm, vias 6 -> 0
- net A14: track 162.4 -> 0.00 mm, vias 6 -> 0
- net A10: track 133.0 -> 0.00 mm, vias 2 -> 0
- net A13: track 124.8 -> 0.00 mm, vias 2 -> 0
- net A7: track 114.4 -> 0.00 mm, vias 2 -> 0
- net A12: track 93.1 -> 0.00 mm, vias 2 -> 0
- net D7: track 92.3 -> 0.00 mm, vias 3 -> 0
- net D3: track 86.2 -> 0.00 mm, vias 1 -> 0
- net A11: track 86.1 -> 0.00 mm, vias 3 -> 0
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Other:
- board text removed: "3v"
- board text removed: "4"
- board text removed: "5"
- board text removed: "5v"
- board text removed: "M3"
- board text removed: "M4"
- board text removed: "logic:"
