File: Flash Drive/USBStick.sch (EAGLE design)
At the start: 3 parts, among them X1 USB-A-H

Commit message: S
Parts:
- removed B1: SD_MMC_CARDSD_PCB, SparkFun-Boards:SD_MMC_CARDSD_PCB
- added J1: (no value), Wurth_Elektronik_Electromechanic_Input-Output_Connectors_rev17b:693071010811
- added J2, J3: USB_A_SMT_FEMALE, SparkFun-Connectors:USB_A_SMT_FEMALE
- added J4: SD_CARD_SOCKET, SparkFun-Connectors:SD_CARD_SOCKET
- added U$2: USB-TYPE-C, lio:USB-TYPE-C
Changed lines of the file:
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@@
 <part name="X1" library="SparkFun" deviceset="USB" device="-A-H"/>
 <part name="U$1" library="lio" deviceset="USB-TYPE-C" device=""/>
-<part name="B1" library="SparkFun-Boards" deviceset="SD_MMC_CARD" device="SD_PCB"/>
+<part name="J1" library="Wurth_Elektronik_Electromechanic_Input-Output_Connectors_rev17b" library_urn="urn:adsk.eagle:library:449" deviceset="693071010811" device=""/>
+<part name="J2" library="SparkFun-Connectors" deviceset="USB_A" device="_SMT_FEMALE"/>
+<part name="J3" library="SparkFun-Connectors" deviceset="USB_A" device="_SMT_FEMALE"/>
+<part name="J4" library="SparkFun-Connectors" deviceset="SD_CARD_SOCKET" device=""/>
+<part name="U$2" library="lio" deviceset="USB-TYPE-C" device=""/>
 </parts>
 <sheets>
@@
 <instance part="X1" gate="G$1" x="45.72" y="27.94"/>
 <instance part="U$1" gate="G$1" x="45.72" y="2.54"/>
-<instance part="B1" gate="G$1" x="48.26" y="58.42"/>
+<instance part="J1" gate="G$1" x="48.26" y="93.98"/>
+<instance part="J2" gate="G$1" x="2.54" y="-25.4"/>
+<instance part="J3" gate="G$1" x="2.54" y="-7.62"/>
+<instance part="J4" gate="G$1" x="83.82" y="96.52"/>
+<instance part="U$2" gate="G$1" x="83.82" y="2.54"/>
 </instances>
 <busses>
@@
 </schematic>
 </drawing>
+<compatibility>
+<note version="8.2" severity="warning">
+Since Version 8.2, EAGLE supports online libraries. The ids
+of those online libraries will not be understood (or retained)
+with this version.
+</note>
+</compatibility>
 </eagle>
