File: pchub/pchub.brd (EAGLE design)
At the start: 317.2 x 201.9 mm, 138 parts

Commit message: s
s
Parts:
- removed J3, J4: (no value), Wurth_Elektronik_Electromechanic_Input-Output_Connectors_rev17b:685119134923
- removed S10, S100, S101, S102, S103, S104, S105, S106, S107, S108, S109, S11, S110, S111, S112, S113, S114, S115, S116, S117, S118, S119, S12, S120, S121, S122, S123, S124, S125, S126, S127, S128, S13, S14, S15, S16, S17, S18, S19, S20, S21, S22, S23, S24, S25, S26, S27, S28, S29, S30, S31, S32, S33, S34, S35, S36, S37, S38, S39, S40, S41, S42, S43, S44, S45, S46, S47, S48, S49, S5, S50, S51, S52, S53, S54, S55, S56, S57, S58, S59, S6, S60, S7, S8, S81, S82, S83, S84, S85, S86, S87, S88, S89, S9, S90, S91, S92, S93, S94, S95, S96, S97, S98, S99: (no value), SparkFun-Switches:SWITCH_SP3T_SMD
- added U1, U2, U3, U4: SN74CBT16214DGGR, SN74CBT16214DGGR:SOP50P810X120-56N
- added U5: TMDS361BPAG, TMDS361BPAG:QFP50P1200X1200X120-64N
- moved U$5 311.6 mm to (303.5, -31.8), turned to 90 degrees
- moved J2 310.2 mm to (-2.54, -130.8), turned to 0 degrees
- moved U$2 236.2 mm to (303.5, -82.5), turned to 90 degrees
- moved S1 189.2 mm to (289.6, -118.1), turned to 0 degrees
- moved U$3 179.3 mm to (303.5, -108.0), turned to 90 degrees
- moved S2 152.4 mm to (289.6, -94.0), turned to 0 degrees
- moved U$4 144.9 mm to (303.5, -57.1), turned to 90 degrees
- moved S4 139.9 mm to (289.6, -68.6), turned to 0 degrees
- moved S3 88.9 mm to (289.6, -43.2), turned to 0 degrees
Connections:
- removed net N$121: S93.3, U$2.5
- removed net N$122: S85.3, U$2.3, U$2.B3
- removed net N$123: S84.3, U$2.2, U$2.B2
- removed net N$124: S83.3, U$2.1, U$2.12, U$2.B1, U$2.B12
- removed net N$125: S82.3, U$2.P$1, U$2.P$10, U$2.P$11, U$2.P$12, U$2.P$13, U$2.P$14, U$2.P$15, U$2.P$16, U$2.P$17, U$2.P$18, U$2.P$19, U$2.P$2, U$2.P$20, U$2.P$21, U$2.P$22, U$2.P$23, U$2.P$24, U$2.P$25, U$2.P$26, U$2.P$27, U$2.P$28, U$2.P$3, U$2.P$4, U$2.P$5, U$2.P$6, U$2.P$7, U$2.P$8, U$2.P$9
- removed net N$126: S81.3, U$2.B5
- removed net N$127: S92.3, U$2.6, U$2.B6
- removed net N$128: S91.3, U$2.7, U$2.B7
- removed net N$129: S90.3, U$2.8, U$2.B8
- removed net N$130: S89.3, U$2.10, U$2.B10
- removed net N$131: S88.3, U$2.11, U$2.B11
- removed net N$143: S116.3, U$4.5
- removed net N$144: S109.3, U$4.3, U$4.B3
- removed net N$145: S108.3, U$4.2, U$4.B2
- removed net N$146: S107.3, U$4.1, U$4.12, U$4.B1, U$4.B12
- removed net N$147: S106.3, U$4.P$1, U$4.P$10, U$4.P$11, U$4.P$12, U$4.P$13, U$4.P$14, U$4.P$15, U$4.P$16, U$4.P$17, U$4.P$18, U$4.P$19, U$4.P$2, U$4.P$20, U$4.P$21, U$4.P$22, U$4.P$23, U$4.P$24, U$4.P$25, U$4.P$26, U$4.P$27, U$4.P$28, U$4.P$3, U$4.P$4, U$4.P$5, U$4.P$6, U$4.P$7, U$4.P$8, U$4.P$9
- removed net N$148: S105.3, U$4.B5
- removed net N$149: S115.3, U$4.6, U$4.B6
- removed net N$150: S114.3, U$4.7, U$4.B7
- removed net N$151: S113.3, U$4.8, U$4.B8
- removed net N$152: S112.3, U$4.10, U$4.B10
- removed net N$153: S111.3, U$4.11, U$4.B11
- removed net N$154: S128.3, U$5.5
- removed net N$155: S121.3, U$5.3, U$5.B3
- removed net N$156: S120.3, U$5.2, U$5.B2
- removed net N$157: S119.3, U$5.1, U$5.12, U$5.B1, U$5.B12
- removed net N$158: S118.3, U$5.P$1, U$5.P$10, U$5.P$11, U$5.P$12, U$5.P$13, U$5.P$14, U$5.P$15, U$5.P$16, U$5.P$17, U$5.P$18, U$5.P$19, U$5.P$2, U$5.P$20, U$5.P$21, U$5.P$22, U$5.P$23, U$5.P$24, U$5.P$25, U$5.P$26, U$5.P$27, U$5.P$28, U$5.P$3, U$5.P$4, U$5.P$5, U$5.P$6, U$5.P$7, U$5.P$8, U$5.P$9
- removed net N$159: S117.3, U$5.B5
- removed net N$160: S127.3, U$5.6, U$5.B6
- removed net N$161: S126.3, U$5.7, U$5.B7
- removed net N$162: S125.3, U$5.8, U$5.B8
- removed net N$163: S124.3, U$5.10, U$5.B10
- removed net N$164: S123.3, U$5.11, U$5.B11
- removed net N$61: J4.SHELL, J4.SHELL1, J4.SHELL2, J4.SHELL3, S60.3
- removed net N$62: J4.19, S51.3
- removed net N$63: J4.18, S52.3
- removed net N$64: J4.17, S53.3
- removed net N$65: J4.16, S54.3
- removed net N$66: J4.15, S55.3
- removed net N$67: J4.14, S56.3
- removed net N$68: J4.13, S57.3
- removed net N$69: J4.12, S58.3
- removed net N$70: J4.11, S59.3
- removed net N$71: J4.10, S50.3
- removed net N$72: J4.9, S49.3
- removed net N$73: J4.8, S48.3
- removed net N$74: J4.7, S47.3
- removed net N$75: J4.6, S46.3
- removed net N$76: J4.5, S45.3
- removed net N$77: J4.4, S44.3
- removed net N$80: J4.3, S43.3
- removed net N$81: J4.2, S42.3
- removed net N$82: J4.1, S41.3
- removed net N$94: J3.SHELL, J3.SHELL1, J3.SHELL2, J3.SHELL3, S20.3
- new net 5.5V: S1.3, S2.3, S3.3, S4.3, U1.17, U2.17, U3.17, U4.17
- new net GND: U1.19, U1.38, U1.49, U1.8, U2.19, U2.38, U2.49, U2.8, U3.19, U3.38, U3.49, U3.8, U4.19, U4.38, U4.49, U4.8
- new net N$22: U$4.11, U$4.B11, U3.6
- new net N$23: U$5.5, U4.18
- new net N$24: U$5.3, U$5.B3, U4.23
- new net N$25: U$5.2, U$5.B2, U4.25
- new net N$26: U$5.1, U$5.12, U$5.B1, U$5.B12, U4.27
- new net N$27: U$5.P$1, U$5.P$10, U$5.P$11, U$5.P$12, U$5.P$13, U$5.P$14, U$5.P$15, U$5.P$16, U$5.P$17, U$5.P$18, U$5.P$19, U$5.P$2, U$5.P$20, U$5.P$21, U$5.P$22, U$5.P$23, U$5.P$24, U$5.P$25, U$5.P$26, U$5.P$27, U$5.P$28, U$5.P$3, U$5.P$4, U$5.P$5, U$5.P$6, U$5.P$7, U$5.P$8, U$5.P$9, U4.2
- new net N$28: U$5.B5, U4.4
- new net N$29: U$5.6, U$5.B6, U4.15
- new net N$30: U$5.7, U$5.B7, U4.13
- new net N$52: J2.12, U5.27
- new net N$53: J2.10, U5.26
- new net PC1HDMI-SHEILD: S80.4
- new net VCC: U5.61
- new net VCC_2: U5.6
- new net VCC_3: U5.12
- new net VCC_4: U5.19
- new net VCC_5: U5.25
- new net VCC_6: U5.40
- new net VCC_7: U5.46
- new net VCC_8: U5.55
- net N$1: now also U$2.5, U2.18; no longer J3.19, S11.3
- net N$10: now also U$2.10, U$2.B10, U2.9; no longer J3.11, S15.3
- net N$11: now also U$2.11, U$2.B11, U2.6; no longer J3.10, S10.3
- net N$12: now also U$4.5, U3.18; no longer J3.9, S9.3
- net N$13: now also U$4.3, U$4.B3, U3.23; no longer J3.8, S8.3
- net N$132: now also U1.18; no longer S104.3
- net N$133: now also U1.23; no longer S97.3
- net N$134: now also U1.25; no longer S96.3
- net N$135: now also U1.27; no longer S95.3
- net N$136: now also U1.2; no longer S94.3
- net N$137: now also U1.4; no longer S87.3
- net N$138: now also U1.15; no longer S103.3
- net N$139: now also U1.13; no longer S102.3
- net N$14: now also U$4.2, U$4.B2, U3.25; no longer J3.7, S7.3
- net N$140: now also U1.11; no longer S101.3
- net N$141: now also U1.9; no longer S100.3
- net N$142: now also U1.6; no longer S99.3
- net N$15: now also U$4.1, U$4.12, U$4.B1, U$4.B12, U3.27; no longer J3.6, S6.3
- net N$16: now also U$4.P$1, U$4.P$10, U$4.P$11, U$4.P$12, U$4.P$13, U$4.P$14, U$4.P$15, U$4.P$16, U$4.P$17, U$4.P$18, U$4.P$19, U$4.P$2, U$4.P$20, U$4.P$21, U$4.P$22, U$4.P$23, U$4.P$24, U$4.P$25, U$4.P$26, U$4.P$27, U$4.P$28, U$4.P$3, U$4.P$4, U$4.P$5, U$4.P$6, U$4.P$7, U$4.P$8, U$4.P$9, U3.2; no longer J3.5, S5.3
- net N$17: now also U$4.B5, U3.4; no longer J3.4, S4.3
- net N$18: now also U$4.6, U$4.B6, U3.15; no longer J3.3, S1.3
- net N$19: now also U$4.7, U$4.B7, U3.13; no longer J3.2, S3.3
- net N$2: now also U$2.3, U$2.B3, U2.23; no longer J3.18, S16.3
- net N$20: now also U$4.8, U$4.B8, U3.11; no longer J3.1, S2.3
- net N$21: now also U$4.10, U$4.B10, U3.9; no longer S22.2
- net N$3: now also U$2.2, U$2.B2, U2.25; no longer J3.17, S17.3
- net N$31: now also U$5.8, U$5.B8, U4.11; no longer J2.SHELL, J2.SHELL1, J2.SHELL2, J2.SHELL3, S40.3
- net N$32: now also U$5.10, U$5.B10, U4.9; no longer J2.19, S31.3
- net N$33: now also U$5.11, U$5.B11, U4.6; no longer J2.18, S32.3
- net N$34: now also S2.4, U2.56; no longer J2.17, S33.3
- net N$35: now also S1.4, U1.56; no longer J2.16, S34.3
- net N$36: now also S1.2, U1.55; no longer J2.15, S35.3
- net N$37: now also S1.1, U1.1; no longer J2.14, S36.3
- net N$38: now also S2.2, U2.55; no longer J2.13, S37.3
- net N$39: now also S2.1, U2.1; no longer J2.12, S38.3
- net N$4: now also U$2.1, U$2.12, U$2.B1, U$2.B12, U2.27; no longer S3.2
- net N$40: now also S3.4, U4.56; no longer J2.11, S39.3
- net N$41: now also S3.2, U4.55; no longer J2.10, S30.3
- net N$42: now also S3.1, U4.1; no longer J2.9, S29.3
- net N$43: now also S4.4, U3.56; no longer J2.8, S28.3
- net N$44: now also S4.2, U3.55; no longer J2.7, S27.3
- net N$45: now also S4.1, U3.1; no longer J2.6, S26.3
- net N$46: now also J2.3, U5.18; no longer J2.5, S25.3
- net N$47: now also J2.1, U5.17; no longer J2.4, S24.3
- net N$48: now also J2.6, U5.21; no longer J2.3, S23.3
- net N$49: now also J2.4, U5.20; no longer J2.2, S22.3
- net N$5: now also U$2.P$1, U$2.P$10, U$2.P$11, U$2.P$12, U$2.P$13, U$2.P$14, U$2.P$15, U$2.P$16, U$2.P$17, U$2.P$18, U$2.P$19, U$2.P$2, U$2.P$20, U$2.P$21, U$2.P$22, U$2.P$23, U$2.P$24, U$2.P$25, U$2.P$26, U$2.P$27, U$2.P$28, U$2.P$3, U$2.P$4, U$2.P$5, U$2.P$6, U$2.P$7, U$2.P$8, U$2.P$9, U2.2; no longer J3.16, S18.3
- net N$50: now also J2.9, U5.24; no longer J2.1, S21.3
- net N$51: now also J2.7, U5.23; no longer S42.2
- net N$6: now also U$2.B5, U2.4; no longer J3.15, S19.3
- net N$7: now also U$2.6, U$2.B6, U2.15; no longer J3.14, S12.3
- net N$8: now also U$2.7, U$2.B7, U2.13; no longer J3.13, S13.3
- net N$9: now also U$2.8, U$2.B8, U2.11; no longer J3.12, S14.3
- net PC1HDMI-+5V: no longer S16.4, S32.4, S52.4
- net PC1HDMI-CEC: no longer S13.4, S37.4, S57.4
- net PC1HDMI-DCC: no longer S17.4, S33.4, S53.4
- net PC1HDMI-HOT: no longer S11.4, S31.4, S51.4
- net PC1HDMI-SCL: no longer S19.4, S35.4, S55.4
- net PC1HDMI-SDA: no longer S18.4, S34.4, S54.4
- net PC1HDMI-TMD0S: no longer S28.4, S48.4, S8.4
- net PC1HDMI-TMDS1+: no longer S24.4, S4.4, S44.4
- net PC1HDMI-TMDS1-: no longer S26.4, S46.4, S6.4
- net PC1HDMI-TMDSC+: no longer S10.4, S30.4, S50.4
- net PC1HDMI-TMDSC-: no longer S14.4, S38.4, S58.4
- net PC1HDMI-TMDSCS: no longer S15.4, S39.4, S59.4
- net PC1HDMI-TMDSD0+: no longer S27.4, S47.4, S7.4
- net PC1HDMI-TMDSD0-: no longer S29.4, S49.4, S9.4
- net PC1HDMI-TMDSD1S: no longer S25.4, S45.4, S5.4
- net PC1HDMI-TMDSD2+: no longer S2.4, S21.4, S41.4
- net PC1HDMI-TMDSD2-: no longer S1.4, S23.4, S43.4
- net PC1HDMI-TMDSD2S: no longer S22.4, S3.4, S42.4
- net PC1HDMI-UTL+: no longer S12.4, S36.4, S56.4
- net PC1USBC-CC1: now also U1.39, U2.39, U3.39, U4.39; no longer S104.4, S116.4, S128.4, S93.4
- net PC1USBC-CC2: now also U1.52, U2.52, U3.52, U4.52; no longer S105.4, S117.4, S81.4, S87.4
- net PC1USBC-D+: now also U1.41, U2.41, U3.41, U4.41; no longer S103.4, S115.4, S127.4, S92.4
- net PC1USBC-D-: now also U1.43, U2.43, U3.43, U4.43; no longer S102.4, S114.4, S126.4, S91.4
- net PC1USBC-GND: now also U1.30, U2.30, U3.30, U4.30; no longer S107.4, S119.4, S83.4, S95.4
- net PC1USBC-SBU: now also U1.45, U2.45, U3.45, U4.45; no longer S101.4, S113.4, S125.4, S90.4
- net PC1USBC-SHIELD: now also U1.54, U2.54, U3.54, U4.54; no longer S106.4, S118.4, S82.4, S94.4
- net PC1USBC-SSRX+: now also U1.50, U2.50, U3.50, U4.50; no longer S111.4, S123.4, S88.4, S99.4
- net PC1USBC-SSRX-: now also U1.47, U2.47, U3.47, U4.47; no longer S100.4, S112.4, S124.4, S89.4
- net PC1USBC-SSTX+: now also U1.32, U2.32, U3.32, U4.32; no longer S108.4, S120.4, S84.4, S96.4
- net PC1USBC-SSTX-: now also U1.34, U2.34, U3.34, U4.34; no longer S109.4, S121.4, S85.4, S97.4
- net PC1USBC-VBUS: now also U1.36, U2.36, U3.36, U4.36; no longer S110.4, S122.4, S86.4, S98.4
- net PC2HDMI-+5V: no longer S16.2, S32.2, S52.2
- net PC2HDMI-CEC: no longer S13.2, S37.2, S57.2
- net PC2HDMI-DCC: no longer S17.2, S33.2, S53.2
- net PC2HDMI-HOT: no longer S11.2, S31.2, S51.2
- net PC2HDMI-SCL: no longer S19.2, S35.2, S55.2
- net PC2HDMI-SDA: no longer S18.2, S34.2, S54.2
- net PC2HDMI-SHEILD: no longer S20.2, S40.2, S60.2
- net PC2HDMI-TMD0S: no longer S28.2, S48.2, S8.2
- net PC2HDMI-TMDS1+: no longer S24.2, S4.2, S44.2
- net PC2HDMI-TMDS1-: no longer S26.2, S46.2, S6.2
- net PC2HDMI-TMDSC+: no longer S10.2, S30.2, S50.2
- net PC2HDMI-TMDSC-: no longer S14.2, S38.2, S58.2
- net PC2HDMI-TMDSCS: no longer S15.2, S39.2, S59.2
- net PC2HDMI-TMDSD0+: no longer S27.2, S47.2, S7.2
- net PC2HDMI-TMDSD0-: no longer S29.2, S49.2, S9.2
- net PC2HDMI-TMDSD1S: no longer S25.2, S45.2, S5.2
- net PC2HDMI-TMDSD2+: no longer S2.2, S21.2, S41.2
- net PC2HDMI-TMDSD2-: no longer S1.2, S23.2, S43.2
- net PC2HDMI-UTL+: no longer S12.2, S36.2, S56.2
- net PC2USBC-CC1: now also U1.37, U2.37, U3.37, U4.37; no longer S104.2, S116.2, S128.2, S93.2
- net PC2USBC-CC2: now also U1.51, U2.51, U3.51, U4.51; no longer S105.2, S117.2, S81.2, S87.2
- net PC2USBC-D+: now also U1.40, U2.40, U3.40, U4.40; no longer S103.2, S115.2, S127.2, S92.2
- net PC2USBC-D-: now also U1.42, U2.42, U3.42, U4.42; no longer S102.2, S114.2, S126.2, S91.2
- net PC2USBC-GND: now also U1.29, U2.29, U3.29, U4.29; no longer S107.2, S119.2, S83.2, S95.2
- net PC2USBC-SBU: now also U1.44, U2.44, U3.44, U4.44; no longer S101.2, S113.2, S125.2, S90.2
- net PC2USBC-SHIELD: now also U1.53, U2.53, U3.53, U4.53; no longer S106.2, S118.2, S82.2, S94.2
- net PC2USBC-SSRX+: now also U1.48, U2.48, U3.48, U4.48; no longer S111.2, S123.2, S88.2, S99.2
- net PC2USBC-SSRX-: now also U1.46, U2.46, U3.46, U4.46; no longer S100.2, S112.2, S124.2, S89.2
- net PC2USBC-SSTX+: now also U1.31, U2.31, U3.31, U4.31; no longer S108.2, S120.2, S84.2, S96.2
- net PC2USBC-SSTX-: now also U1.33, U2.33, U3.33, U4.33; no longer S109.2, S121.2, S85.2, S97.2
- net PC2USBC-VBUS: now also U1.35, U2.35, U3.35, U4.35; no longer S110.2, S122.2, S86.2, S98.2
- net PC3HDMI-+5V: no longer S16.1, S32.1, S52.1
- net PC3HDMI-CEC: no longer S13.1, S37.1, S57.1
- net PC3HDMI-DCC: no longer S17.1, S33.1, S53.1
- net PC3HDMI-HOT: no longer S11.1, S31.1, S51.1
- net PC3HDMI-SCL: no longer S19.1, S35.1, S55.1
- net PC3HDMI-SDA: no longer S18.1, S34.1, S54.1
- net PC3HDMI-SHEILD: no longer S20.1, S40.1, S60.1
- net PC3HDMI-TMD0S: no longer S28.1, S48.1, S8.1
- net PC3HDMI-TMDS1+: no longer S24.1, S4.1, S44.1
- net PC3HDMI-TMDS1-: no longer S26.1, S46.1, S6.1
- net PC3HDMI-TMDSC+: no longer S10.1, S30.1, S50.1
- net PC3HDMI-TMDSC-: no longer S14.1, S38.1, S58.1
- net PC3HDMI-TMDSCS: no longer S15.1, S39.1, S59.1
- net PC3HDMI-TMDSD0+: no longer S27.1, S47.1, S7.1
- net PC3HDMI-TMDSD0-: no longer S29.1, S49.1, S9.1
- net PC3HDMI-TMDSD1S: no longer S25.1, S45.1, S5.1
- net PC3HDMI-TMDSD2+: no longer S2.1, S21.1, S41.1
- net PC3HDMI-TMDSD2-: no longer S1.1, S23.1, S43.1
- net PC3HDMI-TMDSD2S: no longer S22.1, S3.1, S42.1
- net PC3HDMI-UTL+: no longer S12.1, S36.1, S56.1
- net PC3USBC-CC1: now also U1.20, U2.20, U3.20, U4.20; no longer S104.1, S116.1, S128.1, S93.1
- net PC3USBC-CC2: now also U1.5, U2.5, U3.5, U4.5; no longer S105.1, S117.1, S81.1, S87.1
- net PC3USBC-D+: now also U1.16, U2.16, U3.16, U4.16; no longer S103.1, S115.1, S127.1, S92.1
- net PC3USBC-D-: now also U1.14, U2.14, U3.14, U4.14; no longer S102.1, S114.1, S126.1, S91.1
- net PC3USBC-GND: now also U1.28, U2.28, U3.28, U4.28; no longer S107.1, S119.1, S83.1, S95.1
- net PC3USBC-SBU: now also U1.12, U2.12, U3.12, U4.12; no longer S101.1, S113.1, S125.1, S90.1
- net PC3USBC-SHIELD: now also U1.3, U2.3, U3.3, U4.3; no longer S106.1, S118.1, S82.1, S94.1
- net PC3USBC-SSRX+: now also U1.7, U2.7, U3.7, U4.7; no longer S111.1, S123.1, S88.1, S99.1
- net PC3USBC-SSRX-: now also U1.10, U2.10, U3.10, U4.10; no longer S100.1, S112.1, S124.1, S89.1
- net PC3USBC-SSTX+: now also U1.26, U2.26, U3.26, U4.26; no longer S108.1, S120.1, S84.1, S96.1
- net PC3USBC-SSTX-: now also U1.24, U2.24, U3.24, U4.24; no longer S109.1, S121.1, S85.1, S97.1
- net PC3USBC-VBUS: now also U1.22, U2.22, U3.22, U4.22; no longer S110.1, S122.1, S86.1, S98.1
- net VBUS: now also U1.21, U2.21, U3.21, U4.21; no longer S110.3, S122.3, S86.3, S98.3

Commit message: s
s
Parts:
- removed S61, S62, S63, S64, S65, S66, S67, S68, S69, S70, S71, S72, S73, S74, S75, S76, S77, S78, S79, S80: (no value), SparkFun-Switches:SWITCH_SP3T_SMD
- added D1, D10, D11, D12, D2, D3, D4, D5, D6, D7, D8, D9: (no value), SparkFun-LED:FKIT-LED-1206
- added J3, J4: (no value), Wurth_Elektronik_Electromechanic_Input-Output_Connectors_rev17b:685119134923
- added J6, J7: 2040210-1, 2040210-1:TE_2040210-1
- added S10, S11, S12, S13, S14, S15, S16, S5, S6, S7, S8, S9: (no value), SparkFun-Switches:SWITCH_SP3T_SMD
- added U10, U11, U12, U13, U14, U15, U16, U17, U18, U19, U20, U9: FSUSB63UMX, FSUSB63UMX:QFN40P180X180X55-12N
- added U6, U7, U8: TMDS361BPAG, TMDS361BPAG:QFP50P1200X1200X120-64N
- added X1, X10, X11, X12, X13, X2, X3, X4, X5, X6, X7, X8, X9: USB, SparkFun:USB-A-S-NOSILK-FEMALE
- moved U5 373.1 mm to (284.5, 69.8), turned to 270 degrees
- moved J2 364.9 mm to (302.3, 69.8), turned to 90 degrees
- moved J5 8.52 mm to (302.3, 5.08), turned to 90 degrees
Connections:
- removed net PC1HDMI-+5V: J1.18, S72.4
- removed net PC1HDMI-CEC: J1.13, S77.4
- removed net PC1HDMI-DCC: J1.17, S73.4
- removed net PC1HDMI-SHEILD: S80.4
- removed net PC1HDMI-TMD0S: J1.8, S68.4
- removed net PC1HDMI-TMDSCS: J1.11, S79.4
- removed net PC1HDMI-TMDSD1S: J1.5, S65.4
- removed net PC1HDMI-TMDSD2S: J1.2, S62.4
- removed net PC1HDMI-UTL+: J1.14, S76.4
- removed net PC2HDMI-+5V: S72.2
- removed net PC2HDMI-CEC: S77.2
- removed net PC2HDMI-DCC: S73.2
- removed net PC2HDMI-SHEILD: S80.2
- removed net PC2HDMI-TMD0S: S68.2
- removed net PC2HDMI-TMDSCS: S79.2
- removed net PC2HDMI-TMDSD1S: S65.2
- removed net PC2HDMI-UTL+: S76.2
- removed net PC3HDMI-+5V: S72.1
- removed net PC3HDMI-CEC: S77.1
- removed net PC3HDMI-DCC: S73.1
- removed net PC3HDMI-SHEILD: S80.1
- removed net PC3HDMI-TMD0S: S68.1
- removed net PC3HDMI-TMDSCS: S79.1
- removed net PC3HDMI-TMDSD1S: S65.1
- removed net PC3HDMI-TMDSD2S: S62.1
- removed net PC3HDMI-UTL+: S76.1
- removed net VCC: U5.61
- removed net VCC_2: U5.6
- removed net VCC_3: U5.12
- removed net VCC_4: U5.19
- removed net VCC_5: U5.25
- removed net VCC_6: U5.40
- removed net VCC_7: U5.46
- removed net VCC_8: U5.55
- new net CEC: J1.13, J2.13, J3.13, J4.13, J5.13
- new net HDMIGND: J1.11, J1.17, J1.2, J1.5, J1.8, J2.11, J2.17, J2.2, J2.5, J2.8, J2.SHELL, J2.SHELL1, J2.SHELL2, J2.SHELL3, J3.11, J3.17, J3.2, J3.5, J3.8, J3.SHELL, J3.SHELL1, J3.SHELL2, J3.SHELL3, J4.11, J4.17, J4.2, J4.5, J4.8, J4.SHELL, J4.SHELL1, J4.SHELL2, J4.SHELL3, J5.11, J5.17, J5.2, J5.5, J5.8, J5.SHELL, J5.SHELL1, J5.SHELL2, J5.SHELL3, U5.15, U5.22, U5.28, U5.3, U5.43, U5.58, U5.9, U6.15, U6.22, U6.28, U6.3, U6.43, U6.58, U6.9, U7.15, U7.22, U7.28, U7.3, U7.43, U7.58, U7.9, U8.15, U8.22, U8.28, U8.3, U8.43, U8.58, U8.9
- new net HDMIVCC: J1.18, J2.18, J3.18, J4.18, J5.18, U5.12, U5.19, U5.25, U5.40, U5.46, U5.55, U5.6, U5.61, U6.12, U6.19, U6.25, U6.40, U6.46, U6.55, U6.6, U6.61, U7.12, U7.19, U7.25, U7.40, U7.46, U7.55, U7.6, U7.61, U8.12, U8.19, U8.25, U8.40, U8.46, U8.55, U8.6, U8.61
- new net HEAC+: J1.14, J2.14, J3.14, J4.14, J5.14
- new net N$100: D5.C, S9.1, U13.4
- new net N$121: D10.A, S14.2, S14.4, U18.11
- new net N$122: U19.2, X12.D-
- new net N$123: U19.1, X12.D+
- new net N$124: D11.C, S15.1, U19.4
- new net N$125: D11.A, S15.2, S15.4, U19.11
- new net N$126: U20.2, X13.D-
- new net N$127: U20.1, X13.D+
- new net N$128: D12.C, S16.1, U20.4
- new net N$129: D12.A, S16.2, S16.4, U20.11
- new net N$54: J2.19, U5.31
- new net N$55: J3.3, U6.18
- new net N$56: J3.1, U6.17
- new net N$57: J3.6, U6.21
- new net N$58: J3.4, U6.20
- new net N$59: J3.9, U6.24
- new net N$60: J3.7, U6.23
- new net N$61: J3.12, U6.27
- new net N$62: J3.10, U6.26
- new net N$63: J3.19, U6.31
- new net N$64: J4.3, U7.18
- new net N$65: J4.1, U7.17
- new net N$66: J4.6, U7.21
- new net N$67: J4.4, U7.20
- new net N$68: J4.9, U7.24
- new net N$69: J4.7, U7.23
- new net N$70: J4.12, U7.27
- new net N$71: J4.10, U7.26
- new net N$72: J4.19, U7.31
- new net N$73: J5.3, U8.18
- new net N$74: J5.1, U8.17
- new net N$75: J5.6, U8.21
- new net N$76: J5.4, U8.20
- new net N$77: J5.9, U8.24
- new net N$78: J5.7, U8.23
- new net N$79: J5.12, U8.27
- new net N$80: J5.10, U8.26
- new net N$81: J5.19, U8.31
- new net N$82: U9.2, X1.D-
- new net N$84: D1.C, S5.1, U9.4
- new net N$85: U10.2, X3.D-
- new net N$86: U10.1, X3.D+
- new net N$87: D1.A, S5.2, S5.4, U9.11
- new net N$88: D2.C, S6.1, U10.4
- new net N$89: D2.A, S6.2, S6.4, U10.11
- new net N$90: U11.2, X4.D-
- new net N$91: U11.1, X4.D+
- new net N$92: D3.C, S7.1, U11.4
- new net N$93: D3.A, S7.2, S7.4, U11.11
- new net N$94: U12.2, X5.D-
- new net N$95: U12.1, X5.D+
- new net N$96: D4.C, S8.1, U12.4
- new net N$97: D4.A, S8.2, S8.4, U12.11
- new net N$98: U13.2, X6.D-
- new net N$99: U13.1, X6.D+
- new net PC1D+: U10.6, U11.6, U12.6, U13.6, U14.6, U15.6, U16.6, U17.6, U18.6, U19.6, U20.6, U9.6, X2.D+
- new net PC1D-: U10.5, U11.5, U12.5, U13.5, U14.5, U15.5, U16.5, U17.5, U18.5, U19.5, U20.5, U9.5, X2.D-
- new net PC2D+: U10.8, U11.8, U12.8, U13.8, U14.8, U15.8, U16.8, U17.8, U18.8, U19.8, U20.8, U9.8
- new net PC2D-: U10.7, U11.7, U12.7, U13.7, U14.7, U15.7, U16.7, U17.7, U18.7, U19.7, U20.7, U9.7
- new net PC3D+: U10.10, U11.10, U12.10, U13.10, U14.10, U15.10, U16.10, U17.10, U18.10, U19.10, U20.10, U9.10
- new net PC3D-: U10.9, U11.9, U12.9, U13.9, U14.9, U15.9, U16.9, U17.9, U18.9, U19.9, U20.9, U9.9
- new net SCL: J2.15, J3.15, J4.15, J5.15, U5.29, U6.29, U7.29, U8.29
- new net SDA: J2.16, J3.16, J4.16, J5.16, U5.30, U6.30, U7.30, U8.30
- new net USBGND: U10.3, U11.3, U12.3, U13.3, U14.3, U15.3, U16.3, U17.3, U18.3, U19.3, U20.3, U9.3, X1.GND, X10.GND, X11.GND, X12.GND, X13.GND, X2.GND, X3.GND, X4.GND, X5.GND, X6.GND, X7.GND, X8.GND, X9.GND
- new net USBVCC: S10.3, S11.3, S12.3, S13.3, S14.3, S15.3, S16.3, S5.3, S6.3, S7.3, S8.3, S9.3, U10.12, U11.12, U12.12, U13.12, U14.12, U15.12, U16.12, U17.12, U18.12, U19.12, U20.12, U9.12, X1.VBUS, X10.VBUS, X11.VBUS, X12.VBUS, X13.VBUS, X2.VBUS, X3.VBUS, X4.VBUS, X5.VBUS, X6.VBUS, X7.VBUS, X8.VBUS, X9.VBUS
- net N$101: now also D5.A, S9.2, S9.4, U13.11; no longer J5.SHELL, J5.SHELL1, J5.SHELL2, J5.SHELL3, S80.3
- net N$102: now also U14.2, X7.D-; no longer J5.19, S71.3
- net N$103: now also U14.1, X7.D+; no longer J5.18, S72.3
- net N$104: now also D6.C, S10.1, U14.4; no longer J5.17, S73.3
- net N$105: now also D6.A, S10.2, S10.4, U14.11; no longer J5.16, S74.3
- net N$106: now also U15.2, X8.D-; no longer J5.15, S75.3
- net N$107: now also U15.1, X8.D+; no longer J5.14, S76.3
- net N$108: now also D7.C, S11.1, U15.4; no longer J5.13, S77.3
- net N$109: now also D7.A, S11.2, S11.4, U15.11; no longer J5.12, S78.3
- net N$110: now also U16.2, X9.D-; no longer J5.11, S79.3
- net N$111: now also U16.1, X9.D+; no longer J5.10, S70.3
- net N$112: now also D8.C, S12.1, U16.4; no longer J5.9, S69.3
- net N$113: now also D8.A, S12.2, S12.4, U16.11; no longer J5.8, S68.3
- net N$114: now also U17.2, X10.D-; no longer J5.7, S67.3
- net N$115: now also U17.1, X10.D+; no longer J5.6, S66.3
- net N$116: now also D9.C, S13.1, U17.4; no longer J5.5, S65.3
- net N$117: now also D9.A, S13.2, S13.4, U17.11; no longer J5.4, S64.3
- net N$118: now also U18.2, X11.D-; no longer J5.3, S63.3
- net N$119: now also U18.1, X11.D+; no longer J5.2, S62.3
- net N$120: now also D10.C, S14.1, U18.4; no longer J5.1, S61.3
- net N$83: now also U9.1, X1.D+; no longer S62.2
- net PC1HDMI-HOT: now also U5.35, U6.35, U7.35, U8.35; no longer S71.4
- net PC1HDMI-SCL: now also U5.37, U6.37, U7.37, U8.37; no longer S75.4
- net PC1HDMI-SDA: now also U5.36, U6.36, U7.36, U8.36; no longer S74.4
- net PC1HDMI-TMDS1+: now also U5.45, U6.45, U7.45, U8.45; no longer S64.4
- net PC1HDMI-TMDS1-: now also U5.44, U6.44, U7.44, U8.44; no longer S66.4
- net PC1HDMI-TMDSC+: now also U5.39, U6.39, U7.39, U8.39; no longer S70.4
- net PC1HDMI-TMDSC-: now also U5.38, U6.38, U7.38, U8.38; no longer S78.4
- net PC1HDMI-TMDSD0+: now also U5.42, U6.42, U7.42, U8.42; no longer S67.4
- net PC1HDMI-TMDSD0-: now also U5.41, U6.41, U7.41, U8.41; no longer S69.4
- net PC1HDMI-TMDSD2+: now also U5.48, U6.48, U7.48, U8.48; no longer S61.4
- net PC1HDMI-TMDSD2-: now also U5.47, U6.47, U7.47, U8.47; no longer S63.4
- net PC2HDMI-HOT: now also U5.50, U6.50, U7.50, U8.50; no longer S71.2
- net PC2HDMI-SCL: now also U5.2, U6.2, U7.2, U8.2; no longer S75.2
- net PC2HDMI-SDA: now also U5.51, U6.51, U7.51, U8.51; no longer S74.2
- net PC2HDMI-TMDS1+: now also U5.60, U6.60, U7.60, U8.60; no longer S64.2
- net PC2HDMI-TMDS1-: now also U5.59, U6.59, U7.59, U8.59; no longer S66.2
- net PC2HDMI-TMDSC+: now also U5.54, U6.54, U7.54, U8.54; no longer S70.2
- net PC2HDMI-TMDSC-: now also U5.53, U6.53, U7.53, U8.53; no longer S78.2
- net PC2HDMI-TMDSD0+: now also U5.57, U6.57, U7.57, U8.57; no longer S67.2
- net PC2HDMI-TMDSD0-: now also U5.56, U6.56, U7.56, U8.56; no longer S69.2
- net PC2HDMI-TMDSD2+: now also U5.63, U6.63, U7.63, U8.63; no longer S61.2
- net PC2HDMI-TMDSD2-: now also U5.62, U6.62, U7.62, U8.62; no longer S63.2
- net PC3HDMI-HOT: now also U5.64, U6.64, U7.64, U8.64; no longer S71.1
- net PC3HDMI-SCL: now also U5.52, U6.52, U7.52, U8.52; no longer S75.1
- net PC3HDMI-SDA: now also U5.1, U6.1, U7.1, U8.1; no longer S74.1
- net PC3HDMI-TMDS1+: now also U5.11, U6.11, U7.11, U8.11; no longer S64.1
- net PC3HDMI-TMDS1-: now also U5.10, U6.10, U7.10, U8.10; no longer S66.1
- net PC3HDMI-TMDSC+: now also U5.5, U6.5, U7.5, U8.5; no longer S70.1
- net PC3HDMI-TMDSC-: now also U5.4, U6.4, U7.4, U8.4; no longer S78.1
- net PC3HDMI-TMDSD0+: now also U5.8, U6.8, U7.8, U8.8; no longer S67.1
- net PC3HDMI-TMDSD0-: now also U5.7, U6.7, U7.7, U8.7; no longer S69.1
- net PC3HDMI-TMDSD2+: now also U5.14, U6.14, U7.14, U8.14; no longer S61.1
- net PC3HDMI-TMDSD2-: now also U5.13, U6.13, U7.13, U8.13; no longer S63.1

Commit message: m
,
Parts:
- added S17: (no value), SparkFun-Switches:SWITCH_SP3T_SMD
- added U$10, U$11, U$12, U$13, U$14, U$15, U$16, U$17, U$18, U$6, U$7, U$8, U$9: RJ45-8PTH, SparkFun:RJ45-8
- added U21, U22: MAX4998ETIT, MAX4998ETIT:21-0184D
- moved J6 667.6 mm to (-109.2, 54.6)
- moved J7 667.6 mm to (-132.1, 54.6)
- moved S13 667.6 mm to (-22.9, 105.4)
- moved X12 667.6 mm to (-81.3, 85.1)
- moved X13 667.6 mm to (-47.0, 85.1)
- moved D10 667.6 mm to (-76.2, 50.8)
- moved D11 667.6 mm to (-71.1, 50.8)
- moved D12 667.6 mm to (-66.0, 50.8)
- moved D9 667.6 mm to (-81.3, 50.8)
- moved S14 667.6 mm to (-90.2, 58.4)
- moved S15 667.6 mm to (-76.2, 58.4)
- moved S16 667.6 mm to (-62.2, 58.4)
- moved U17 667.6 mm to (-53.3, 58.4)
- moved U18 667.6 mm to (-39.4, 58.4)
- moved U19 667.6 mm to (-25.4, 58.4)
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Connections:
- new net ETH1: U$10.1, U$11.1, U$12.1, U$13.1, U$14.1, U$15.1, U$16.1, U$17.1, U$18.1, U$6.1, U$7.1, U$8.1, U$9.1
- new net ETH2: U$10.2, U$11.2, U$12.2, U$13.2, U$14.2, U$15.2, U$16.2, U$17.2, U$18.2, U$6.2, U$7.2, U$8.2, U$9.2
- new net ETH3: U$10.3, U$11.3, U$12.3, U$13.3, U$14.3, U$15.3, U$16.3, U$17.3, U$18.3, U$6.3, U$7.3, U$8.3, U$9.3
- new net ETH4: U$10.4, U$11.4, U$12.4, U$13.4, U$14.4, U$15.4, U$16.4, U$17.4, U$18.4, U$6.4, U$7.4, U$8.4, U$9.4
- new net ETH5: U$10.5, U$11.5, U$12.5, U$13.5, U$14.5, U$15.5, U$16.5, U$17.5, U$18.5, U$6.5, U$7.5, U$8.5, U$9.5
- new net ETH6: U$10.6, U$11.6, U$12.6, U$13.6, U$14.6, U$15.6, U$16.6, U$17.6, U$18.6, U$6.6, U$7.6, U$8.6, U$9.6
- new net ETH7: U$10.7, U$11.7, U$12.7, U$13.7, U$14.7, U$15.7, U$16.7, U$17.7, U$18.7, U$6.7, U$7.7, U$8.7, U$9.7
- new net ETH8: U$10.8, U$11.8, U$12.8, U$13.8, U$14.8, U$15.8, U$16.8, U$17.8, U$18.8, U$6.8, U$7.8, U$8.8, U$9.8
- new net VDD: U21.19, U22.19
- new net VDD_2: U21.7, U22.7
- new net VDD_3: U21.9, U22.9
- new net VDD_4: U21.15, U22.15
- net GND: now also U21.24, U22.24
- net HDMIGND: now also J1.SHELL, J1.SHELL1, J1.SHELL2, J1.SHELL3

Commit message: sd
asdsa
Connections:
- new net N$130: J7.1, U22.1
- new net N$131: J7.3, U22.2
Changed lines of the file:
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@@
 <wire x1="-299.2882" y1="-319.024" x2="-305.6382" y2="-319.024" width="0" layer="19" extent="1-1"/>
+</signal>
+<signal name="N$130">
+<contactref element="U22" pad="1"/>
+<contactref element="J7" pad="1"/>
+<wire x1="-126.58" y1="62.84" x2="-309.0418" y2="-316.484" width="0" layer="19" extent="1-1"/>
+</signal>
+<signal name="N$131">
+<contactref element="J7" pad="3"/>
+<contactref element="U22" pad="2"/>
+<wire x1="-127.58" y1="64.34" x2="-309.0418" y2="-316.992" width="0" layer="19" extent="1-1"/>
 </signal>
 </signals>

Commit message: s
s
Parts:
- removed U$10, U$11, U$12, U$13, U$14, U$15, U$16, U$17, U$18, U$7, U$8, U$9: RJ45-8PTH, SparkFun:RJ45-8
- added J10, J8, J9: 2040210-1, 2040210-1:TE_2040210-1
- added J11, J12: AUDIO_JACK_TRRSSMD_RA, SparkFun-Connectors:AUDIO_JACK_3.5MM_TRRS_SMD_RA
- added S18, S19, S20: (no value), SparkFun-Switches:SWITCH_SP3T_SMD
- added U$19, U$20, U$21, U$22, U$23, U$24, U$25, U$26, U$27, U$28, U$29, U$30: RJ45-8PTH, SparkFun:RJ45-8
- added U23, U24, U25, U26, U27, U28: SN74CBT16214DGGR, SN74CBT16214DGGR:SOP50P810X120-56N
- U21, U22: value MAX4998ETIT -> SN74CBT16214DGGR; device MAX4998ETIT:21-0184D -> SN74CBT16214DGGR:SOP50P810X120-56N
- moved U22 43.3 mm to (-304.8, -361.9)
- moved U21 23.2 mm to (-304.8, -341.6)
Connections:
- removed net VDD: U21.19, U22.19
- removed net VDD_2: U21.7, U22.7
- removed net VDD_3: U21.9, U22.9
- removed net VDD_4: U21.15, U22.15
- new net B$1: U21.23, U23.23, U25.23, U27.23
- new net B$2: U21.25, U23.25, U25.25, U27.25
- new net GND-1: U21.38, U22.38, U23.38, U24.38, U25.38, U26.38, U27.38, U28.38
- new net GND-2: U21.49, U22.49, U23.49, U24.49, U25.49, U26.49, U27.49, U28.49
- new net GND-3: U21.8, U22.8, U23.8, U24.8, U25.8, U26.8, U27.8, U28.8
- new net N$143: J7.3, U21.6
- new net N$144: J7.4, U21.9
- new net N$145: J7.5, U21.11
- new net N$146: J7.6, U21.13
- new net N$147: J7.7, U21.15
- new net N$148: J7.8, U21.18
- new net N$149: J7.9, U21.21
- new net N$150: J7.10
- new net N$151: J7.11
- new net N$152: J7.12, U21.27
- new net N$153: J7.13, U22.2
- new net N$154: J7.14, U22.4
- new net N$155: J7.15, U22.6
- new net N$156: J7.16, U22.9
- new net N$157: J7.17, U22.11
- new net N$158: J7.18, U22.13
- new net N$159: J7.19, U22.15
- new net N$160: J7.SH1, J7.SH2, J7.SH3, J7.SH4, U22.21
- new net N$161: J8.1, U23.2
- new net N$162: J8.2, U23.4
- new net N$163: J7.20, U22.18
- new net N$164: J8.3, U23.6
- new net N$165: J8.4, U23.9
- new net N$166: J8.5, U23.11
- new net N$167: J8.6, U23.13
- new net N$168: J8.7, U23.15
- new net N$169: J8.8, U23.18
- new net N$170: J8.9, U23.21
- new net N$171: J8.10
- new net N$172: J8.11
- new net N$173: J8.12, U23.27
- new net N$174: J8.13, U24.2
- new net N$175: J8.14, U24.4
- new net N$176: J8.15, U24.6
- new net N$177: J8.16, U24.9
- new net N$178: J8.17, U24.11
- new net N$179: J8.18, U24.13
- new net N$180: J8.19, U24.15
- new net N$181: J8.SH1, J8.SH2, J8.SH3, J8.SH4, U24.21
- new net N$182: J8.20, U24.18
- new net N$183: J9.1, U25.2
- new net N$184: J9.2, U25.4
- new net N$185: J9.3, U25.6
- new net N$186: J9.4, U25.9
- new net N$187: J9.5, U25.11
- new net N$188: J9.6, U25.13
- new net N$189: J9.7, U25.15
- new net N$190: J9.8, U25.18
- new net N$191: J9.9, U25.21
- new net N$192: J9.10
- new net N$193: J9.11
- new net N$194: J9.12, U25.27
- new net N$195: J9.13, U26.2
- new net N$196: J9.14, U26.4
- new net N$197: J9.15, U26.6
- new net N$198: J9.16, U26.9
- new net N$199: J9.17, U26.11
- new net N$200: J9.18, U26.13
- new net N$201: J9.19, U26.15
- new net N$202: J9.SH1, J9.SH2, J9.SH3, J9.SH4, U26.21
- new net N$203: J9.20, U26.18
- new net N$204: J10.1, U27.2
- new net N$205: J10.2, U27.4
- new net N$206: J10.3, U27.6
- new net N$207: J10.4, U27.9
- new net N$208: J10.5, U27.11
- new net N$209: J10.6, U27.13
- new net N$210: J10.7, U27.15
- new net N$211: J10.8, U27.18
- new net N$212: J10.9, U27.21
- new net N$213: J10.10
- new net N$214: J10.11
- new net N$215: J10.12, U27.27
- new net N$216: J10.13, U28.2
- new net N$217: J10.14, U28.4
- new net N$218: J10.15, U28.6
- new net N$219: J10.16, U28.9
- new net N$220: J10.17, U28.11
- new net N$221: J10.18, U28.13
- new net N$222: J10.19, U28.15
- new net N$223: J10.SH1, J10.SH2, J10.SH3, J10.SH4, U28.21
- new net N$224: J10.20, U28.18
- new net PC1A1: J11.RING2, J12.RING2
- new net PC1A2: J11.TIP, J12.TIP
- new net PC1A3: J11.RING1, J12.RING1
- new net PC1A4: J11.EARTH, J12.EARTH
- new net PC1DP1: J6.1, U21.54, U23.54, U25.54, U27.54
- new net PC1DP10: J6.10, U21.34, U23.34, U25.34, U27.34
- new net PC1DP11: J6.11, U21.32, U23.32, U25.32, U27.32
- new net PC1DP12: J6.12, U21.30, U23.30, U25.30, U27.30
- new net PC1DP13: J6.13, U22.54, U24.54, U26.54, U28.54
- new net PC1DP14: J6.14, U22.52, U24.52, U26.52, U28.52
- new net PC1DP15: J6.15, U22.50, U24.50, U26.50, U28.50
- new net PC1DP16: J6.16, U22.47, U24.47, U26.47, U28.47
- new net PC1DP17: J6.17, U22.45, U24.45, U26.45, U28.45
- new net PC1DP18: J6.18, U22.43, U24.43, U26.43, U28.43
- new net PC1DP19: J6.19, U22.41, U24.41, U26.41, U28.41
- new net PC1DP2: J6.2, U21.52, U23.52, U25.52, U27.52
- new net PC1DP20: J6.20, U22.39, U24.39, U26.39, U28.39
- new net PC1DP3: J6.3, U21.50, U23.50, U25.50, U27.50
- new net PC1DP4: J6.4, U21.47, U23.47, U25.47, U27.47
- new net PC1DP5: J6.5, U21.45, U23.45, U25.45, U27.45
- new net PC1DP6: J6.6, U21.43, U23.43, U25.43, U27.43
- new net PC1DP7: J6.7, U21.41, U23.41, U25.41, U27.41
- new net PC1DP8: J6.8, U21.39, U23.39, U25.39, U27.39
- new net PC1DP9: J6.9, U21.36, U23.36, U25.36, U27.36
- new net PC1DPS: J6.SH1, J6.SH2, J6.SH3, J6.SH4, U22.36, U24.36, U26.36, U28.36
- new net PC2DP1: U21.53, U23.53, U25.53, U27.53
- new net PC2DP10: U21.33, U23.33, U25.33, U27.33
- new net PC2DP11: U21.31, U23.31, U25.31, U27.31
- new net PC2DP12: U21.29, U23.29, U25.29, U27.29
- new net PC2DP13: U22.53, U24.53, U26.53, U28.53
- new net PC2DP14: U22.51, U24.51, U26.51, U28.51
- new net PC2DP15: U22.48, U24.48, U26.48, U28.48
- new net PC2DP16: U22.46, U24.46, U26.46, U28.46
- new net PC2DP17: U22.44, U24.44, U26.44, U28.44
- new net PC2DP18: U22.42, U24.42, U26.42, U28.42
- new net PC2DP19: U22.40, U24.40, U26.40, U28.40
- new net PC2DP2: U21.51, U23.51, U25.51, U27.51
- new net PC2DP20: U22.37, U24.37, U26.37, U28.37
- new net PC2DP3: U21.48, U23.48, U25.48, U27.48
- new net PC2DP4: U21.46, U23.46, U25.46, U27.46
- new net PC2DP5: U21.44, U23.44, U25.44, U27.44
- new net PC2DP6: U21.42, U23.42, U25.42, U27.42
- new net PC2DP7: U21.40, U23.40, U25.40, U27.40
- new net PC2DP8: U21.37, U23.37, U25.37, U27.37
- new net PC2DP9: U21.35, U23.35, U25.35, U27.35
- new net PC2DPS: U22.35, U24.35, U26.35, U28.35
- new net PC3DP1: U21.3, U23.3, U25.3, U27.3
- new net PC3DP10: U21.24, U23.24, U25.24, U27.24
- new net PC3DP11: U21.26, U23.26, U25.26, U27.26
- new net PC3DP12: U21.28, U23.28, U25.28, U27.28
- new net PC3DP13: U22.3, U24.3, U26.3, U28.3
- new net PC3DP14: U22.5, U24.5, U26.5, U28.5
- new net PC3DP15: U22.7, U24.7, U26.7, U28.7
- new net PC3DP16: U22.10, U24.10, U26.10, U28.10
- new net PC3DP17: U22.12, U24.12, U26.12, U28.12
- new net PC3DP18: U22.14, U24.14, U26.14, U28.14
- new net PC3DP19: U22.16, U24.16, U26.16, U28.16
- new net PC3DP2: U21.5, U23.5, U25.5, U27.5
- new net PC3DP20: U22.20, U24.20, U26.20, U28.20
- new net PC3DP3: U21.7, U23.7, U25.7, U27.7
- new net PC3DP4: U21.10, U23.10, U25.10, U27.10
- new net PC3DP5: U21.12, U23.12, U25.12, U27.12
- new net PC3DP6: U21.14, U23.14, U25.14, U27.14
- new net PC3DP7: U21.16, U23.16, U25.16, U27.16
- new net PC3DP8: U21.20, U23.20, U25.20, U27.20
- new net PC3DP9: U21.22, U23.22, U25.22, U27.22
- new net PC3DPS: U22.22, U24.22, U26.22, U28.22
- new net VCC: U21.17, U22.17, U23.17, U24.17, U25.17, U26.17, U27.17, U28.17
- net ETH1: now also U$19.1, U$20.1, U$21.1, U$22.1, U$23.1, U$24.1, U$25.1, U$26.1, U$27.1, U$28.1, U$29.1, U$30.1; no longer U$10.1, U$11.1, U$12.1, U$13.1, U$14.1, U$15.1, U$16.1, U$17.1, U$18.1, U$7.1, U$8.1, U$9.1
- net ETH2: now also U$19.2, U$20.2, U$21.2, U$22.2, U$23.2, U$24.2, U$25.2, U$26.2, U$27.2, U$28.2, U$29.2, U$30.2; no longer U$10.2, U$11.2, U$12.2, U$13.2, U$14.2, U$15.2, U$16.2, U$17.2, U$18.2, U$7.2, U$8.2, U$9.2
- net ETH3: now also U$19.3, U$20.3, U$21.3, U$22.3, U$23.3, U$24.3, U$25.3, U$26.3, U$27.3, U$28.3, U$29.3, U$30.3; no longer U$10.3, U$11.3, U$12.3, U$13.3, U$14.3, U$15.3, U$16.3, U$17.3, U$18.3, U$7.3, U$8.3, U$9.3
- net ETH4: now also U$19.4, U$20.4, U$21.4, U$22.4, U$23.4, U$24.4, U$25.4, U$26.4, U$27.4, U$28.4, U$29.4, U$30.4; no longer U$10.4, U$11.4, U$12.4, U$13.4, U$14.4, U$15.4, U$16.4, U$17.4, U$18.4, U$7.4, U$8.4, U$9.4
- net ETH5: now also U$19.5, U$20.5, U$21.5, U$22.5, U$23.5, U$24.5, U$25.5, U$26.5, U$27.5, U$28.5, U$29.5, U$30.5; no longer U$10.5, U$11.5, U$12.5, U$13.5, U$14.5, U$15.5, U$16.5, U$17.5, U$18.5, U$7.5, U$8.5, U$9.5
- net ETH6: now also U$19.6, U$20.6, U$21.6, U$22.6, U$23.6, U$24.6, U$25.6, U$26.6, U$27.6, U$28.6, U$29.6, U$30.6; no longer U$10.6, U$11.6, U$12.6, U$13.6, U$14.6, U$15.6, U$16.6, U$17.6, U$18.6, U$7.6, U$8.6, U$9.6
- net ETH7: now also U$19.7, U$20.7, U$21.7, U$22.7, U$23.7, U$24.7, U$25.7, U$26.7, U$27.7, U$28.7, U$29.7, U$30.7; no longer U$10.7, U$11.7, U$12.7, U$13.7, U$14.7, U$15.7, U$16.7, U$17.7, U$18.7, U$7.7, U$8.7, U$9.7
- net ETH8: now also U$19.8, U$20.8, U$21.8, U$22.8, U$23.8, U$24.8, U$25.8, U$26.8, U$27.8, U$28.8, U$29.8, U$30.8; no longer U$10.8, U$11.8, U$12.8, U$13.8, U$14.8, U$15.8, U$16.8, U$17.8, U$18.8, U$7.8, U$8.8, U$9.8
- net GND: now also U21.19, U22.19, U23.19, U24.19, U25.19, U26.19, U27.19, U28.19; no longer U21.24, U22.24
- net N$130: now also U21.2; no longer U22.1
- net N$131: now also J7.2, U21.4; no longer J7.3, U22.2
