File: pchub/pchub.sch (EAGLE design)
At the start: 37 parts

Commit message: s
s
Parts:
- removed J11, J12, J17, J18: (no value), Wurth_Elektronik_Electromechanic_Input-Output_Connectors_rev17b:632723100011
- removed J14, J15, J20, J21: (no value), Wurth_Elektronik_Electromechanic_Input-Output_Connectors_rev17b:685119134923
- removed J4, J5, J6, J8, J9: (no value), Wurth_Elektronik_Electromechanic_Input-Output_Connectors_rev17b:61400416021
- removed SW11, SW12, SW3, SW4, SW5, SW6, SW7, SW8, SW9: (no value), special:SW-C10
- added JP1, JP2, JP3: JUMPER-SMT_2_NC_TRACE_NO-SILK, SparkFun-Jumpers:JUMPER-SMT_2_NC_TRACE_NO-SILK
- added LED5, LED6, LED7, LED8: (no value), adafruit:LEDCHIPLED_0603
- added R1: (no value), BaseApp:RESISTOR
- added S1: (no value), adafruit:EG1218S
- added T1, T10, T11, T12, T13, T14, T15, T16, T17, T18, T19, T2, T20, T21, T22, T23, T24, T25, T26, T27, T28, T29, T3, T30, T31, T32, T33, T34, T35, T36, T37, T38, T39, T4, T40, T41, T42, T43, T44, T45, T46, T47, T48, T49, T5, T50, T51, T52, T53, T54, T55, T56, T57, T58, T59, T6, T60, T61, T62, T63, T64, T65, T66, T67, T68, T69, T7, T70, T71, T72, T73, T74, T75, T76, T77, T78, T79, T8, T80, T9: BCR119F, digital-transistors-2:BCR119F
- J2, J3: device Wurth_Elektronik_Electromechanic_Input-Output_Connectors_rev17b:61400416021 -> Wurth_Elektronik_Electromechanic_Input-Output_Connectors_rev17b:685119134923
- LED1, LED2, LED3, LED4: device adafruit:LEDCHIP-LED0603 -> adafruit:LEDCHIPLED_0603
Connections:
- removed net N$1: J1.VBUS, SW1.C
- removed net N$6: LED4.A
- new net +5V: J13G$1.+5VPOWER, SW1.C, T25.C
- new net +5V1: J2G$1.+5VPOWER, J3G$1.+5VPOWER, T59.C, T79.C
- new net 1HDMI1: J13G$1.TMDSDATA2+, J2G$1.TMDSDATA2+, J3G$1.TMDSDATA2+, T7.C
- new net 1HDMI10: J13G$1.TMDSCLOCK+, J2G$1.TMDSCLOCK+, J3G$1.TMDSCLOCK+, T16.C
- new net 1HDMI11: J13G$1.TMDSCLOCKSHIELD, J2G$1.TMDSCLOCKSHIELD, J3G$1.TMDSCLOCKSHIELD, T18.C, T52.C, T72.C
- new net 1HDMI12: J13G$1.TMDSCLOCK-, J2G$1.TMDSCLOCK-, J3G$1.TMDSCLOCK-, T19.C
- new net 1HDMI13: J13G$1.CEC, J2G$1.CEC, J3G$1.CEC, T20.C, T54.C, T74.C
- new net 1HDMI14: J13G$1.UTILITY/HEAC+, J2G$1.UTILITY/HEAC+, J3G$1.UTILITY/HEAC+, T21.C
- new net 1HDMI15: J13G$1.SCL, J2G$1.SCL, J3G$1.SCL, T22.C, T56.C, T76.C
- new net 1HDMI16: J13G$1.SDA, J2G$1.SDA, J3G$1.SDA, T23.C
- new net 1HDMI17: J13G$1.DDC/CECGROUND, J2G$1.DDC/CECGROUND, J3G$1.DDC/CECGROUND, T24.C, T58.C, T78.C
- new net 1HDMI19: J13G$1.HOTPLUGDETECT/HEAC-, J2G$1.HOTPLUGDETECT/HEAC-, J3G$1.HOTPLUGDETECT/HEAC-, T26.C
- new net 1HDMI2: J13G$1.TMDSDATA2SHIELD, J2G$1.TMDSDATA2SHIELD, J3G$1.TMDSDATA2SHIELD, T42.C, T62.C, T8.C
- new net 1HDMI3: J13G$1.TMDSDATA2-, J2G$1.TMDSDATA2-, J3G$1.TMDSDATA2-, T9.C
- new net 1HDMI4: J13G$1.TMDSDATA1+, J2G$1.TMDSDATA1+, J3G$1.TMDSDATA1+, T10.C, T44.C, T64.C
- new net 1HDMI5: J13G$1.TMDSDATA1SHIELD, J2G$1.TMDSDATA1SHIELD, J3G$1.TMDSDATA1SHIELD, T11.C, T45.C, T65.C
- new net 1HDMI6: J13G$1.TMDSDATA1-, J2G$1.TMDSDATA1-, J3G$1.TMDSDATA1-, T12.C
- new net 1HDMI7: J13G$1.TMDSDATA0+, J2G$1.TMDSDATA0+, J3G$1.TMDSDATA0+, T13.C, T47.C, T67.C
- new net 1HDMI8: J13G$1.TMDSDATA0SHIELD, J2G$1.TMDSDATA0SHIELD, J3G$1.TMDSDATA0SHIELD, T14.C
- new net 1HDMI9: J13G$1.TMDSDATA0-, J2G$1.TMDSDATA0-, J3G$1.TMDSDATA0-, T15.C, T49.C, T69.C
- new net 1PC1: JP3.2, LED1.A, SW2.1
- new net 1PC2: JP2.2, LED2.A, SW2.2
- new net 1PC3: JP1.2, LED3.A, SW2.4
- new net GND: J10G$1.GND, J10G$1.GND2, J7.GND
- new net HDMI1-1: J19G$1.TMDSDATA2+, T7.E
- new net HDMI1-10: J19G$1.TMDSCLOCK+, T16.E, T50.E
- new net HDMI1-11: J19G$1.TMDSCLOCKSHIELD, T18.E
- new net HDMI1-12: J19G$1.TMDSCLOCK-, T19.E, T53.E
- new net HDMI1-13: J19G$1.CEC, T20.E
- new net HDMI1-14: J19G$1.UTILITY/HEAC+, T21.E, T55.E
- new net HDMI1-15: J19G$1.SCL, T22.E
- new net HDMI1-16: J19G$1.SDA, T23.E, T57.E
- new net HDMI1-17: J19G$1.DDC/CECGROUND, T24.E, T58.E
- new net HDMI1-18: J19G$1.+5VPOWER, T25.E
- new net HDMI1-19: J19G$1.HOTPLUGDETECT/HEAC-, T26.E, T60.E
- new net HDMI1-2: J19G$1.TMDSDATA2SHIELD, T42.E, T8.E
- new net HDMI1-20: T80.E
- new net HDMI1-22: T78.E
- new net HDMI1-23: T77.E
- new net HDMI1-24: T75.E
- new net HDMI1-26: T73.E
- new net HDMI1-28: T70.E
- new net HDMI1-3: J19G$1.TMDSDATA2-, T9.E
- new net HDMI1-30: T68.E
- new net HDMI1-31: T66.E
- new net HDMI1-33: T64.E
- new net HDMI1-35: T62.E
- new net HDMI1-4: J19G$1.TMDSDATA1+, T10.E, T44.E
- new net HDMI1-5: J19G$1.TMDSDATA1SHIELD, T11.E
- new net HDMI1-6: J19G$1.TMDSDATA1-, T12.E, T46.E
- new net HDMI1-7: J19G$1.TMDSDATA0+, T13.E
- new net HDMI1-8: J19G$1.TMDSDATA0SHIELD, T14.E, T48.E
- new net HDMI1-9: J19G$1.TMDSDATA0-, T15.E
- new net HDMI1OFF: LED8.C
- new net HDMI1PC1: LED5.C, T10.B, T11.B, T12.B, T13.B, T14.B, T15.B, T16.B, T18.B, T19.B, T20.B, T21.B, T22.B, T23.B, T24.B, T25.B, T26.B, T7.B, T8.B, T9.B
- new net HDMI1PC2: LED6.C, T41.B, T42.B, T43.B, T44.B, T45.B, T46.B, T47.B, T48.B, T49.B, T50.B, T52.B, T53.B, T54.B, T55.B, T56.B, T57.B, T58.B, T59.B, T60.B
- new net HDMI1PC3: LED7.C, T61.B, T62.B, T63.B, T64.B, T65.B, T66.B, T67.B, T68.B, T69.B, T70.B, T72.B, T73.B, T74.B, T75.B, T76.B, T77.B, T78.B, T79.B, T80.B
- new net N$10: J10G$1.CC1, T38.E
- new net N$11: J10G$1.SSTXN1, T39.E
- new net N$12: J10G$1.SSTXP1, T40.E
- new net N$13: J10G$1.SSTXP2, T27.E
- new net N$130: LED5.A, SW1.1
- new net N$131: LED6.A, SW1.2
- new net N$132: LED7.A, SW1.4
- new net N$133: LED8.A, SW1.8
- new net N$14: J10G$1.SSTXN2, T28.E
- new net N$15: J10G$1.CC2, T29.E
- new net N$16: J10G$1.DP2, T30.E
- new net N$17: J10G$1.DN2, T31.E
- new net N$19: J10G$1.SBU2, T32.E
- new net N$39: J10G$1.SSRXP1, T34.E
- new net N$40: J10G$1.SSRXN1, T33.E
- new net OFF: LED4.C
- new net PC1: LED1.C, S1.P, T27.B, T28.B, T29.B, T30.B, T31.B, T32.B, T33.B, T34.B, T35.B, T36.B, T37.B, T38.B, T39.B, T40.B
- new net PC1A: S1.S, T1.B, T2.B
- new net PC1AD+: J7.D+, T1.C
- new net PC1AD-: J7.D-, T2.E
- new net PC1C: S1.O, T3.B, T4.B
- new net PC1CD+: J10G$1.DP1, T3.C
- new net PC1CD-: J10G$1.DN1, T4.C, T4.E
- new net PC1D+: T1.E, T3.E, T5.C
- new net PC1D-: T2.C, T6.E
- new net PC2: LED2.C
- new net PC3: LED3.C
- new net USB1D+: J1.D+, T5.E
- new net USB1D-: J1.D-, T6.C
- new net USB1ON: JP1.1, JP3.1, T5.B, T6.B
- new net VBUS: J10G$1.VBUS, J10G$1.VBUS2, J7.VBUS, R1.1
- net N$2: now also J10G$1.GND1, J10G$1.GND3; no longer LED4.C, SW1.8
- net N$3: now also J10G$1.VBUS1, J10G$1.VBUS3; no longer LED3.C, SW1.4
- net N$4: now also J10G$1.SSRXP2, T35.E; no longer LED2.C, SW1.2
- net N$5: now also R1.2, SW2.C; no longer LED1.C, SW1.1
- net N$7: now also J10G$1.SSRXN2, T36.E; no longer LED3.A
- net N$8: now also J10G$1.SBU1, T37.E; no longer LED2.A
- net N$9: now also LED4.A, SW2.8; no longer LED1.A
Other:
- moved on the sheet: J10SHIELD, J13G$1, J13SHIELD, J19G$1, J19SHIELD, LED1, LED2, LED3, LED4, SW1, SW2

Commit message: ,
,
Parts:
- removed J10, J16: (no value), Wurth_Elektronik_Electromechanic_Input-Output_Connectors_rev17b:632723100011
- removed J13, J19: (no value), Wurth_Elektronik_Electromechanic_Input-Output_Connectors_rev17b:685119134923
- removed J7: (no value), Wurth_Elektronik_Electromechanic_Input-Output_Connectors_rev17b:61400416021
- removed JP1, JP2, JP3: JUMPER-SMT_2_NC_TRACE_NO-SILK, SparkFun-Jumpers:JUMPER-SMT_2_NC_TRACE_NO-SILK
- removed LED1, LED2, LED3, LED4, LED5, LED6, LED7, LED8: (no value), adafruit:LEDCHIPLED_0603
- removed R1: (no value), BaseApp:RESISTOR
- removed SW1, SW10, SW2: (no value), special:SW-C10
- removed T1, T10, T11, T12, T13, T14, T15, T16, T17, T18, T19, T2, T20, T21, T22, T23, T24, T25, T26, T27, T28, T29, T3, T30, T31, T32, T33, T34, T35, T36, T37, T38, T39, T4, T40, T41, T42, T43, T44, T45, T46, T47, T48, T49, T5, T50, T51, T52, T53, T54, T55, T56, T57, T58, T59, T6, T60, T61, T62, T63, T64, T65, T66, T67, T68, T69, T7, T70, T71, T72, T73, T74, T75, T76, T77, T78, T79, T8, T80, T9: BCR119F, digital-transistors-2:BCR119F
- added J4, J5: (no value), Wurth_Elektronik_Electromechanic_Input-Output_Connectors_rev17b:685119134923
- added S10, S100, S101, S102, S103, S104, S105, S106, S107, S108, S109, S11, S110, S111, S112, S113, S114, S115, S116, S117, S118, S119, S12, S120, S121, S122, S123, S124, S125, S126, S127, S128, S13, S14, S15, S16, S17, S18, S19, S2, S20, S21, S22, S23, S24, S25, S26, S27, S28, S29, S3, S30, S31, S32, S33, S34, S35, S36, S37, S38, S39, S4, S40, S41, S42, S43, S44, S45, S46, S47, S48, S49, S5, S50, S51, S52, S53, S54, S55, S56, S57, S58, S59, S6, S60, S61, S62, S63, S64, S65, S66, S67, S68, S69, S7, S70, S71, S72, S73, S74, S75, S76, S77, S78, S79, S8, S80, S81, S82, S83, S84, S85, S86, S87, S88, S89, S9, S90, S91, S92, S93, S94, S95, S96, S97, S98, S99: (no value), SparkFun-Switches:SWITCH-SP3T-SMD
- added U$1, U$2, U$3, U$4, U$5: USB-TYPE-C, lio:USB-TYPE-C
- J1: device Wurth_Elektronik_Electromechanic_Input-Output_Connectors_rev17b:61400416021 -> Wurth_Elektronik_Electromechanic_Input-Output_Connectors_rev17b:685119134923
- S1: device adafruit:EG1218S -> SparkFun-Switches:SWITCH-SP3T-SMD
Connections:
- removed net +5V: J13G$1.+5VPOWER, SW1.C, T25.C
- removed net +5V1: J2G$1.+5VPOWER, J3G$1.+5VPOWER, T59.C, T79.C
- removed net 1HDMI1: J13G$1.TMDSDATA2+, J2G$1.TMDSDATA2+, J3G$1.TMDSDATA2+, T7.C
- removed net 1HDMI10: J13G$1.TMDSCLOCK+, J2G$1.TMDSCLOCK+, J3G$1.TMDSCLOCK+, T16.C
- removed net 1HDMI11: J13G$1.TMDSCLOCKSHIELD, J2G$1.TMDSCLOCKSHIELD, J3G$1.TMDSCLOCKSHIELD, T18.C, T52.C, T72.C
- removed net 1HDMI12: J13G$1.TMDSCLOCK-, J2G$1.TMDSCLOCK-, J3G$1.TMDSCLOCK-, T19.C
- removed net 1HDMI13: J13G$1.CEC, J2G$1.CEC, J3G$1.CEC, T20.C, T54.C, T74.C
- removed net 1HDMI14: J13G$1.UTILITY/HEAC+, J2G$1.UTILITY/HEAC+, J3G$1.UTILITY/HEAC+, T21.C
- removed net 1HDMI15: J13G$1.SCL, J2G$1.SCL, J3G$1.SCL, T22.C, T56.C, T76.C
- removed net 1HDMI16: J13G$1.SDA, J2G$1.SDA, J3G$1.SDA, T23.C
- removed net 1HDMI17: J13G$1.DDC/CECGROUND, J2G$1.DDC/CECGROUND, J3G$1.DDC/CECGROUND, T24.C, T58.C, T78.C
- removed net 1HDMI19: J13G$1.HOTPLUGDETECT/HEAC-, J2G$1.HOTPLUGDETECT/HEAC-, J3G$1.HOTPLUGDETECT/HEAC-, T26.C
- removed net 1HDMI2: J13G$1.TMDSDATA2SHIELD, J2G$1.TMDSDATA2SHIELD, J3G$1.TMDSDATA2SHIELD, T42.C, T62.C, T8.C
- removed net 1HDMI3: J13G$1.TMDSDATA2-, J2G$1.TMDSDATA2-, J3G$1.TMDSDATA2-, T9.C
- removed net 1HDMI4: J13G$1.TMDSDATA1+, J2G$1.TMDSDATA1+, J3G$1.TMDSDATA1+, T10.C, T44.C, T64.C
- removed net 1HDMI5: J13G$1.TMDSDATA1SHIELD, J2G$1.TMDSDATA1SHIELD, J3G$1.TMDSDATA1SHIELD, T11.C, T45.C, T65.C
- removed net 1HDMI6: J13G$1.TMDSDATA1-, J2G$1.TMDSDATA1-, J3G$1.TMDSDATA1-, T12.C
- removed net 1HDMI7: J13G$1.TMDSDATA0+, J2G$1.TMDSDATA0+, J3G$1.TMDSDATA0+, T13.C, T47.C, T67.C
- removed net 1HDMI8: J13G$1.TMDSDATA0SHIELD, J2G$1.TMDSDATA0SHIELD, J3G$1.TMDSDATA0SHIELD, T14.C
- removed net 1HDMI9: J13G$1.TMDSDATA0-, J2G$1.TMDSDATA0-, J3G$1.TMDSDATA0-, T15.C, T49.C, T69.C
- removed net 1PC1: JP3.2, LED1.A, SW2.1
- removed net 1PC2: JP2.2, LED2.A, SW2.2
- removed net 1PC3: JP1.2, LED3.A, SW2.4
- removed net GND: J10G$1.GND, J10G$1.GND2, J7.GND
- removed net HDMI1-1: J19G$1.TMDSDATA2+, T7.E
- removed net HDMI1-10: J19G$1.TMDSCLOCK+, T16.E, T50.E
- removed net HDMI1-11: J19G$1.TMDSCLOCKSHIELD, T18.E
- removed net HDMI1-12: J19G$1.TMDSCLOCK-, T19.E, T53.E
- removed net HDMI1-13: J19G$1.CEC, T20.E
- removed net HDMI1-14: J19G$1.UTILITY/HEAC+, T21.E, T55.E
- removed net HDMI1-15: J19G$1.SCL, T22.E
- removed net HDMI1-16: J19G$1.SDA, T23.E, T57.E
- removed net HDMI1-17: J19G$1.DDC/CECGROUND, T24.E, T58.E
- removed net HDMI1-18: J19G$1.+5VPOWER, T25.E
- removed net HDMI1-19: J19G$1.HOTPLUGDETECT/HEAC-, T26.E, T60.E
- removed net HDMI1-2: J19G$1.TMDSDATA2SHIELD, T42.E, T8.E
- removed net HDMI1-20: T80.E
- removed net HDMI1-22: T78.E
- removed net HDMI1-23: T77.E
- removed net HDMI1-24: T75.E
- removed net HDMI1-26: T73.E
- removed net HDMI1-28: T70.E
- removed net HDMI1-3: J19G$1.TMDSDATA2-, T9.E
- removed net HDMI1-30: T68.E
- removed net HDMI1-31: T66.E
- removed net HDMI1-33: T64.E
- removed net HDMI1-35: T62.E
- removed net HDMI1-4: J19G$1.TMDSDATA1+, T10.E, T44.E
- removed net HDMI1-5: J19G$1.TMDSDATA1SHIELD, T11.E
- removed net HDMI1-6: J19G$1.TMDSDATA1-, T12.E, T46.E
- removed net HDMI1-7: J19G$1.TMDSDATA0+, T13.E
- removed net HDMI1-8: J19G$1.TMDSDATA0SHIELD, T14.E, T48.E
- removed net HDMI1-9: J19G$1.TMDSDATA0-, T15.E
- removed net HDMI1OFF: LED8.C
- removed net HDMI1PC1: LED5.C, T10.B, T11.B, T12.B, T13.B, T14.B, T15.B, T16.B, T18.B, T19.B, T20.B, T21.B, T22.B, T23.B, T24.B, T25.B, T26.B, T7.B, T8.B, T9.B
- removed net HDMI1PC2: LED6.C, T41.B, T42.B, T43.B, T44.B, T45.B, T46.B, T47.B, T48.B, T49.B, T50.B, T52.B, T53.B, T54.B, T55.B, T56.B, T57.B, T58.B, T59.B, T60.B
- removed net HDMI1PC3: LED7.C, T61.B, T62.B, T63.B, T64.B, T65.B, T66.B, T67.B, T68.B, T69.B, T70.B, T72.B, T73.B, T74.B, T75.B, T76.B, T77.B, T78.B, T79.B, T80.B
- removed net OFF: LED4.C
- removed net PC1: LED1.C, S1.P, T27.B, T28.B, T29.B, T30.B, T31.B, T32.B, T33.B, T34.B, T35.B, T36.B, T37.B, T38.B, T39.B, T40.B
- removed net PC1A: S1.S, T1.B, T2.B
- removed net PC1AD+: J7.D+, T1.C
- removed net PC1AD-: J7.D-, T2.E
- removed net PC1C: S1.O, T3.B, T4.B
- removed net PC1CD+: J10G$1.DP1, T3.C
- removed net PC1CD-: J10G$1.DN1, T4.C, T4.E
- removed net PC1D+: T1.E, T3.E, T5.C
- removed net PC1D-: T2.C, T6.E
- removed net PC2: LED2.C
- removed net PC3: LED3.C
- removed net USB1D+: J1.D+, T5.E
- removed net USB1D-: J1.D-, T6.C
- removed net USB1ON: JP1.1, JP3.1, T5.B, T6.B
- new net N$1: J3G$1.HOTPLUGDETECT/HEAC-, S11.3
- new net N$101: J5SHIELD.SHIELD, S80.3
- new net N$102: J5G$1.HOTPLUGDETECT/HEAC-, S71.3
- new net N$103: J5G$1.+5VPOWER, S72.3
- new net N$104: J5G$1.DDC/CECGROUND, S73.3
- new net N$105: J5G$1.SDA, S74.3
- new net N$106: J5G$1.SCL, S75.3
- new net N$107: J5G$1.UTILITY/HEAC+, S76.3
- new net N$108: J5G$1.CEC, S77.3
- new net N$109: J5G$1.TMDSCLOCK-, S78.3
- new net N$110: J5G$1.TMDSCLOCKSHIELD, S79.3
- new net N$111: J5G$1.TMDSCLOCK+, S70.3
- new net N$112: J5G$1.TMDSDATA0-, S69.3
- new net N$113: J5G$1.TMDSDATA0SHIELD, S68.3
- new net N$114: J5G$1.TMDSDATA0+, S67.3
- new net N$115: J5G$1.TMDSDATA1-, S66.3
- new net N$116: J5G$1.TMDSDATA1SHIELD, S65.3
- new net N$117: J5G$1.TMDSDATA1+, S64.3
- new net N$118: J5G$1.TMDSDATA2-, S63.3
- new net N$119: J5G$1.TMDSDATA2SHIELD, S62.3
- new net N$120: J5G$1.TMDSDATA2+, S61.3
- new net N$121: S93.3, U$2.CC1/VCONN
- new net N$122: S85.3, U$2.SSTX-
- new net N$123: S84.3, U$2.SSTX+
- new net N$124: S83.3, U$2.GND
- new net N$125: S82.3, U$2.SHIELD
- new net N$126: S81.3, U$2.CC2/VCONN
- new net N$127: S92.3, U$2.D+
- new net N$128: S91.3, U$2.D-
- new net N$129: S90.3, U$2.SBU
- new net N$134: S96.3, U$3.SSTX+
- new net N$135: S95.3, U$3.GND
- new net N$136: S94.3, U$3.SHIELD
- new net N$137: S87.3, U$3.CC2/VCONN
- new net N$138: S103.3, U$3.D+
- new net N$139: S102.3, U$3.D-
- new net N$140: S101.3, U$3.SBU
- new net N$141: S100.3, U$3.SSRX-
- new net N$142: S99.3, U$3.SSRX+
- new net N$143: S116.3, U$4.CC1/VCONN
- new net N$144: S109.3, U$4.SSTX-
- new net N$145: S108.3, U$4.SSTX+
- new net N$146: S107.3, U$4.GND
- new net N$147: S106.3, U$4.SHIELD
- new net N$148: S105.3, U$4.CC2/VCONN
- new net N$149: S115.3, U$4.D+
- new net N$150: S114.3, U$4.D-
- new net N$151: S113.3, U$4.SBU
- new net N$152: S112.3, U$4.SSRX-
- new net N$153: S111.3, U$4.SSRX+
- new net N$154: S128.3, U$5.CC1/VCONN
- new net N$155: S121.3, U$5.SSTX-
- new net N$156: S120.3, U$5.SSTX+
- new net N$157: S119.3, U$5.GND
- new net N$158: S118.3, U$5.SHIELD
- new net N$159: S117.3, U$5.CC2/VCONN
- new net N$160: S127.3, U$5.D+
- new net N$161: S126.3, U$5.D-
- new net N$162: S125.3, U$5.SBU
- new net N$163: S124.3, U$5.SSRX-
- new net N$164: S123.3, U$5.SSRX+
- new net N$18: J3G$1.TMDSDATA2-, S1.3
- new net N$20: J3G$1.TMDSDATA2+, S2.3
- new net N$21: S22.2
- new net N$31: J2SHIELD.SHIELD, S40.3
- new net N$32: J2G$1.HOTPLUGDETECT/HEAC-, S31.3
- new net N$33: J2G$1.+5VPOWER, S32.3
- new net N$34: J2G$1.DDC/CECGROUND, S33.3
- new net N$35: J2G$1.SDA, S34.3
- new net N$36: J2G$1.SCL, S35.3
- new net N$37: J2G$1.UTILITY/HEAC+, S36.3
- new net N$38: J2G$1.CEC, S37.3
- new net N$41: J2G$1.TMDSCLOCK+, S30.3
- new net N$42: J2G$1.TMDSDATA0-, S29.3
- new net N$43: J2G$1.TMDSDATA0SHIELD, S28.3
- new net N$44: J2G$1.TMDSDATA0+, S27.3
- new net N$45: J2G$1.TMDSDATA1-, S26.3
- new net N$46: J2G$1.TMDSDATA1SHIELD, S25.3
- new net N$47: J2G$1.TMDSDATA1+, S24.3
- new net N$48: J2G$1.TMDSDATA2-, S23.3
- new net N$49: J2G$1.TMDSDATA2SHIELD, S22.3
- new net N$50: J2G$1.TMDSDATA2+, S21.3
- new net N$51: S42.2
- new net N$6: J3G$1.SCL, S19.3
- new net N$61: J4SHIELD.SHIELD, S60.3
- new net N$62: J4G$1.HOTPLUGDETECT/HEAC-, S51.3
- new net N$63: J4G$1.+5VPOWER, S52.3
- new net N$64: J4G$1.DDC/CECGROUND, S53.3
- new net N$65: J4G$1.SDA, S54.3
- new net N$66: J4G$1.SCL, S55.3
- new net N$67: J4G$1.UTILITY/HEAC+, S56.3
- new net N$68: J4G$1.CEC, S57.3
- new net N$69: J4G$1.TMDSCLOCK-, S58.3
- new net N$70: J4G$1.TMDSCLOCKSHIELD, S59.3
- new net N$71: J4G$1.TMDSCLOCK+, S50.3
- new net N$72: J4G$1.TMDSDATA0-, S49.3
- new net N$73: J4G$1.TMDSDATA0SHIELD, S48.3
- new net N$74: J4G$1.TMDSDATA0+, S47.3
- new net N$75: J4G$1.TMDSDATA1-, S46.3
- new net N$76: J4G$1.TMDSDATA1SHIELD, S45.3
- new net N$77: J4G$1.TMDSDATA1+, S44.3
- new net N$80: J4G$1.TMDSDATA2-, S43.3
- new net N$81: J4G$1.TMDSDATA2SHIELD, S42.3
- new net N$82: J4G$1.TMDSDATA2+, S41.3
- new net N$83: S62.2
- new net N$94: J3SHIELD.SHIELD, S20.3
- new net PC1HDMI-+5V: J1G$1.+5VPOWER, S16.4, S32.4, S52.4, S72.4
- new net PC1HDMI-CEC: J1G$1.CEC, S13.4, S37.4, S57.4, S77.4
- new net PC1HDMI-DCC: J1G$1.DDC/CECGROUND, S17.4, S33.4, S53.4, S73.4
- new net PC1HDMI-HOT: J1G$1.HOTPLUGDETECT/HEAC-, S11.4, S31.4, S51.4, S71.4
- new net PC1HDMI-SCL: J1G$1.SCL, S19.4, S35.4, S55.4, S75.4
- new net PC1HDMI-SDA: J1G$1.SDA, S18.4, S34.4, S54.4, S74.4
- new net PC1HDMI-TMD0S: J1G$1.TMDSDATA0SHIELD, S28.4, S48.4, S68.4, S8.4
- new net PC1HDMI-TMDS1+: J1G$1.TMDSDATA1+, S24.4, S4.4, S44.4, S64.4
- new net PC1HDMI-TMDS1-: J1G$1.TMDSDATA1-, S26.4, S46.4, S6.4, S66.4
- new net PC1HDMI-TMDSC+: J1G$1.TMDSCLOCK+, S10.4, S30.4, S50.4, S70.4
- new net PC1HDMI-TMDSC-: J1G$1.TMDSCLOCK-, S14.4, S38.4, S58.4, S78.4
- new net PC1HDMI-TMDSCS: J1G$1.TMDSCLOCKSHIELD, S15.4, S39.4, S59.4, S79.4
- new net PC1HDMI-TMDSD0+: J1G$1.TMDSDATA0+, S27.4, S47.4, S67.4, S7.4
- new net PC1HDMI-TMDSD0-: J1G$1.TMDSDATA0-, S29.4, S49.4, S69.4, S9.4
- new net PC1HDMI-TMDSD1S: J1G$1.TMDSDATA1SHIELD, S25.4, S45.4, S5.4, S65.4
- new net PC1HDMI-TMDSD2+: J1G$1.TMDSDATA2+, S2.4, S21.4, S41.4, S61.4
- new net PC1HDMI-TMDSD2-: J1G$1.TMDSDATA2-, S1.4, S23.4, S43.4, S63.4
- new net PC1HDMI-TMDSD2S: J1G$1.TMDSDATA2SHIELD, S22.4, S3.4, S42.4, S62.4
- new net PC1HDMI-UTL+: J1G$1.UTILITY/HEAC+, S12.4, S36.4, S56.4, S76.4
- new net PC1USBC-CC1: S104.4, S116.4, S128.4, S93.4, U$1.CC1/VCONN
- new net PC1USBC-CC2: S105.4, S117.4, S81.4, S87.4, U$1.CC2/VCONN
- new net PC1USBC-D+: S103.4, S115.4, S127.4, S92.4, U$1.D+
- new net PC1USBC-D-: S102.4, S114.4, S126.4, S91.4, U$1.D-
- new net PC1USBC-GND: S107.4, S119.4, S83.4, S95.4, U$1.GND
- new net PC1USBC-SBU: S101.4, S113.4, S125.4, S90.4, U$1.SBU
- new net PC1USBC-SHIELD: S106.4, S118.4, S82.4, S94.4, U$1.SHIELD
- new net PC1USBC-SSRX+: S111.4, S123.4, S88.4, S99.4, U$1.SSRX+
- new net PC1USBC-SSRX-: S100.4, S112.4, S124.4, S89.4, U$1.SSRX-
- new net PC1USBC-SSTX+: S108.4, S120.4, S84.4, S96.4, U$1.SSTX+
- new net PC1USBC-SSTX-: S109.4, S121.4, S85.4, S97.4, U$1.SSTX-
- new net PC1USBC-VBUS: S110.4, S122.4, S86.4, S98.4, U$1.VBUS
- new net PC2HDMI-+5V: S16.2, S32.2, S52.2, S72.2
- new net PC2HDMI-CEC: S13.2, S37.2, S57.2, S77.2
- new net PC2HDMI-DCC: S17.2, S33.2, S53.2, S73.2
- new net PC2HDMI-HOT: S11.2, S31.2, S51.2, S71.2
- new net PC2HDMI-SCL: S19.2, S35.2, S55.2, S75.2
- new net PC2HDMI-SDA: S18.2, S34.2, S54.2, S74.2
- new net PC2HDMI-SHEILD: S20.2, S40.2, S60.2, S80.2
- new net PC2HDMI-TMD0S: S28.2, S48.2, S68.2, S8.2
- new net PC2HDMI-TMDS1+: S24.2, S4.2, S44.2, S64.2
- new net PC2HDMI-TMDS1-: S26.2, S46.2, S6.2, S66.2
- new net PC2HDMI-TMDSC+: S10.2, S30.2, S50.2, S70.2
- new net PC2HDMI-TMDSC-: S14.2, S38.2, S58.2, S78.2
- new net PC2HDMI-TMDSCS: S15.2, S39.2, S59.2, S79.2
- new net PC2HDMI-TMDSD0+: S27.2, S47.2, S67.2, S7.2
- new net PC2HDMI-TMDSD0-: S29.2, S49.2, S69.2, S9.2
- new net PC2HDMI-TMDSD1S: S25.2, S45.2, S5.2, S65.2
- new net PC2HDMI-TMDSD2+: S2.2, S21.2, S41.2, S61.2
- new net PC2HDMI-TMDSD2-: S1.2, S23.2, S43.2, S63.2
- new net PC2HDMI-UTL+: S12.2, S36.2, S56.2, S76.2
- new net PC2USBC-CC1: S104.2, S116.2, S128.2, S93.2
- new net PC2USBC-CC2: S105.2, S117.2, S81.2, S87.2
- new net PC2USBC-D+: S103.2, S115.2, S127.2, S92.2
- new net PC2USBC-D-: S102.2, S114.2, S126.2, S91.2
- new net PC2USBC-GND: S107.2, S119.2, S83.2, S95.2
- new net PC2USBC-SBU: S101.2, S113.2, S125.2, S90.2
- new net PC2USBC-SHIELD: S106.2, S118.2, S82.2, S94.2
- new net PC2USBC-SSRX+: S111.2, S123.2, S88.2, S99.2
- new net PC2USBC-SSRX-: S100.2, S112.2, S124.2, S89.2
- new net PC2USBC-SSTX+: S108.2, S120.2, S84.2, S96.2
- new net PC2USBC-SSTX-: S109.2, S121.2, S85.2, S97.2
- new net PC2USBC-VBUS: S110.2, S122.2, S86.2, S98.2
- new net PC3HDMI-+5V: S16.1, S32.1, S52.1, S72.1
- new net PC3HDMI-CEC: S13.1, S37.1, S57.1, S77.1
- new net PC3HDMI-DCC: S17.1, S33.1, S53.1, S73.1
- new net PC3HDMI-HOT: S11.1, S31.1, S51.1, S71.1
- new net PC3HDMI-SCL: S19.1, S35.1, S55.1, S75.1
- new net PC3HDMI-SDA: S18.1, S34.1, S54.1, S74.1
- new net PC3HDMI-SHEILD: S20.1, S40.1, S60.1, S80.1
- new net PC3HDMI-TMD0S: S28.1, S48.1, S68.1, S8.1
- new net PC3HDMI-TMDS1+: S24.1, S4.1, S44.1, S64.1
- new net PC3HDMI-TMDS1-: S26.1, S46.1, S6.1, S66.1
- new net PC3HDMI-TMDSC+: S10.1, S30.1, S50.1, S70.1
- new net PC3HDMI-TMDSC-: S14.1, S38.1, S58.1, S78.1
- new net PC3HDMI-TMDSCS: S15.1, S39.1, S59.1, S79.1
- new net PC3HDMI-TMDSD0+: S27.1, S47.1, S67.1, S7.1
- new net PC3HDMI-TMDSD0-: S29.1, S49.1, S69.1, S9.1
- new net PC3HDMI-TMDSD1S: S25.1, S45.1, S5.1, S65.1
- new net PC3HDMI-TMDSD2+: S2.1, S21.1, S41.1, S61.1
- new net PC3HDMI-TMDSD2-: S1.1, S23.1, S43.1, S63.1
- new net PC3HDMI-TMDSD2S: S22.1, S3.1, S42.1, S62.1
- new net PC3HDMI-UTL+: S12.1, S36.1, S56.1, S76.1
- new net PC3USBC-CC1: S104.1, S116.1, S128.1, S93.1
- new net PC3USBC-CC2: S105.1, S117.1, S81.1, S87.1
- new net PC3USBC-D+: S103.1, S115.1, S127.1, S92.1
- new net PC3USBC-D-: S102.1, S114.1, S126.1, S91.1
- new net PC3USBC-GND: S107.1, S119.1, S83.1, S95.1
- new net PC3USBC-SBU: S101.1, S113.1, S125.1, S90.1
- new net PC3USBC-SHIELD: S106.1, S118.1, S82.1, S94.1
- new net PC3USBC-SSRX+: S111.1, S123.1, S88.1, S99.1
- new net PC3USBC-SSRX-: S100.1, S112.1, S124.1, S89.1
- new net PC3USBC-SSTX+: S108.1, S120.1, S84.1, S96.1
- new net PC3USBC-SSTX-: S109.1, S121.1, S85.1, S97.1
- new net PC3USBC-VBUS: S110.1, S122.1, S86.1, S98.1
- net N$10: now also J3G$1.TMDSCLOCKSHIELD, S15.3; no longer J10G$1.CC1, T38.E
- net N$11: now also J3G$1.TMDSCLOCK+, S10.3; no longer J10G$1.SSTXN1, T39.E
- net N$12: now also J3G$1.TMDSDATA0-, S9.3; no longer J10G$1.SSTXP1, T40.E
- net N$13: now also J3G$1.TMDSDATA0SHIELD, S8.3; no longer J10G$1.SSTXP2, T27.E
- net N$130: now also S89.3, U$2.SSRX-; no longer LED5.A, SW1.1
- net N$131: now also S88.3, U$2.SSRX+; no longer LED6.A, SW1.2
- net N$132: now also S104.3, U$3.CC1/VCONN; no longer LED7.A, SW1.4
- net N$133: now also S97.3, U$3.SSTX-; no longer LED8.A, SW1.8
- net N$14: now also J3G$1.TMDSDATA0+, S7.3; no longer J10G$1.SSTXN2, T28.E
- net N$15: now also J3G$1.TMDSDATA1-, S6.3; no longer J10G$1.CC2, T29.E
- net N$16: now also J3G$1.TMDSDATA1SHIELD, S5.3; no longer J10G$1.DP2, T30.E
- net N$17: now also J3G$1.TMDSDATA1+, S4.3; no longer J10G$1.DN2, T31.E
- net N$19: now also J3G$1.TMDSDATA2SHIELD, S3.3; no longer J10G$1.SBU2, T32.E
- net N$2: now also J3G$1.+5VPOWER, S16.3; no longer J10G$1.GND1, J10G$1.GND3
- net N$3: now also J3G$1.DDC/CECGROUND, S17.3; no longer J10G$1.VBUS1, J10G$1.VBUS3
- net N$39: now also J2G$1.TMDSCLOCK-, S38.3; no longer J10G$1.SSRXP1, T34.E
- net N$4: now also S3.2; no longer J10G$1.SSRXP2, T35.E
- net N$40: now also J2G$1.TMDSCLOCKSHIELD, S39.3; no longer J10G$1.SSRXN1, T33.E
- net N$5: now also J3G$1.SDA, S18.3; no longer R1.2, SW2.C
- net N$7: now also J3G$1.UTILITY/HEAC+, S12.3; no longer J10G$1.SSRXN2, T36.E
- net N$8: now also J3G$1.CEC, S13.3; no longer J10G$1.SBU1, T37.E
- net N$9: now also J3G$1.TMDSCLOCK-, S14.3; no longer LED4.A, SW2.8
- net VBUS: now also S110.3, S122.3, S86.3, S98.3, U$2.VBUS, U$3.VBUS, U$4.VBUS, U$5.VBUS; no longer J10G$1.VBUS, J10G$1.VBUS2, J7.VBUS, R1.1
Other:
- note added: "PC1"
- moved on the sheet: J2G$1, J2SHIELD, J3G$1, J3SHIELD

Commit message: s
s
Parts:
- removed J3, J4: (no value), Wurth_Elektronik_Electromechanic_Input-Output_Connectors_rev17b:685119134923
- removed S10, S100, S101, S102, S103, S104, S105, S106, S107, S108, S109, S11, S110, S111, S112, S113, S114, S115, S116, S117, S118, S119, S12, S120, S121, S122, S123, S124, S125, S126, S127, S128, S13, S14, S15, S16, S17, S18, S19, S20, S21, S22, S23, S24, S25, S26, S27, S28, S29, S30, S31, S32, S33, S34, S35, S36, S37, S38, S39, S40, S41, S42, S43, S44, S45, S46, S47, S48, S49, S5, S50, S51, S52, S53, S54, S55, S56, S57, S58, S59, S6, S60, S7, S8, S81, S82, S83, S84, S85, S86, S87, S88, S89, S9, S90, S91, S92, S93, S94, S95, S96, S97, S98, S99: (no value), SparkFun-Switches:SWITCH-SP3T-SMD
- added U1, U2, U3, U4: SN74CBT16214DGGR, SN74CBT16214DGGR:SN74CBT16214DGGR
- added U5: TMDS361BPAG, TMDS361BPAG:TMDS361BPAG
Connections:
- removed net N$121: S93.3, U$2.CC1/VCONN
- removed net N$122: S85.3, U$2.SSTX-
- removed net N$123: S84.3, U$2.SSTX+
- removed net N$124: S83.3, U$2.GND
- removed net N$125: S82.3, U$2.SHIELD
- removed net N$126: S81.3, U$2.CC2/VCONN
- removed net N$127: S92.3, U$2.D+
- removed net N$128: S91.3, U$2.D-
- removed net N$129: S90.3, U$2.SBU
- removed net N$130: S89.3, U$2.SSRX-
- removed net N$131: S88.3, U$2.SSRX+
- removed net N$143: S116.3, U$4.CC1/VCONN
- removed net N$144: S109.3, U$4.SSTX-
- removed net N$145: S108.3, U$4.SSTX+
- removed net N$146: S107.3, U$4.GND
- removed net N$147: S106.3, U$4.SHIELD
- removed net N$148: S105.3, U$4.CC2/VCONN
- removed net N$149: S115.3, U$4.D+
- removed net N$150: S114.3, U$4.D-
- removed net N$151: S113.3, U$4.SBU
- removed net N$152: S112.3, U$4.SSRX-
- removed net N$153: S111.3, U$4.SSRX+
- removed net N$154: S128.3, U$5.CC1/VCONN
- removed net N$155: S121.3, U$5.SSTX-
- removed net N$156: S120.3, U$5.SSTX+
- removed net N$157: S119.3, U$5.GND
- removed net N$158: S118.3, U$5.SHIELD
- removed net N$159: S117.3, U$5.CC2/VCONN
- removed net N$160: S127.3, U$5.D+
- removed net N$161: S126.3, U$5.D-
- removed net N$162: S125.3, U$5.SBU
- removed net N$163: S124.3, U$5.SSRX-
- removed net N$164: S123.3, U$5.SSRX+
- removed net N$61: J4SHIELD.SHIELD, S60.3
- removed net N$62: J4G$1.HOTPLUGDETECT/HEAC-, S51.3
- removed net N$63: J4G$1.+5VPOWER, S52.3
- removed net N$64: J4G$1.DDC/CECGROUND, S53.3
- removed net N$65: J4G$1.SDA, S54.3
- removed net N$66: J4G$1.SCL, S55.3
- removed net N$67: J4G$1.UTILITY/HEAC+, S56.3
- removed net N$68: J4G$1.CEC, S57.3
- removed net N$69: J4G$1.TMDSCLOCK-, S58.3
- removed net N$70: J4G$1.TMDSCLOCKSHIELD, S59.3
- removed net N$71: J4G$1.TMDSCLOCK+, S50.3
- removed net N$72: J4G$1.TMDSDATA0-, S49.3
- removed net N$73: J4G$1.TMDSDATA0SHIELD, S48.3
- removed net N$74: J4G$1.TMDSDATA0+, S47.3
- removed net N$75: J4G$1.TMDSDATA1-, S46.3
- removed net N$76: J4G$1.TMDSDATA1SHIELD, S45.3
- removed net N$77: J4G$1.TMDSDATA1+, S44.3
- removed net N$80: J4G$1.TMDSDATA2-, S43.3
- removed net N$81: J4G$1.TMDSDATA2SHIELD, S42.3
- removed net N$82: J4G$1.TMDSDATA2+, S41.3
- removed net N$94: J3SHIELD.SHIELD, S20.3
- new net 5.5V: S1.3, S2.3, S3.3, S4.3, U1.VCC, U2.VCC, U3.VCC, U4.VCC
- new net GND: U1.GND, U1.GND-1, U1.GND-2, U1.GND-3, U2.GND, U2.GND-1, U2.GND-2, U2.GND-3, U3.GND, U3.GND-1, U3.GND-2, U3.GND-3, U4.GND, U4.GND-1, U4.GND-2, U4.GND-3
- new net N$22: U$4.SSRX+, U3.3A
- new net N$23: U$5.CC1/VCONN, U4.8A
- new net N$24: U$5.SSTX-, U4.10A
- new net N$25: U$5.SSTX+, U4.11A
- new net N$26: U$5.GND, U4.12A
- new net N$27: U$5.SHIELD, U4.1A
- new net N$28: U$5.CC2/VCONN, U4.2A
- new net N$29: U$5.D+, U4.7A
- new net N$30: U$5.D-, U4.6A
- new net N$52: J2G$1.TMDSCLOCK-, U5.CLK-_SINK
- new net N$53: J2G$1.TMDSCLOCK+, U5.CLK+_SINK
- new net PC1HDMI-SHEILD: S80.4
- net N$1: now also U$2.CC1/VCONN, U2.8A; no longer J3G$1.HOTPLUGDETECT/HEAC-, S11.3
- net N$10: now also U$2.SSRX-, U2.4A; no longer J3G$1.TMDSCLOCKSHIELD, S15.3
- net N$11: now also U$2.SSRX+, U2.3A; no longer J3G$1.TMDSCLOCK+, S10.3
- net N$12: now also U$4.CC1/VCONN, U3.8A; no longer J3G$1.TMDSDATA0-, S9.3
- net N$13: now also U$4.SSTX-, U3.10A; no longer J3G$1.TMDSDATA0SHIELD, S8.3
- net N$132: now also U1.8A; no longer S104.3
- net N$133: now also U1.10A; no longer S97.3
- net N$134: now also U1.11A; no longer S96.3
- net N$135: now also U1.12A; no longer S95.3
- net N$136: now also U1.1A; no longer S94.3
- net N$137: now also U1.2A; no longer S87.3
- net N$138: now also U1.7A; no longer S103.3
- net N$139: now also U1.6A; no longer S102.3
- net N$14: now also U$4.SSTX+, U3.11A; no longer J3G$1.TMDSDATA0+, S7.3
- net N$140: now also U1.5A; no longer S101.3
- net N$141: now also U1.4A; no longer S100.3
- net N$142: now also U1.3A; no longer S99.3
- net N$15: now also U$4.GND, U3.12A; no longer J3G$1.TMDSDATA1-, S6.3
- net N$16: now also U$4.SHIELD, U3.1A; no longer J3G$1.TMDSDATA1SHIELD, S5.3
- net N$17: now also U$4.CC2/VCONN, U3.2A; no longer J3G$1.TMDSDATA1+, S4.3
- net N$18: now also U$4.D+, U3.7A; no longer J3G$1.TMDSDATA2-, S1.3
- net N$19: now also U$4.D-, U3.6A; no longer J3G$1.TMDSDATA2SHIELD, S3.3
- net N$2: now also U$2.SSTX-, U2.10A; no longer J3G$1.+5VPOWER, S16.3
- net N$20: now also U$4.SBU, U3.5A; no longer J3G$1.TMDSDATA2+, S2.3
- net N$21: now also U$4.SSRX-, U3.4A; no longer S22.2
- net N$3: now also U$2.SSTX+, U2.11A; no longer J3G$1.DDC/CECGROUND, S17.3
- net N$31: now also U$5.SBU, U4.5A; no longer J2SHIELD.SHIELD, S40.3
- net N$32: now also U$5.SSRX-, U4.4A; no longer J2G$1.HOTPLUGDETECT/HEAC-, S31.3
- net N$33: now also U$5.SSRX+, U4.3A; no longer J2G$1.+5VPOWER, S32.3
- net N$34: now also S2.4, U2.S1; no longer J2G$1.DDC/CECGROUND, S33.3
- net N$35: now also S1.4, U1.S1; no longer J2G$1.SDA, S34.3
- net N$36: now also S1.2, U1.S2; no longer J2G$1.SCL, S35.3
- net N$37: now also S1.1, U1.SO; no longer J2G$1.UTILITY/HEAC+, S36.3
- net N$38: now also S2.2, U2.S2; no longer J2G$1.CEC, S37.3
- net N$39: now also S2.1, U2.SO; no longer J2G$1.TMDSCLOCK-, S38.3
- net N$4: now also U$2.GND, U2.12A; no longer S3.2
- net N$40: now also S3.4, U4.S1; no longer J2G$1.TMDSCLOCKSHIELD, S39.3
- net N$41: now also S3.2, U4.S2; no longer J2G$1.TMDSCLOCK+, S30.3
- net N$42: now also S3.1, U4.SO; no longer J2G$1.TMDSDATA0-, S29.3
- net N$43: now also S4.4, U3.S1; no longer J2G$1.TMDSDATA0SHIELD, S28.3
- net N$44: now also S4.2, U3.S2; no longer J2G$1.TMDSDATA0+, S27.3
- net N$45: now also S4.1, U3.SO; no longer J2G$1.TMDSDATA1-, S26.3
- net N$46: now also J2G$1.TMDSDATA2-, U5.D2-_SINK; no longer J2G$1.TMDSDATA1SHIELD, S25.3
- net N$47: now also J2G$1.TMDSDATA2+, U5.D2+_SINK; no longer J2G$1.TMDSDATA1+, S24.3
- net N$48: now also J2G$1.TMDSDATA1-, U5.D1-_SINK; no longer J2G$1.TMDSDATA2-, S23.3
- net N$49: now also J2G$1.TMDSDATA1+, U5.D1+_SINK; no longer J2G$1.TMDSDATA2SHIELD, S22.3
- net N$5: now also U$2.SHIELD, U2.1A; no longer J3G$1.SDA, S18.3
- net N$50: now also J2G$1.TMDSDATA0-, U5.D0-_SINK; no longer J2G$1.TMDSDATA2+, S21.3
- net N$51: now also J2G$1.TMDSDATA0+, U5.D0+_SINK; no longer S42.2
- net N$6: now also U$2.CC2/VCONN, U2.2A; no longer J3G$1.SCL, S19.3
- net N$7: now also U$2.D+, U2.7A; no longer J3G$1.UTILITY/HEAC+, S12.3
- net N$8: now also U$2.D-, U2.6A; no longer J3G$1.CEC, S13.3
- net N$9: now also U$2.SBU, U2.5A; no longer J3G$1.TMDSCLOCK-, S14.3
- net PC1HDMI-+5V: no longer S16.4, S32.4, S52.4
- net PC1HDMI-CEC: no longer S13.4, S37.4, S57.4
- net PC1HDMI-DCC: no longer S17.4, S33.4, S53.4
- net PC1HDMI-HOT: no longer S11.4, S31.4, S51.4
- net PC1HDMI-SCL: no longer S19.4, S35.4, S55.4
- net PC1HDMI-SDA: no longer S18.4, S34.4, S54.4
- net PC1HDMI-TMD0S: no longer S28.4, S48.4, S8.4
- net PC1HDMI-TMDS1+: no longer S24.4, S4.4, S44.4
- net PC1HDMI-TMDS1-: no longer S26.4, S46.4, S6.4
- net PC1HDMI-TMDSC+: no longer S10.4, S30.4, S50.4
- net PC1HDMI-TMDSC-: no longer S14.4, S38.4, S58.4
- net PC1HDMI-TMDSCS: no longer S15.4, S39.4, S59.4
- net PC1HDMI-TMDSD0+: no longer S27.4, S47.4, S7.4
- net PC1HDMI-TMDSD0-: no longer S29.4, S49.4, S9.4
- net PC1HDMI-TMDSD1S: no longer S25.4, S45.4, S5.4
- net PC1HDMI-TMDSD2+: no longer S2.4, S21.4, S41.4
- net PC1HDMI-TMDSD2-: no longer S1.4, S23.4, S43.4
- net PC1HDMI-TMDSD2S: no longer S22.4, S3.4, S42.4
- net PC1HDMI-UTL+: no longer S12.4, S36.4, S56.4
- net PC1USBC-CC1: now also U1.8B1, U2.8B1, U3.8B1, U4.8B1; no longer S104.4, S116.4, S128.4, S93.4
- net PC1USBC-CC2: now also U1.2B1, U2.2B1, U3.2B1, U4.2B1; no longer S105.4, S117.4, S81.4, S87.4
- net PC1USBC-D+: now also U1.7B1, U2.7B1, U3.7B1, U4.7B1; no longer S103.4, S115.4, S127.4, S92.4
- net PC1USBC-D-: now also U1.6B1, U2.6B1, U3.6B1, U4.6B1; no longer S102.4, S114.4, S126.4, S91.4
- net PC1USBC-GND: now also U1.12B1, U2.12B1, U3.12B1, U4.12B1; no longer S107.4, S119.4, S83.4, S95.4
- net PC1USBC-SBU: now also U1.5B1, U2.5B1, U3.5B1, U4.5B1; no longer S101.4, S113.4, S125.4, S90.4
- net PC1USBC-SHIELD: now also U1.1B1, U2.1B1, U3.1B1, U4.1B1; no longer S106.4, S118.4, S82.4, S94.4
- net PC1USBC-SSRX+: now also U1.3B1, U2.3B1, U3.3B1, U4.3B1; no longer S111.4, S123.4, S88.4, S99.4
- net PC1USBC-SSRX-: now also U1.4B1, U2.4B1, U3.4B1, U4.4B1; no longer S100.4, S112.4, S124.4, S89.4
- net PC1USBC-SSTX+: now also U1.11B1, U2.11B1, U3.11B1, U4.11B1; no longer S108.4, S120.4, S84.4, S96.4
- net PC1USBC-SSTX-: now also U1.10B1, U2.10B1, U3.10B1, U4.10B1; no longer S109.4, S121.4, S85.4, S97.4
- net PC1USBC-VBUS: now also U1.9B1, U2.9B1, U3.9B1, U4.9B1; no longer S110.4, S122.4, S86.4, S98.4
- net PC2HDMI-+5V: no longer S16.2, S32.2, S52.2
- net PC2HDMI-CEC: no longer S13.2, S37.2, S57.2
- net PC2HDMI-DCC: no longer S17.2, S33.2, S53.2
- net PC2HDMI-HOT: no longer S11.2, S31.2, S51.2
- net PC2HDMI-SCL: no longer S19.2, S35.2, S55.2
- net PC2HDMI-SDA: no longer S18.2, S34.2, S54.2
- net PC2HDMI-SHEILD: no longer S20.2, S40.2, S60.2
- net PC2HDMI-TMD0S: no longer S28.2, S48.2, S8.2
- net PC2HDMI-TMDS1+: no longer S24.2, S4.2, S44.2
- net PC2HDMI-TMDS1-: no longer S26.2, S46.2, S6.2
- net PC2HDMI-TMDSC+: no longer S10.2, S30.2, S50.2
- net PC2HDMI-TMDSC-: no longer S14.2, S38.2, S58.2
- net PC2HDMI-TMDSCS: no longer S15.2, S39.2, S59.2
- net PC2HDMI-TMDSD0+: no longer S27.2, S47.2, S7.2
- net PC2HDMI-TMDSD0-: no longer S29.2, S49.2, S9.2
- net PC2HDMI-TMDSD1S: no longer S25.2, S45.2, S5.2
- net PC2HDMI-TMDSD2+: no longer S2.2, S21.2, S41.2
- net PC2HDMI-TMDSD2-: no longer S1.2, S23.2, S43.2
- net PC2HDMI-UTL+: no longer S12.2, S36.2, S56.2
- net PC2USBC-CC1: now also U1.8B2, U2.8B2, U3.8B2, U4.8B2; no longer S104.2, S116.2, S128.2, S93.2
- net PC2USBC-CC2: now also U1.2B2, U2.2B2, U3.2B2, U4.2B2; no longer S105.2, S117.2, S81.2, S87.2
- net PC2USBC-D+: now also U1.7B2, U2.7B2, U3.7B2, U4.7B2; no longer S103.2, S115.2, S127.2, S92.2
- net PC2USBC-D-: now also U1.6B2, U2.6B2, U3.6B2, U4.6B2; no longer S102.2, S114.2, S126.2, S91.2
- net PC2USBC-GND: now also U1.12B2, U2.12B2, U3.12B2, U4.12B2; no longer S107.2, S119.2, S83.2, S95.2
- net PC2USBC-SBU: now also U1.5B2, U2.5B2, U3.5B2, U4.5B2; no longer S101.2, S113.2, S125.2, S90.2
- net PC2USBC-SHIELD: now also U1.1B2, U2.1B2, U3.1B2, U4.1B2; no longer S106.2, S118.2, S82.2, S94.2
- net PC2USBC-SSRX+: now also U1.3B2, U2.3B2, U3.3B2, U4.3B2; no longer S111.2, S123.2, S88.2, S99.2
- net PC2USBC-SSRX-: now also U1.4B2, U2.4B2, U3.4B2, U4.4B2; no longer S100.2, S112.2, S124.2, S89.2
- net PC2USBC-SSTX+: now also U1.11B2, U2.11B2, U3.11B2, U4.11B2; no longer S108.2, S120.2, S84.2, S96.2
- net PC2USBC-SSTX-: now also U1.10B2, U2.10B2, U3.10B2, U4.10B2; no longer S109.2, S121.2, S85.2, S97.2
- net PC2USBC-VBUS: now also U1.9B2, U2.9B2, U3.9B2, U4.9B2; no longer S110.2, S122.2, S86.2, S98.2
- net PC3HDMI-+5V: no longer S16.1, S32.1, S52.1
- net PC3HDMI-CEC: no longer S13.1, S37.1, S57.1
- net PC3HDMI-DCC: no longer S17.1, S33.1, S53.1
- net PC3HDMI-HOT: no longer S11.1, S31.1, S51.1
- net PC3HDMI-SCL: no longer S19.1, S35.1, S55.1
- net PC3HDMI-SDA: no longer S18.1, S34.1, S54.1
- net PC3HDMI-SHEILD: no longer S20.1, S40.1, S60.1
- net PC3HDMI-TMD0S: no longer S28.1, S48.1, S8.1
- net PC3HDMI-TMDS1+: no longer S24.1, S4.1, S44.1
- net PC3HDMI-TMDS1-: no longer S26.1, S46.1, S6.1
- net PC3HDMI-TMDSC+: no longer S10.1, S30.1, S50.1
- net PC3HDMI-TMDSC-: no longer S14.1, S38.1, S58.1
- net PC3HDMI-TMDSCS: no longer S15.1, S39.1, S59.1
- net PC3HDMI-TMDSD0+: no longer S27.1, S47.1, S7.1
- net PC3HDMI-TMDSD0-: no longer S29.1, S49.1, S9.1
- net PC3HDMI-TMDSD1S: no longer S25.1, S45.1, S5.1
- net PC3HDMI-TMDSD2+: no longer S2.1, S21.1, S41.1
- net PC3HDMI-TMDSD2-: no longer S1.1, S23.1, S43.1
- net PC3HDMI-TMDSD2S: no longer S22.1, S3.1, S42.1
- net PC3HDMI-UTL+: no longer S12.1, S36.1, S56.1
- net PC3USBC-CC1: now also U1.8B3, U2.8B3, U3.8B3, U4.8B3; no longer S104.1, S116.1, S128.1, S93.1
- net PC3USBC-CC2: now also U1.2B3, U2.2B3, U3.2B3, U4.2B3; no longer S105.1, S117.1, S81.1, S87.1
- net PC3USBC-D+: now also U1.7B3, U2.7B3, U3.7B3, U4.7B3; no longer S103.1, S115.1, S127.1, S92.1
- net PC3USBC-D-: now also U1.6B3, U2.6B3, U3.6B3, U4.6B3; no longer S102.1, S114.1, S126.1, S91.1
- net PC3USBC-GND: now also U1.12B3, U2.12B3, U3.12B3, U4.12B3; no longer S107.1, S119.1, S83.1, S95.1
- net PC3USBC-SBU: now also U1.5B3, U2.5B3, U3.5B3, U4.5B3; no longer S101.1, S113.1, S125.1, S90.1
- net PC3USBC-SHIELD: now also U1.1B3, U2.1B3, U3.1B3, U4.1B3; no longer S106.1, S118.1, S82.1, S94.1
- net PC3USBC-SSRX+: now also U1.3B3, U2.3B3, U3.3B3, U4.3B3; no longer S111.1, S123.1, S88.1, S99.1
- net PC3USBC-SSRX-: now also U1.4B3, U2.4B3, U3.4B3, U4.4B3; no longer S100.1, S112.1, S124.1, S89.1
- net PC3USBC-SSTX+: now also U1.11B3, U2.11B3, U3.11B3, U4.11B3; no longer S108.1, S120.1, S84.1, S96.1
- net PC3USBC-SSTX-: now also U1.10B3, U2.10B3, U3.10B3, U4.10B3; no longer S109.1, S121.1, S85.1, S97.1
- net PC3USBC-VBUS: now also U1.9B3, U2.9B3, U3.9B3, U4.9B3; no longer S110.1, S122.1, S86.1, S98.1
- net VBUS: now also U1.9A, U2.9A, U3.9A, U4.9A; no longer S110.3, S122.3, S86.3, S98.3
Other:
- note added: "USB Type C IN/OUT"
- moved on the sheet: J2G$1, J5G$1, J5SHIELD, S1, S2, S3, S4, S61, S62, S63, S64, S65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
