File: pchub/pchub.sch (EAGLE design)
At the start: 37 parts, among them U1 SN74CBT16214DGGR, U2 SN74CBT16214DGGR, U3 SN74CBT16214DGGR, U4 SN74CBT16214DGGR, U5 TMDS361BPAG

Commit message: s
s
Parts:
- removed S61, S62, S63, S64, S65, S66, S67, S68, S69, S70, S71, S72, S73, S74, S75, S76, S77, S78, S79, S80: (no value), SparkFun-Switches:SWITCH-SP3T-SMD
- added D1, D10, D11, D12, D2, D3, D4, D5, D6, D7, D8, D9: (no value), SparkFun-LED:LED-FKIT-1206
- added J3, J4: (no value), Wurth_Elektronik_Electromechanic_Input-Output_Connectors_rev17b:685119134923
- added J6, J7: 2040210-1, 2040210-1:2040210-1
- added S10, S11, S12, S13, S14, S15, S16, S5, S6, S7, S8, S9: (no value), SparkFun-Switches:SWITCH-SP3T-SMD
- added U10, U11, U12, U13, U14, U15, U16, U17, U18, U19, U20, U9: FSUSB63UMX, FSUSB63UMX:FSUSB63UMX
- added U6, U7, U8: TMDS361BPAG, TMDS361BPAG:TMDS361BPAG
- added X1, X10, X11, X12, X13, X2, X3, X4, X5, X6, X7, X8, X9: USB, SparkFun:USB
Connections:
- removed net PC1HDMI-+5V: J1G$1.+5VPOWER, S72.4
- removed net PC1HDMI-CEC: J1G$1.CEC, S77.4
- removed net PC1HDMI-DCC: J1G$1.DDC/CECGROUND, S73.4
- removed net PC1HDMI-SHEILD: S80.4
- removed net PC1HDMI-TMD0S: J1G$1.TMDSDATA0SHIELD, S68.4
- removed net PC1HDMI-TMDSCS: J1G$1.TMDSCLOCKSHIELD, S79.4
- removed net PC1HDMI-TMDSD1S: J1G$1.TMDSDATA1SHIELD, S65.4
- removed net PC1HDMI-TMDSD2S: J1G$1.TMDSDATA2SHIELD, S62.4
- removed net PC1HDMI-UTL+: J1G$1.UTILITY/HEAC+, S76.4
- removed net PC2HDMI-+5V: S72.2
- removed net PC2HDMI-CEC: S77.2
- removed net PC2HDMI-DCC: S73.2
- removed net PC2HDMI-SHEILD: S80.2
- removed net PC2HDMI-TMD0S: S68.2
- removed net PC2HDMI-TMDSCS: S79.2
- removed net PC2HDMI-TMDSD1S: S65.2
- removed net PC2HDMI-UTL+: S76.2
- removed net PC3HDMI-+5V: S72.1
- removed net PC3HDMI-CEC: S77.1
- removed net PC3HDMI-DCC: S73.1
- removed net PC3HDMI-SHEILD: S80.1
- removed net PC3HDMI-TMD0S: S68.1
- removed net PC3HDMI-TMDSCS: S79.1
- removed net PC3HDMI-TMDSD1S: S65.1
- removed net PC3HDMI-TMDSD2S: S62.1
- removed net PC3HDMI-UTL+: S76.1
- new net CEC: J1G$1.CEC, J2G$1.CEC, J3G$1.CEC, J4G$1.CEC, J5G$1.CEC
- new net HDMIGND: J1G$1.DDC/CECGROUND, J1G$1.TMDSCLOCKSHIELD, J1G$1.TMDSDATA0SHIELD, J1G$1.TMDSDATA1SHIELD, J1G$1.TMDSDATA2SHIELD, J2G$1.DDC/CECGROUND, J2G$1.TMDSCLOCKSHIELD, J2G$1.TMDSDATA0SHIELD, J2G$1.TMDSDATA1SHIELD, J2G$1.TMDSDATA2SHIELD, J2SHIELD.SHIELD, J3G$1.DDC/CECGROUND, J3G$1.TMDSCLOCKSHIELD, J3G$1.TMDSDATA0SHIELD, J3G$1.TMDSDATA1SHIELD, J3G$1.TMDSDATA2SHIELD, J3SHIELD.SHIELD, J4G$1.DDC/CECGROUND, J4G$1.TMDSCLOCKSHIELD, J4G$1.TMDSDATA0SHIELD, J4G$1.TMDSDATA1SHIELD, J4G$1.TMDSDATA2SHIELD, J4SHIELD.SHIELD, J5G$1.DDC/CECGROUND, J5G$1.TMDSCLOCKSHIELD, J5G$1.TMDSDATA0SHIELD, J5G$1.TMDSDATA1SHIELD, J5G$1.TMDSDATA2SHIELD, J5SHIELD.SHIELD, U5.GND, U5.GND_2, U5.GND_3, U5.GND_4, U5.GND_5, U5.GND_6, U5.GND_7, U6.GND, U6.GND_2, U6.GND_3, U6.GND_4, U6.GND_5, U6.GND_6, U6.GND_7, U7.GND, U7.GND_2, U7.GND_3, U7.GND_4, U7.GND_5, U7.GND_6, U7.GND_7, U8.GND, U8.GND_2, U8.GND_3, U8.GND_4, U8.GND_5, U8.GND_6, U8.GND_7
- new net HDMIVCC: J1G$1.+5VPOWER, J2G$1.+5VPOWER, J3G$1.+5VPOWER, J4G$1.+5VPOWER, J5G$1.+5VPOWER, U5.VCC, U5.VCC_2, U5.VCC_3, U5.VCC_4, U5.VCC_5, U5.VCC_6, U5.VCC_7, U5.VCC_8, U6.VCC, U6.VCC_2, U6.VCC_3, U6.VCC_4, U6.VCC_5, U6.VCC_6, U6.VCC_7, U6.VCC_8, U7.VCC, U7.VCC_2, U7.VCC_3, U7.VCC_4, U7.VCC_5, U7.VCC_6, U7.VCC_7, U7.VCC_8, U8.VCC, U8.VCC_2, U8.VCC_3, U8.VCC_4, U8.VCC_5, U8.VCC_6, U8.VCC_7, U8.VCC_8
- new net HEAC+: J1G$1.UTILITY/HEAC+, J2G$1.UTILITY/HEAC+, J3G$1.UTILITY/HEAC+, J4G$1.UTILITY/HEAC+, J5G$1.UTILITY/HEAC+
- new net N$100: D5.C, S9.1, U13.SEL0
- new net N$121: D10.A, S14.2, S14.4, U18.SEL1
- new net N$122: U19.D-, X12.D-
- new net N$123: U19.D+, X12.D+
- new net N$124: D11.C, S15.1, U19.SEL0
- new net N$125: D11.A, S15.2, S15.4, U19.SEL1
- new net N$126: U20.D-, X13.D-
- new net N$127: U20.D+, X13.D+
- new net N$128: D12.C, S16.1, U20.SEL0
- new net N$129: D12.A, S16.2, S16.4, U20.SEL1
- new net N$54: J2G$1.HOTPLUGDETECT/HEAC-, U5.HPD_SINK
- new net N$55: J3G$1.TMDSDATA2-, U6.D2-_SINK
- new net N$56: J3G$1.TMDSDATA2+, U6.D2+_SINK
- new net N$57: J3G$1.TMDSDATA1-, U6.D1-_SINK
- new net N$58: J3G$1.TMDSDATA1+, U6.D1+_SINK
- new net N$59: J3G$1.TMDSDATA0-, U6.D0-_SINK
- new net N$60: J3G$1.TMDSDATA0+, U6.D0+_SINK
- new net N$61: J3G$1.TMDSCLOCK-, U6.CLK-_SINK
- new net N$62: J3G$1.TMDSCLOCK+, U6.CLK+_SINK
- new net N$63: J3G$1.HOTPLUGDETECT/HEAC-, U6.HPD_SINK
- new net N$64: J4G$1.TMDSDATA2-, U7.D2-_SINK
- new net N$65: J4G$1.TMDSDATA2+, U7.D2+_SINK
- new net N$66: J4G$1.TMDSDATA1-, U7.D1-_SINK
- new net N$67: J4G$1.TMDSDATA1+, U7.D1+_SINK
- new net N$68: J4G$1.TMDSDATA0-, U7.D0-_SINK
- new net N$69: J4G$1.TMDSDATA0+, U7.D0+_SINK
- new net N$70: J4G$1.TMDSCLOCK-, U7.CLK-_SINK
- new net N$71: J4G$1.TMDSCLOCK+, U7.CLK+_SINK
- new net N$72: J4G$1.HOTPLUGDETECT/HEAC-, U7.HPD_SINK
- new net N$73: J5G$1.TMDSDATA2-, U8.D2-_SINK
- new net N$74: J5G$1.TMDSDATA2+, U8.D2+_SINK
- new net N$75: J5G$1.TMDSDATA1-, U8.D1-_SINK
- new net N$76: J5G$1.TMDSDATA1+, U8.D1+_SINK
- new net N$77: J5G$1.TMDSDATA0-, U8.D0-_SINK
- new net N$78: J5G$1.TMDSDATA0+, U8.D0+_SINK
- new net N$79: J5G$1.TMDSCLOCK-, U8.CLK-_SINK
- new net N$80: J5G$1.TMDSCLOCK+, U8.CLK+_SINK
- new net N$81: J5G$1.HOTPLUGDETECT/HEAC-, U8.HPD_SINK
- new net N$82: U9.D-, X1.D-
- new net N$84: D1.C, S5.1, U9.SEL0
- new net N$85: U10.D-, X3.D-
- new net N$86: U10.D+, X3.D+
- new net N$87: D1.A, S5.2, S5.4, U9.SEL1
- new net N$88: D2.C, S6.1, U10.SEL0
- new net N$89: D2.A, S6.2, S6.4, U10.SEL1
- new net N$90: U11.D-, X4.D-
- new net N$91: U11.D+, X4.D+
- new net N$92: D3.C, S7.1, U11.SEL0
- new net N$93: D3.A, S7.2, S7.4, U11.SEL1
- new net N$94: U12.D-, X5.D-
- new net N$95: U12.D+, X5.D+
- new net N$96: D4.C, S8.1, U12.SEL0
- new net N$97: D4.A, S8.2, S8.4, U12.SEL1
- new net N$98: U13.D-, X6.D-
- new net N$99: U13.D+, X6.D+
- new net PC1D+: U10.HSD1+, U11.HSD1+, U12.HSD1+, U13.HSD1+, U14.HSD1+, U15.HSD1+, U16.HSD1+, U17.HSD1+, U18.HSD1+, U19.HSD1+, U20.HSD1+, U9.HSD1+, X2.D+
- new net PC1D-: U10.HSD1-, U11.HSD1-, U12.HSD1-, U13.HSD1-, U14.HSD1-, U15.HSD1-, U16.HSD1-, U17.HSD1-, U18.HSD1-, U19.HSD1-, U20.HSD1-, U9.HSD1-, X2.D-
- new net PC2D+: U10.HSD2+, U11.HSD2+, U12.HSD2+, U13.HSD2+, U14.HSD2+, U15.HSD2+, U16.HSD2+, U17.HSD2+, U18.HSD2+, U19.HSD2+, U20.HSD2+, U9.HSD2+
- new net PC2D-: U10.HSD2-, U11.HSD2-, U12.HSD2-, U13.HSD2-, U14.HSD2-, U15.HSD2-, U16.HSD2-, U17.HSD2-, U18.HSD2-, U19.HSD2-, U20.HSD2-, U9.HSD2-
- new net PC3D+: U10.HSD3+, U11.HSD3+, U12.HSD3+, U13.HSD3+, U14.HSD3+, U15.HSD3+, U16.HSD3+, U17.HSD3+, U18.HSD3+, U19.HSD3+, U20.HSD3+, U9.HSD3+
- new net PC3D-: U10.HSD3-, U11.HSD3-, U12.HSD3-, U13.HSD3-, U14.HSD3-, U15.HSD3-, U16.HSD3-, U17.HSD3-, U18.HSD3-, U19.HSD3-, U20.HSD3-, U9.HSD3-
- new net SCL: J2G$1.SCL, J3G$1.SCL, J4G$1.SCL, J5G$1.SCL, U5.SCL_SINK, U6.SCL_SINK, U7.SCL_SINK, U8.SCL_SINK
- new net SDA: J2G$1.SDA, J3G$1.SDA, J4G$1.SDA, J5G$1.SDA, U5.SDA_SINK, U6.SDA_SINK, U7.SDA_SINK, U8.SDA_SINK
- new net USBGND: U10.GND, U11.GND, U12.GND, U13.GND, U14.GND, U15.GND, U16.GND, U17.GND, U18.GND, U19.GND, U20.GND, U9.GND, X1.GND, X10.GND, X11.GND, X12.GND, X13.GND, X2.GND, X3.GND, X4.GND, X5.GND, X6.GND, X7.GND, X8.GND, X9.GND
- new net USBVCC: S10.3, S11.3, S12.3, S13.3, S14.3, S15.3, S16.3, S5.3, S6.3, S7.3, S8.3, S9.3, U10.VCC, U11.VCC, U12.VCC, U13.VCC, U14.VCC, U15.VCC, U16.VCC, U17.VCC, U18.VCC, U19.VCC, U20.VCC, U9.VCC, X1.VBUS, X10.VBUS, X11.VBUS, X12.VBUS, X13.VBUS, X2.VBUS, X3.VBUS, X4.VBUS, X5.VBUS, X6.VBUS, X7.VBUS, X8.VBUS, X9.VBUS
- net N$101: now also D5.A, S9.2, S9.4, U13.SEL1; no longer J5SHIELD.SHIELD, S80.3
- net N$102: now also U14.D-, X7.D-; no longer J5G$1.HOTPLUGDETECT/HEAC-, S71.3
- net N$103: now also U14.D+, X7.D+; no longer J5G$1.+5VPOWER, S72.3
- net N$104: now also D6.C, S10.1, U14.SEL0; no longer J5G$1.DDC/CECGROUND, S73.3
- net N$105: now also D6.A, S10.2, S10.4, U14.SEL1; no longer J5G$1.SDA, S74.3
- net N$106: now also U15.D-, X8.D-; no longer J5G$1.SCL, S75.3
- net N$107: now also U15.D+, X8.D+; no longer J5G$1.UTILITY/HEAC+, S76.3
- net N$108: now also D7.C, S11.1, U15.SEL0; no longer J5G$1.CEC, S77.3
- net N$109: now also D7.A, S11.2, S11.4, U15.SEL1; no longer J5G$1.TMDSCLOCK-, S78.3
- net N$110: now also U16.D-, X9.D-; no longer J5G$1.TMDSCLOCKSHIELD, S79.3
- net N$111: now also U16.D+, X9.D+; no longer J5G$1.TMDSCLOCK+, S70.3
- net N$112: now also D8.C, S12.1, U16.SEL0; no longer J5G$1.TMDSDATA0-, S69.3
- net N$113: now also D8.A, S12.2, S12.4, U16.SEL1; no longer J5G$1.TMDSDATA0SHIELD, S68.3
- net N$114: now also U17.D-, X10.D-; no longer J5G$1.TMDSDATA0+, S67.3
- net N$115: now also U17.D+, X10.D+; no longer J5G$1.TMDSDATA1-, S66.3
- net N$116: now also D9.C, S13.1, U17.SEL0; no longer J5G$1.TMDSDATA1SHIELD, S65.3
- net N$117: now also D9.A, S13.2, S13.4, U17.SEL1; no longer J5G$1.TMDSDATA1+, S64.3
- net N$118: now also U18.D-, X11.D-; no longer J5G$1.TMDSDATA2-, S63.3
- net N$119: now also U18.D+, X11.D+; no longer J5G$1.TMDSDATA2SHIELD, S62.3
- net N$120: now also D10.C, S14.1, U18.SEL0; no longer J5G$1.TMDSDATA2+, S61.3
- net N$83: now also U9.D+, X1.D+; no longer S62.2
- net PC1HDMI-HOT: now also U5.HPD1, U6.HPD1, U7.HPD1, U8.HPD1; no longer S71.4
- net PC1HDMI-SCL: now also U5.SCL1, U6.SCL1, U7.SCL1, U8.SCL1; no longer S75.4
- net PC1HDMI-SDA: now also U5.SDA1, U6.SDA1, U7.SDA1, U8.SDA1; no longer S74.4
- net PC1HDMI-TMDS1+: now also U5.D1+_1, U6.D1+_1, U7.D1+_1, U8.D1+_1; no longer S64.4
- net PC1HDMI-TMDS1-: now also U5.D1-_1, U6.D1-_1, U7.D1-_1, U8.D1-_1; no longer S66.4
- net PC1HDMI-TMDSC+: now also U5.CLK+_1, U6.CLK+_1, U7.CLK+_1, U8.CLK+_1; no longer S70.4
- net PC1HDMI-TMDSC-: now also U5.CLK-_1, U6.CLK-_1, U7.CLK-_1, U8.CLK-_1; no longer S78.4
- net PC1HDMI-TMDSD0+: now also U5.D0+_1, U6.D0+_1, U7.D0+_1, U8.D0+_1; no longer S67.4
- net PC1HDMI-TMDSD0-: now also U5.D0-_1, U6.D0-_1, U7.D0-_1, U8.D0-_1; no longer S69.4
- net PC1HDMI-TMDSD2+: now also U5.D2+_1, U6.D2+_1, U7.D2+_1, U8.D2+_1; no longer S61.4
- net PC1HDMI-TMDSD2-: now also U5.D2-_1, U6.D2-_1, U7.D2-_1, U8.D2-_1; no longer S63.4
- net PC2HDMI-HOT: now also U5.HPD2, U6.HPD2, U7.HPD2, U8.HPD2; no longer S71.2
- net PC2HDMI-SCL: now also U5.SCL3, U6.SCL3, U7.SCL3, U8.SCL3; no longer S75.2
- net PC2HDMI-SDA: now also U5.SDA2, U6.SDA2, U7.SDA2, U8.SDA2; no longer S74.2
- net PC2HDMI-TMDS1+: now also U5.D1+_2, U6.D1+_2, U7.D1+_2, U8.D1+_2; no longer S64.2
- net PC2HDMI-TMDS1-: now also U5.D1-_2, U6.D1-_2, U7.D1-_2, U8.D1-_2; no longer S66.2
- net PC2HDMI-TMDSC+: now also U5.CLK+_2, U6.CLK+_2, U7.CLK+_2, U8.CLK+_2; no longer S70.2
- net PC2HDMI-TMDSC-: now also U5.CLK-_2, U6.CLK-_2, U7.CLK-_2, U8.CLK-_2; no longer S78.2
- net PC2HDMI-TMDSD0+: now also U5.D0+_2, U6.D0+_2, U7.D0+_2, U8.D0+_2; no longer S67.2
- net PC2HDMI-TMDSD0-: now also U5.D0-_2, U6.D0-_2, U7.D0-_2, U8.D0-_2; no longer S69.2
- net PC2HDMI-TMDSD2+: now also U5.D2+_2, U6.D2+_2, U7.D2+_2, U8.D2+_2; no longer S61.2
- net PC2HDMI-TMDSD2-: now also U5.D2-_2, U6.D2-_2, U7.D2-_2, U8.D2-_2; no longer S63.2
- net PC3HDMI-HOT: now also U5.HPD3, U6.HPD3, U7.HPD3, U8.HPD3; no longer S71.1
- net PC3HDMI-SCL: now also U5.SCL2, U6.SCL2, U7.SCL2, U8.SCL2; no longer S75.1
- net PC3HDMI-SDA: now also U5.SDA3, U6.SDA3, U7.SDA3, U8.SDA3; no longer S74.1
- net PC3HDMI-TMDS1+: now also U5.D1+_3, U6.D1+_3, U7.D1+_3, U8.D1+_3; no longer S64.1
- net PC3HDMI-TMDS1-: now also U5.D1-_3, U6.D1-_3, U7.D1-_3, U8.D1-_3; no longer S66.1
- net PC3HDMI-TMDSC+: now also U5.CLK+_3, U6.CLK+_3, U7.CLK+_3, U8.CLK+_3; no longer S70.1
- net PC3HDMI-TMDSC-: now also U5.CLK-_3, U6.CLK-_3, U7.CLK-_3, U8.CLK-_3; no longer S78.1
- net PC3HDMI-TMDSD0+: now also U5.D0+_3, U6.D0+_3, U7.D0+_3, U8.D0+_3; no longer S67.1
- net PC3HDMI-TMDSD0-: now also U5.D0-_3, U6.D0-_3, U7.D0-_3, U8.D0-_3; no longer S69.1
- net PC3HDMI-TMDSD2+: now also U5.D2+_3, U6.D2+_3, U7.D2+_3, U8.D2+_3; no longer S61.1
- net PC3HDMI-TMDSD2-: now also U5.D2-_3, U6.D2-_3, U7.D2-_3, U8.D2-_3; no longer S63.1
Other:
- note added: "HDMI"
- note added: "USB A"
- moved on the sheet: J2G$1, J5G$1, J5SHIELD, U5

Commit message: m
,
Parts:
- added S17: (no value), SparkFun-Switches:SWITCH-SP3T-SMD
- added U$10, U$11, U$12, U$13, U$14, U$15, U$16, U$17, U$18, U$6, U$7, U$8, U$9: RJ45-8PTH, SparkFun:RJ45-8PTH
- added U21, U22: MAX4998ETIT, MAX4998ETIT:MAX4998ETIT
Connections:
- new net ETH1: U$10.1, U$11.1, U$12.1, U$13.1, U$14.1, U$15.1, U$16.1, U$17.1, U$18.1, U$6.1, U$7.1, U$8.1, U$9.1
- new net ETH2: U$10.2, U$11.2, U$12.2, U$13.2, U$14.2, U$15.2, U$16.2, U$17.2, U$18.2, U$6.2, U$7.2, U$8.2, U$9.2
- new net ETH3: U$10.3, U$11.3, U$12.3, U$13.3, U$14.3, U$15.3, U$16.3, U$17.3, U$18.3, U$6.3, U$7.3, U$8.3, U$9.3
- new net ETH4: U$10.4, U$11.4, U$12.4, U$13.4, U$14.4, U$15.4, U$16.4, U$17.4, U$18.4, U$6.4, U$7.4, U$8.4, U$9.4
- new net ETH5: U$10.5, U$11.5, U$12.5, U$13.5, U$14.5, U$15.5, U$16.5, U$17.5, U$18.5, U$6.5, U$7.5, U$8.5, U$9.5
- new net ETH6: U$10.6, U$11.6, U$12.6, U$13.6, U$14.6, U$15.6, U$16.6, U$17.6, U$18.6, U$6.6, U$7.6, U$8.6, U$9.6
- new net ETH7: U$10.7, U$11.7, U$12.7, U$13.7, U$14.7, U$15.7, U$16.7, U$17.7, U$18.7, U$6.7, U$7.7, U$8.7, U$9.7
- new net ETH8: U$10.8, U$11.8, U$12.8, U$13.8, U$14.8, U$15.8, U$16.8, U$17.8, U$18.8, U$6.8, U$7.8, U$8.8, U$9.8
- net HDMIGND: now also J1SHIELD.SHIELD
Other:
- note added: "ETHERNET"
- moved on the sheet: J1G$1, J1SHIELD, J6, J7

Commit message: sd
asdsa
Connections:
- new net N$130: J7.1, U22.COM0+
- new net N$131: J7.3, U22.COM0-
Other:
- moved on the sheet: J7, S17, U22
Changed lines of the file:
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@@
 <layer number="59" name="tCarbon" color="7" fill="1" visible="no" active="no"/>
 <layer number="60" name="bCarbon" color="7" fill="1" visible="no" active="no"/>
-<layer number="88" name="SimResults" color="9" fill="1" visible="yes" active="yes"/>
+<layer number="88" name="SimResults" color="9" fill="1" visible="no" active="yes"/>
 <layer number="89" name="SimProbes" color="9" fill="1" visible="yes" active="yes"/>
 <layer number="90" name="Modules" color="5" fill="1" visible="yes" active="yes"/>
@@
 <instance part="D12" gate="G$1" x="-431.8" y="190.5" rot="R270"/>
 <instance part="J6" gate="G$1" x="-601.98" y="231.14"/>
-<instance part="J7" gate="G$1" x="-213.36" y="-119.38"/>
+<instance part="J7" gate="G$1" x="-218.44" y="-91.44" rot="R180"/>
 <instance part="U$6" gate="G$1" x="-601.98" y="287.02"/>
 <instance part="U$11" gate="G$1" x="-317.5" y="127"/>
@@
 <instance part="U$18" gate="G$1" x="-424.18" y="30.48"/>
 <instance part="U21" gate="A" x="-368.3" y="-129.54"/>
-<instance part="U22" gate="A" x="-368.3" y="-73.66"/>
-<instance part="S17" gate="G$1" x="-289.56" y="-119.38" rot="R180"/>
+<instance part="U22" gate="A" x="-231.14" y="-119.38" rot="R180"/>
+<instance part="S17" gate="G$1" x="-340.36" y="-111.76" rot="R180"/>
 </instances>
 <busses>
@@
 </segment>
 </net>
+<net name="N$130" class="0">
+<segment>
+<pinref part="U22" gate="A" pin="COM0+"/>
+<pinref part="J7" gate="G$1" pin="1"/>
+<wire x1="-231.14" y1="-119.38" x2="-208.28" y2="-119.38" width="0.1524" layer="91"/>
+</segment>
+</net>
+<net name="N$131" class="0">
+<segment>
+<pinref part="J7" gate="G$1" pin="3"/>
+<wire x1="-208.28" y1="-114.3" x2="-226.06" y2="-114.3" width="0.1524" layer="91"/>
+<wire x1="-226.06" y1="-114.3" x2="-226.06" y2="-116.84" width="0.1524" layer="91"/>
+<pinref part="U22" gate="A" pin="COM0-"/>
+<wire x1="-226.06" y1="-116.84" x2="-231.14" y2="-116.84" width="0.1524" layer="91"/>
+</segment>
+</net>

Commit message: s
s
Parts:
- removed U$10, U$11, U$12, U$13, U$14, U$15, U$16, U$17, U$18, U$7, U$8, U$9: RJ45-8PTH, SparkFun:RJ45-8PTH
- added J10, J8, J9: 2040210-1, 2040210-1:2040210-1
- added J11, J12: AUDIO_JACK_TRRSSMD_RA, SparkFun-Connectors:AUDIO_JACK_TRRSSMD_RA
- added S18, S19, S20: (no value), SparkFun-Switches:SWITCH-SP3T-SMD
- added U$19, U$20, U$21, U$22, U$23, U$24, U$25, U$26, U$27, U$28, U$29, U$30: RJ45-8PTH, SparkFun:RJ45-8PTH
- added U23, U24, U25, U26, U27, U28: SN74CBT16214DGGR, SN74CBT16214DGGR:SN74CBT16214DGGR
- U21, U22: value MAX4998ETIT -> SN74CBT16214DGGR; device MAX4998ETIT:MAX4998ETIT -> SN74CBT16214DGGR:SN74CBT16214DGGR
Connections:
- new net B$1: U21.10A, U23.10A, U25.10A, U27.10A
- new net B$2: U21.11A, U23.11A, U25.11A, U27.11A
- new net N$143: J7.3, U21.3A
- new net N$144: J7.4, U21.4A
- new net N$145: J7.5, U21.5A
- new net N$146: J7.6, U21.6A
- new net N$147: J7.7, U21.7A
- new net N$148: J7.8, U21.8A
- new net N$149: J7.9, U21.9A
- new net N$150: J7.10
- new net N$151: J7.11
- new net N$152: J7.12, U21.12A
- new net N$153: J7.13, U22.1A
- new net N$154: J7.14, U22.2A
- new net N$155: J7.15, U22.3A
- new net N$156: J7.16, U22.4A
- new net N$157: J7.17, U22.5A
- new net N$158: J7.18, U22.6A
- new net N$159: J7.19, U22.7A
- new net N$160: J7.SHIELD, U22.9A
- new net N$161: J8.1, U23.1A
- new net N$162: J8.2, U23.2A
- new net N$163: J7.20, U22.8A
- new net N$164: J8.3, U23.3A
- new net N$165: J8.4, U23.4A
- new net N$166: J8.5, U23.5A
- new net N$167: J8.6, U23.6A
- new net N$168: J8.7, U23.7A
- new net N$169: J8.8, U23.8A
- new net N$170: J8.9, U23.9A
- new net N$171: J8.10
- new net N$172: J8.11
- new net N$173: J8.12, U23.12A
- new net N$174: J8.13, U24.1A
- new net N$175: J8.14, U24.2A
- new net N$176: J8.15, U24.3A
- new net N$177: J8.16, U24.4A
- new net N$178: J8.17, U24.5A
- new net N$179: J8.18, U24.6A
- new net N$180: J8.19, U24.7A
- new net N$181: J8.SHIELD, U24.9A
- new net N$182: J8.20, U24.8A
- new net N$183: J9.1, U25.1A
- new net N$184: J9.2, U25.2A
- new net N$185: J9.3, U25.3A
- new net N$186: J9.4, U25.4A
- new net N$187: J9.5, U25.5A
- new net N$188: J9.6, U25.6A
- new net N$189: J9.7, U25.7A
- new net N$190: J9.8, U25.8A
- new net N$191: J9.9, U25.9A
- new net N$192: J9.10
- new net N$193: J9.11
- new net N$194: J9.12, U25.12A
- new net N$195: J9.13, U26.1A
- new net N$196: J9.14, U26.2A
- new net N$197: J9.15, U26.3A
- new net N$198: J9.16, U26.4A
- new net N$199: J9.17, U26.5A
- new net N$200: J9.18, U26.6A
- new net N$201: J9.19, U26.7A
- new net N$202: J9.SHIELD, U26.9A
- new net N$203: J9.20, U26.8A
- new net N$204: J10.1, U27.1A
- new net N$205: J10.2, U27.2A
- new net N$206: J10.3, U27.3A
- new net N$207: J10.4, U27.4A
- new net N$208: J10.5, U27.5A
- new net N$209: J10.6, U27.6A
- new net N$210: J10.7, U27.7A
- new net N$211: J10.8, U27.8A
- new net N$212: J10.9, U27.9A
- new net N$213: J10.10
- new net N$214: J10.11
- new net N$215: J10.12, U27.12A
- new net N$216: J10.13, U28.1A
- new net N$217: J10.14, U28.2A
- new net N$218: J10.15, U28.3A
- new net N$219: J10.16, U28.4A
- new net N$220: J10.17, U28.5A
- new net N$221: J10.18, U28.6A
- new net N$222: J10.19, U28.7A
- new net N$223: J10.SHIELD, U28.9A
- new net N$224: J10.20, U28.8A
- new net PC1A1: J11.RING2, J12.RING2
- new net PC1A2: J11.TIP, J12.TIP
- new net PC1A3: J11.RING1, J12.RING1
- new net PC1A4: J11.EARTH, J12.EARTH
- new net PC1DP1: J6.1, U21.1B1, U23.1B1, U25.1B1, U27.1B1
- new net PC1DP10: J6.10, U21.10B1, U23.10B1, U25.10B1, U27.10B1
- new net PC1DP11: J6.11, U21.11B1, U23.11B1, U25.11B1, U27.11B1
- new net PC1DP12: J6.12, U21.12B1, U23.12B1, U25.12B1, U27.12B1
- new net PC1DP13: J6.13, U22.1B1, U24.1B1, U26.1B1, U28.1B1
- new net PC1DP14: J6.14, U22.2B1, U24.2B1, U26.2B1, U28.2B1
- new net PC1DP15: J6.15, U22.3B1, U24.3B1, U26.3B1, U28.3B1
- new net PC1DP16: J6.16, U22.4B1, U24.4B1, U26.4B1, U28.4B1
- new net PC1DP17: J6.17, U22.5B1, U24.5B1, U26.5B1, U28.5B1
- new net PC1DP18: J6.18, U22.6B1, U24.6B1, U26.6B1, U28.6B1
- new net PC1DP19: J6.19, U22.7B1, U24.7B1, U26.7B1, U28.7B1
- new net PC1DP2: J6.2, U21.2B1, U23.2B1, U25.2B1, U27.2B1
- new net PC1DP20: J6.20, U22.8B1, U24.8B1, U26.8B1, U28.8B1
- new net PC1DP3: J6.3, U21.3B1, U23.3B1, U25.3B1, U27.3B1
- new net PC1DP4: J6.4, U21.4B1, U23.4B1, U25.4B1, U27.4B1
- new net PC1DP5: J6.5, U21.5B1, U23.5B1, U25.5B1, U27.5B1
- new net PC1DP6: J6.6, U21.6B1, U23.6B1, U25.6B1, U27.6B1
- new net PC1DP7: J6.7, U21.7B1, U23.7B1, U25.7B1, U27.7B1
- new net PC1DP8: J6.8, U21.8B1, U23.8B1, U25.8B1, U27.8B1
- new net PC1DP9: J6.9, U21.9B1, U23.9B1, U25.9B1, U27.9B1
- new net PC1DPS: J6.SHIELD, U22.9B1, U24.9B1, U26.9B1, U28.9B1
- new net PC2DP1: U21.1B2, U23.1B2, U25.1B2, U27.1B2
- new net PC2DP10: U21.10B2, U23.10B2, U25.10B2, U27.10B2
- new net PC2DP11: U21.11B2, U23.11B2, U25.11B2, U27.11B2
- new net PC2DP12: U21.12B2, U23.12B2, U25.12B2, U27.12B2
- new net PC2DP13: U22.1B2, U24.1B2, U26.1B2, U28.1B2
- new net PC2DP14: U22.2B2, U24.2B2, U26.2B2, U28.2B2
- new net PC2DP15: U22.3B2, U24.3B2, U26.3B2, U28.3B2
- new net PC2DP16: U22.4B2, U24.4B2, U26.4B2, U28.4B2
- new net PC2DP17: U22.5B2, U24.5B2, U26.5B2, U28.5B2
- new net PC2DP18: U22.6B2, U24.6B2, U26.6B2, U28.6B2
- new net PC2DP19: U22.7B2, U24.7B2, U26.7B2, U28.7B2
- new net PC2DP2: U21.2B2, U23.2B2, U25.2B2, U27.2B2
- new net PC2DP20: U22.8B2, U24.8B2, U26.8B2, U28.8B2
- new net PC2DP3: U21.3B2, U23.3B2, U25.3B2, U27.3B2
- new net PC2DP4: U21.4B2, U23.4B2, U25.4B2, U27.4B2
- new net PC2DP5: U21.5B2, U23.5B2, U25.5B2, U27.5B2
- new net PC2DP6: U21.6B2, U23.6B2, U25.6B2, U27.6B2
- new net PC2DP7: U21.7B2, U23.7B2, U25.7B2, U27.7B2
- new net PC2DP8: U21.8B2, U23.8B2, U25.8B2, U27.8B2
- new net PC2DP9: U21.9B2, U23.9B2, U25.9B2, U27.9B2
- new net PC2DPS: U22.9B2, U24.9B2, U26.9B2, U28.9B2
- new net PC3DP1: U21.1B3, U23.1B3, U25.1B3, U27.1B3
- new net PC3DP10: U21.10B3, U23.10B3, U25.10B3, U27.10B3
- new net PC3DP11: U21.11B3, U23.11B3, U25.11B3, U27.11B3
- new net PC3DP12: U21.12B3, U23.12B3, U25.12B3, U27.12B3
- new net PC3DP13: U22.1B3, U24.1B3, U26.1B3, U28.1B3
- new net PC3DP14: U22.2B3, U24.2B3, U26.2B3, U28.2B3
- new net PC3DP15: U22.3B3, U24.3B3, U26.3B3, U28.3B3
- new net PC3DP16: U22.4B3, U24.4B3, U26.4B3, U28.4B3
- new net PC3DP17: U22.5B3, U24.5B3, U26.5B3, U28.5B3
- new net PC3DP18: U22.6B3, U24.6B3, U26.6B3, U28.6B3
- new net PC3DP19: U22.7B3, U24.7B3, U26.7B3, U28.7B3
- new net PC3DP2: U21.2B3, U23.2B3, U25.2B3, U27.2B3
- new net PC3DP20: U22.8B3, U24.8B3, U26.8B3, U28.8B3
- new net PC3DP3: U21.3B3, U23.3B3, U25.3B3, U27.3B3
- new net PC3DP4: U21.4B3, U23.4B3, U25.4B3, U27.4B3
- new net PC3DP5: U21.5B3, U23.5B3, U25.5B3, U27.5B3
- new net PC3DP6: U21.6B3, U23.6B3, U25.6B3, U27.6B3
- new net PC3DP7: U21.7B3, U23.7B3, U25.7B3, U27.7B3
- new net PC3DP8: U21.8B3, U23.8B3, U25.8B3, U27.8B3
- new net PC3DP9: U21.9B3, U23.9B3, U25.9B3, U27.9B3
- new net PC3DPS: U22.9B3, U24.9B3, U26.9B3, U28.9B3
- net ETH1: now also U$19.1, U$20.1, U$21.1, U$22.1, U$23.1, U$24.1, U$25.1, U$26.1, U$27.1, U$28.1, U$29.1, U$30.1; no longer U$10.1, U$11.1, U$12.1, U$13.1, U$14.1, U$15.1, U$16.1, U$17.1, U$18.1, U$7.1, U$8.1, U$9.1
- net ETH2: now also U$19.2, U$20.2, U$21.2, U$22.2, U$23.2, U$24.2, U$25.2, U$26.2, U$27.2, U$28.2, U$29.2, U$30.2; no longer U$10.2, U$11.2, U$12.2, U$13.2, U$14.2, U$15.2, U$16.2, U$17.2, U$18.2, U$7.2, U$8.2, U$9.2
- net ETH3: now also U$19.3, U$20.3, U$21.3, U$22.3, U$23.3, U$24.3, U$25.3, U$26.3, U$27.3, U$28.3, U$29.3, U$30.3; no longer U$10.3, U$11.3, U$12.3, U$13.3, U$14.3, U$15.3, U$16.3, U$17.3, U$18.3, U$7.3, U$8.3, U$9.3
- net ETH4: now also U$19.4, U$20.4, U$21.4, U$22.4, U$23.4, U$24.4, U$25.4, U$26.4, U$27.4, U$28.4, U$29.4, U$30.4; no longer U$10.4, U$11.4, U$12.4, U$13.4, U$14.4, U$15.4, U$16.4, U$17.4, U$18.4, U$7.4, U$8.4, U$9.4
- net ETH5: now also U$19.5, U$20.5, U$21.5, U$22.5, U$23.5, U$24.5, U$25.5, U$26.5, U$27.5, U$28.5, U$29.5, U$30.5; no longer U$10.5, U$11.5, U$12.5, U$13.5, U$14.5, U$15.5, U$16.5, U$17.5, U$18.5, U$7.5, U$8.5, U$9.5
- net ETH6: now also U$19.6, U$20.6, U$21.6, U$22.6, U$23.6, U$24.6, U$25.6, U$26.6, U$27.6, U$28.6, U$29.6, U$30.6; no longer U$10.6, U$11.6, U$12.6, U$13.6, U$14.6, U$15.6, U$16.6, U$17.6, U$18.6, U$7.6, U$8.6, U$9.6
- net ETH7: now also U$19.7, U$20.7, U$21.7, U$22.7, U$23.7, U$24.7, U$25.7, U$26.7, U$27.7, U$28.7, U$29.7, U$30.7; no longer U$10.7, U$11.7, U$12.7, U$13.7, U$14.7, U$15.7, U$16.7, U$17.7, U$18.7, U$7.7, U$8.7, U$9.7
- net ETH8: now also U$19.8, U$20.8, U$21.8, U$22.8, U$23.8, U$24.8, U$25.8, U$26.8, U$27.8, U$28.8, U$29.8, U$30.8; no longer U$10.8, U$11.8, U$12.8, U$13.8, U$14.8, U$15.8, U$16.8, U$17.8, U$18.8, U$7.8, U$8.8, U$9.8
- net N$130: now also U21.1A; no longer U22.COM0+
- net N$131: now also J7.2, U21.2A; no longer J7.3, U22.COM0-
Other:
- note added: "DP"
- moved on the sheet: J1G$1, J1SHIELD, J6, J7, S17, U$6
