File: projects/Modular Microcontroller/Arduino_MEGA_2560-Rev3.brd (EAGLE design)
At the start: 46 x 45.5 mm, 52 parts, among them IC1 NCP1117ST50T3G, IC3 ATMEGA2560-16AU, IC4 ATMEGA16U2-MU, IC6 LP2985-33DBVR, IC7 LMV358IDGKR, J1 1-2199119-3, T1 FDN340P, X1 POWERSUPPLY_DC21MMX, Y1 CSTCE16M0V53-R0 16MHZ, Y2 16MHz

Commit message: a
s
Parts:
- moved X1 5.69 mm to (40.8, 49.6), turned to 0 degrees
- moved D1 5.50 mm to (42.7, 36.1)
Routing:
- net VIN: track 49.8 -> 44.3 mm
Other:
- board text removed: "0"
- board text removed: "1"
- board text removed: "11"
- board text removed: "12"
- board text removed: "13"
- board text removed: "14"
- board text removed: "15"
- board text removed: "16"
- board text removed: "17"
- board text removed: "18"
- board text removed: "19"
- board text removed: "2"
- board text removed: "20"
- board text removed: "21"
- board text removed: "22"
- board text removed: "24"
- board text removed: "26"
- board text removed: "28"
- board text removed: "3"
- board text removed: "30"
- board text removed: "31"
- board text removed: "32"
- board text removed: "33"
- board text removed: "34"
- board text removed: "35"
- board text removed: "36"
- board text removed: "37"
- board text removed: "38"
- board text removed: "39"
- board text removed: "4"
- board text removed: "40"
- board text removed: "41"
- board text removed: "42"
- board text removed: "43"
- board text removed: "44"
- board text removed: "45"
- board text removed: "46"
- board text removed: "47"
- board text removed: "48"
- board text removed: "49"
- board text removed: "5"
- board text removed: "50"
- board text removed: "51"
- board text removed: "52"
- board text removed: "53"
- board text removed: "6"
- board text removed: "8"
- board text removed: "ANALOG IN"
- board text removed: "AREF"
- board text removed: "Arduino"
- board text removed: "DIGITAL"
- board text removed: "MEGA 2560"
- board text removed: "RX"
- board text removed: "RX1"
- board text removed: "RX2"
- board text removed: "RX3"
- board text removed: "SCL"
- board text removed: "SDA"
- board text removed: "TM"
- board text removed: "TX"
- board text removed: "TX1"
- board text removed: "TX2"
- board text removed: "TX3"
- board text removed: "designed by"
- board text removed: "tinker it"
- board text removed: "www.arduino.cc"
