File: projects/Soccerbot/V4/soccerbot.brd (EAGLE design)
At the start: 149.8 x 101.3 mm, 89 parts, among them CN2 1X4-CLEANBIG, IC1 LM340S-05, IC2 TB6612FNG, IC4 TB6612FNG, J3 1X5, J4 1X5, Q1 AOD417, SW2 SPST_TACT-EVQQ2, U1 PCA9685, X1 NXT-SOCKET, X2 NXT-SOCKET, X3 NXT-SOCKET, X4 NXT-SOCKET

Commit message: fghjk
 vb
Parts:
- removed C1: (no value), rcl:C0805
- removed C11, C7, C8: 0.1uF, microbuilder:0805-NO
- removed C12: 47uF/16v, microbuilder:PANASONIC_C
- removed C13: 47uF+/16v, microbuilder:PANASONIC_C
- removed C15, C16: 10uF, microbuilder:0805-NO
- removed CN2: 1X4-CLEANBIG, adafruit:1X04-CLEANBIG
- removed D0-1, JP6: (no value), adafruit:1X08-CLEANBIG
- removed D1, D2, D3, D4: GREEN, SparkFun-LED:LED-0603
- removed IC2, IC4: TB6612FNG, adafruit:SSOP24
- removed J3, J4: 1X5, adafruit:1X05-3.5MM
- removed JP5: (no value), microbuilder:1X04_ROUND_76
- removed JP7: (no value), microbuilder:1X10_ROUND70
- removed JP8: (no value), microbuilder:1X02_ROUND
- removed LED2: Green, microbuilder:CHIPLED_0805_NOOUTLINE
- removed R15, R16, R17, R19, R20: 10k, microbuilder:0805-NO
- removed R21, R22: 10K, microbuilder:0805-NO
- removed R7: 150ohm, rcl:R0603
- removed SERVO3, SERVO4: (no value), adafruit:1X03
- removed SW2: SPST_TACT-EVQQ2, adafruit:EVQ-Q2
- removed U1: PCA9685, microbuilder:TSSOP28
- added U2, U3, U4, U5: DRV8871DDAR, DRV8871DDAR:SOIC127P600X170-8N
Connections:
- removed net A0: R15.2, U1.1
- removed net A1: R16.2, U1.2
- removed net A2: R17.2, U1.3
- removed net A3: R19.2, U1.4
- removed net A4: R20.2, U1.5
- removed net IOREF1: JP6.7
- removed net M1A1: IC2.1, IC2.2, J3.5
- removed net M1B1: D2.A, IC2.5, IC2.6
- removed net M2A1: D1.C, J3.1
- removed net M2B1: IC2.7, IC2.8, J3.2
- removed net M3A1: IC4.1, IC4.2, J4.1
- removed net M3B1: D4.A, IC4.5, IC4.6
- removed net M4A1: D3.C, J4.5
- removed net M4B1: IC4.7, IC4.8, J4.4
- removed net N$14: D1.A, IC2.11, IC2.12
- removed net PWM0: JP5.1, U1.6
- removed net PWM1: JP5.2, U1.7
- removed net PWM10: IC2.21, U1.17
- removed net PWM11: IC2.17, U1.18
- removed net PWM12: IC2.16, U1.19
- removed net PWM13: IC2.15, U1.20
- removed net PWM14: JP5.3, U1.21
- removed net PWM15: JP5.4, U1.22
- removed net PWM2: IC4.23, U1.8
- removed net PWM3: IC4.22, U1.9
- removed net PWM4: IC4.21, U1.10
- removed net PWM5: IC4.17, U1.11
- removed net PWM6: IC4.16, U1.12
- removed net PWM7: IC4.15, U1.13
- removed net PWM8: IC2.23, U1.15
- removed net PWM9: IC2.22, U1.16
- new net PAD: U2.9, U3.9, U4.9, U5.9
- new net PGND: U2.7, U3.7, U4.7, U5.7
- net 3.3V: no longer JP6.5
- net 5.5V: no longer C11.1, C15.1, C16.1, C7.1, C8.1, IC2.19, IC2.20, IC4.19, IC4.20, JP6.4, LED2.A, R21.2, R22.2, U1.24, U1.28
- net A0A: no longer CN2.4
- net A1A: no longer CN2.3
- net A2A: no longer CN2.2
- net A3A: no longer CN2.1
- net AREF: no longer JP7.3
- net BAT+: no longer C12.+, C13.+, IC2.13, IC2.14, IC2.24, IC4.13, IC4.14, IC4.24, JP6.1
- net D0: no longer D0-1.1
- net D1: no longer D0-1.2
- net D10: no longer JP7.8, SERVO3.3
- net D11: no longer JP7.7
- net D12: no longer JP7.6
- net D13: no longer JP7.5
- net D2: no longer D0-1.3
- net D3: no longer D0-1.4
- net D4: no longer D0-1.5
- net D5: no longer D0-1.6
- net D6: no longer D0-1.7
- net D7: no longer D0-1.8
- net D8: no longer JP7.10
- net D9: no longer JP7.9, SERVO4.3
- net GND: now also U2.1, U3.1, U4.1, U5.1; no longer C1.2, C11.2, C12.-, C13.-, C15.2, C16.2, C7.2, C8.2, IC2.10, IC2.18, IC2.3, IC2.4, IC2.9, IC4.10, IC4.18, IC4.3, IC4.4, IC4.9, J3.3, J4.3, JP6.2, JP6.3, JP7.4, R15.1, R16.1, R17.1, R19.1, R20.1, R7.1, SERVO3.1, SERVO4.1, SW2.A, SW2.A', U1.14, U1.23, U1.25
- net N$1: now also U2.5, U3.5, U4.5, U5.5; no longer LED2.C, R7.2
- net N$13: now also U3.8; no longer D2.C, J3.4
- net N$15: now also U2.6; no longer D4.C, J4.2
- net N$16: now also U2.8; no longer D3.A, IC4.11, IC4.12
- net N$3: now also U3.6; no longer JP6.8
- net RESET: no longer JP6.6, SW2.B, SW2.B'
- net SCL: no longer JP7.1, JP8.1, R22.1, U1.26
- net SDA: no longer JP7.2, JP8.2, R21.1, U1.27
- net SERVO5V: no longer C1.1, SERVO3.2, SERVO4.2
Routing:
- net BAT+: track 503.2 -> 405.6 mm, vias 13 -> 8
- net GND: track 168.4 -> 96.8 mm, vias 31 -> 25
- net RESET: track 51.7 -> 0.00 mm, vias 1 -> 0
- net 5.5V: track 854.7 -> 806.2 mm
- net PWM15: track 42.8 -> 0.00 mm, vias 1 -> 0
- net PWM14: track 41.4 -> 0.00 mm, vias 2 -> 0
- net PWM1: track 38.1 -> 0.00 mm, vias 1 -> 0
- net M4B1: track 32.2 -> 0.00 mm, vias 1 -> 0
- net PWM12: track 31.9 -> 0.00 mm
- net PWM0: track 29.0 -> 0.00 mm, vias 1 -> 0
- net M3A1: track 27.4 -> 0.00 mm, vias 1 -> 0
- net M4A1: track 24.8 -> 0.00 mm, vias 1 -> 0
- net PWM4: track 24.7 -> 0.00 mm, vias 2 -> 0
- net PWM6: track 23.6 -> 0.00 mm, vias 2 -> 0
- net PWM7: track 22.7 -> 0.00 mm
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