File: projects/Soccerbot/V4/soccerbot.sch (EAGLE design)
At the start: 87 parts, among them CN2 1X4-CLEANBIG, IC1 LM340S-05, IC2 TB6612FNG, IC4 TB6612FNG, J3 1X5, J4 1X5, Q1 AOD417, SW2 SPST_TACT-EVQQ2, U1 PCA9685, X1 NXT-SOCKET, X2 NXT-SOCKET, X3 NXT-SOCKET, X4 NXT-SOCKET

Commit message: fghjk
 vb
Parts:
- removed C1: (no value), rcl:C-USC0805
- removed C11, C7, C8: 0.1uF, microbuilder:CAP_CERAMIC0805-NOOUTLINE
- removed C12: 47uF/16v, microbuilder:CAP_ELECTROLYTICPANASONIC_C
- removed C13: 47uF+/16v, microbuilder:CAP_ELECTROLYTICPANASONIC_C
- removed C15, C16: 10uF, microbuilder:CAP_CERAMIC0805-NOOUTLINE
- removed CN2: 1X4-CLEANBIG, adafruit:1X4-CLEANBIG
- removed D0-1, JP6: (no value), adafruit:PINHD-1X8CLEANBIG
- removed D1, D2, D3, D4: GREEN, SparkFun-LED:LED-GREEN0603
- removed IC2, IC4: TB6612FNG, adafruit:TB6612FNG
- removed J3, J4: 1X5, adafruit:1X5
- removed JP5: (no value), microbuilder:HEADER-1X476MIL
- removed JP7: (no value), microbuilder:HEADER-1X1070MIL
- removed JP8: (no value), microbuilder:HEADER-1X2ROUND
- removed LED2: Green, microbuilder:LED0805_NOOUTLINE
- removed R15, R16, R17, R19, R20: 10k, microbuilder:RESISTOR0805_NOOUTLINE
- removed R21, R22: 10K, microbuilder:RESISTOR0805_NOOUTLINE
- removed R7: 150ohm, rcl:R-US_R0603
- removed SERVO3, SERVO4: (no value), adafruit:PINHD-1X3
- removed SW2: SPST_TACT-EVQQ2, adafruit:SPST_TACT-EVQQ2
- removed U1: PCA9685, microbuilder:PCA9685
- added U2, U3, U4, U5: DRV8871DDAR, DRV8871DDAR:DRV8871DDAR
Connections:
- removed net A0: R15.2, U1.A0
- removed net A1: R16.2, U1.A1
- removed net A2: R17.2, U1.A2
- removed net A3: R19.2, U1.A3
- removed net A4: R20.2, U1.A4
- removed net IOREF1: JP6.7
- removed net M1A1: IC2.AO1, IC2.AO1', J3.5
- removed net M1B1: D2.A, IC2.AO2, IC2.AO2'
- removed net M2A1: D1.C, J3.1
- removed net M2B1: IC2.BO2, IC2.BO2', J3.2
- removed net M3A1: IC4.AO1, IC4.AO1', J4.1
- removed net M3B1: D4.A, IC4.AO2, IC4.AO2'
- removed net M4A1: D3.C, J4.5
- removed net M4B1: IC4.BO2, IC4.BO2', J4.4
- removed net N$14: D1.A, IC2.BO1, IC2.BO1'
- removed net PWM0: JP5.1, U1.PWM0
- removed net PWM1: JP5.2, U1.PWM1
- removed net PWM10: IC2.AIN1, U1.PWM10
- removed net PWM11: IC2.BIN1, U1.PWM11
- removed net PWM12: IC2.BIN2, U1.PWM12
- removed net PWM13: IC2.PWMB, U1.PWM13
- removed net PWM14: JP5.3, U1.PWM14
- removed net PWM15: JP5.4, U1.PWM15
- removed net PWM2: IC4.PWMA, U1.PWM2
- removed net PWM3: IC4.AIN2, U1.PWM3
- removed net PWM4: IC4.AIN1, U1.PWM4
- removed net PWM5: IC4.BIN1, U1.PWM5
- removed net PWM6: IC4.BIN2, U1.PWM6
- removed net PWM7: IC4.PWMB, U1.PWM7
- removed net PWM8: IC2.PWMA, U1.PWM8
- removed net PWM9: IC2.AIN2, U1.PWM9
- net 3.3V: no longer JP6.5
- net 5.5V: no longer C11.1, C15.1, C16.1, C7.1, C8.1, IC2.STBY, IC2.VCC, IC4.STBY, IC4.VCC, JP6.4, LED2.A, R21.2, R22.2, U1.A5, U1.VDD
- net A0A: no longer CN2.4
- net A1A: no longer CN2.3
- net A2A: no longer CN2.2
- net A3A: no longer CN2.1
- net AREF: no longer JP7.3
- net BAT+: no longer C12.+, C13.+, IC2.VM1, IC2.VM2, IC2.VM3, IC4.VM1, IC4.VM2, IC4.VM3, JP6.1
- net D0: no longer D0-1.1
- net D1: no longer D0-1.2
- net D10: no longer JP7.8, SERVO3.3
- net D11: no longer JP7.7
- net D12: no longer JP7.6
- net D13: no longer JP7.5
- net D2: no longer D0-1.3
- net D3: no longer D0-1.4
- net D4: no longer D0-1.5
- net D5: no longer D0-1.6
- net D6: no longer D0-1.7
- net D7: no longer D0-1.8
- net D8: no longer JP7.10
- net D9: no longer JP7.9, SERVO4.3
- net GND: no longer C1.2, C11.2, C12.-, C13.-, C15.2, C16.2, C7.2, C8.2, IC2.GND, IC2.PGND1, IC2.PGND1', IC2.PGND2, IC2.PGND2', IC4.GND, IC4.PGND1, IC4.PGND1', IC4.PGND2, IC4.PGND2', J3.3, J4.3, JP6.2, JP6.3, JP7.4, R15.1, R16.1, R17.1, R19.1, R20.1, R7.1, SERVO3.1, SERVO4.1, SW2.P, SW2.P1, U1.#OE, U1.EXTCLK, U1.GND
- net N$1: now also U2.VM, U3.VM, U4.VM, U5.VM; no longer LED2.C, R7.2
- net N$13: now also U3.OUT2; no longer D2.C, J3.4
- net N$15: now also U2.OUT1; no longer D4.C, J4.2
- net N$16: now also U2.OUT2; no longer D3.A, IC4.BO1, IC4.BO1'
- net N$3: now also U3.OUT1; no longer JP6.8
- net RESET: no longer JP6.6, SW2.S, SW2.S1
- net SCL: no longer JP7.1, JP8.1, R22.1, U1.SCL
- net SDA: no longer JP7.2, JP8.2, R21.1, U1.SDA
- net SERVO5V: no longer C1.1, SERVO3.2, SERVO4.2
