File: projects/PocketPrinter3d/Motherboard.brd (EAGLE design)
At the start: 36.8 x 61.9 mm, 16 parts, among them Q1 200mA/40V

Commit message: asd
asd
Parts:
- added JP3: (no value), SparkFun:1X04
- added STEPPERPOWER: (no value), SparkFun:1X02
Connections:
- net 5.5V: now also STEPPERPOWER.1
- net A0: now also JP3.1
- net A1: now also JP3.2
- net A2: now also JP3.3
- net A3: now also JP3.4
- net GND: now also STEPPERPOWER.2
Routing:
- net GND: track 168.2 -> 142.7 mm
- net 5.5V: track 37.8 -> 44.0 mm
- net A3: track 3.81 -> 8.89 mm
- net A2: track 3.81 -> 8.89 mm
- net A1: track 3.81 -> 8.89 mm
- net A0: track 3.81 -> 8.89 mm
Changed lines of the file:
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@@
 <attribute name="VALUE" x="5.715" y="104.14" size="1.27" layer="27" rot="R90"/>
+</element>
+<element name="STEPPERPOWER" library="SparkFun" package="1X02" value="" x="0.635" y="80.01" smashed="yes" rot="R270">
+<attribute name="NAME" x="2.4638" y="81.3562" size="1.27" layer="25" ratio="10" rot="R270"/>
+<attribute name="VALUE" x="-2.54" y="81.28" size="1.27" layer="27" rot="R270"/>
+</element>
+<element name="JP3" library="SparkFun" package="1X04" value="" x="0.635" y="97.79" smashed="yes" rot="R270">
+<attribute name="NAME" x="2.4638" y="99.1362" size="1.27" layer="25" ratio="10" rot="R270"/>
+<attribute name="VALUE" x="-2.54" y="99.06" size="1.27" layer="27" rot="R270"/>
 </element>
 </elements>
@@
 <wire x1="2.54" y1="108.1278" x2="2.54" y2="107.315625" width="0.762" layer="1"/>
 <wire x1="2.54" y1="103.148775" x2="2.54" y2="86.995" width="0.762" layer="1"/>
-<wire x1="2.54" y1="86.995" x2="2.54" y2="72.39" width="0.762" layer="1"/>
 <wire x1="2.54" y1="107.315625" x2="4.0132" y2="105.842425" width="0.762" layer="1"/>
 <wire x1="4.0132" y1="104.621975" x2="2.54" y2="103.148775" width="0.762" layer="1"/>
@@
 <wire x1="8.5443625" y1="94.0626" x2="10.6708375" y2="94.0626" width="0.762" layer="16"/>
 <wire x1="2.54" y1="86.995" x2="4.2418" y2="85.2932" width="0.762" layer="16"/>
-<wire x1="4.2418" y1="85.2932" x2="4.2418" y2="74.319775" width="0.762" layer="16"/>
 <via x="11.7475" y="96.2025" extent="1-16" drill="0.35"/>
 <wire x1="16.49841875" y1="100.95341875" x2="11.7475" y2="96.2025" width="0.762" layer="16"/>
@@
 <wire x1="23.495" y1="109.855" x2="24.765" y2="108.585" width="0.762" layer="16"/>
 <via x="24.765" y="108.585" extent="1-16" drill="0.35"/>
+<contactref element="STEPPERPOWER" pad="2"/>
 </signal>
 <signal name="RST">
@@
 <via x="11.8618" y="66.8782" extent="1-16" drill="0.35"/>
 <wire x1="11.5408" y1="77.0728" x2="11.5408" y2="67.1992" width="0.762" layer="16"/>
+<contactref element="STEPPERPOWER" pad="1"/>
+<wire x1="0.635" y1="80.01" x2="3.175" y2="80.01" width="1.27" layer="1"/>
+<wire x1="3.175" y1="80.01" x2="3.9116" y2="79.2734" width="1.27" layer="1"/>
+<wire x1="3.9116" y1="79.2734" x2="3.9116" y2="79.26300625" width="1.27" layer="1"/>
+<wire x1="3.9116" y1="79.26300625" x2="4.96800625" y2="78.2066" width="1.27" layer="1"/>
+<wire x1="4.96800625" y1="78.2066" x2="4.9784" y2="78.2066" width="1.27" layer="1"/>
+<wire x1="4.9784" y1="78.2066" x2="5.715" y2="77.47" width="1.27" layer="1"/>
 </signal>
 <signal name="A7">
@@
 <contactref element="JP4" pad="9"/>
 <wire x1="9.525" y1="90.17" x2="5.715" y2="90.17" width="2.032" layer="1"/>
+<contactref element="JP3" pad="4"/>
+<wire x1="5.715" y1="90.17" x2="0.635" y2="90.17" width="1.27" layer="16"/>
 </signal>
 <signal name="A2">
@@
 <contactref element="JP4" pad="10"/>
 <wire x1="9.525" y1="92.71" x2="5.715" y2="92.71" width="2.032" layer="1"/>
+<contactref element="JP3" pad="3"/>
+<wire x1="0.635" y1="92.71" x2="5.715" y2="92.71" width="1.27" layer="16"/>
 </signal>
 <signal name="A1">
@@
 <contactref element="JP4" pad="11"/>
 <wire x1="5.715" y1="95.25" x2="9.525" y2="95.25" width="2.032" layer="1"/>
+<contactref element="JP3" pad="2"/>
+<wire x1="5.715" y1="95.25" x2="0.635" y2="95.25" width="1.27" layer="16"/>
 </signal>
 <signal name="A0">
@@
 <contactref element="JP4" pad="12"/>
 <wire x1="9.525" y1="97.79" x2="5.715" y2="97.79" width="2.032" layer="1"/>
+<contactref element="JP3" pad="1"/>
+<wire x1="0.635" y1="97.79" x2="5.715" y2="97.79" width="1.27" layer="16"/>
 </signal>
 <signal name="AREF">
