File: projects/PocketPrinter3d/Motherboard.sch (EAGLE design)
At the start: 16 parts, among them Q1 200mA/40V

Commit message: asd
asd
Parts:
- added JP3: (no value), SparkFun:M04PTH
- added STEPPERPOWER: (no value), SparkFun:M02PTH
Connections:
- net 5.5V: now also STEPPERPOWER.1
- net A0: now also JP3.1
- net A1: now also JP3.2
- net A2: now also JP3.3
- net A3: now also JP3.4
- net GND: now also STEPPERPOWER.2
Changed lines of the file:
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@@
 <part name="UBL9V1" library="BaseApp" deviceset="JUMPER" device=""/>
 <part name="UVBL" library="SparkFun" deviceset="M02" device="LOCK"/>
+<part name="STEPPERPOWER" library="SparkFun" deviceset="M02" device="PTH"/>
+<part name="JP3" library="SparkFun" deviceset="M04" device="PTH"/>
 </parts>
 <sheets>
@@
 <attribute name="VALUE" x="53.34" y="-12.7" size="1.778" layer="96" rot="R90"/>
 <attribute name="NAME" x="42.418" y="-12.7" size="1.778" layer="95" rot="R90"/>
+</instance>
+<instance part="STEPPERPOWER" gate="G$1" x="25.4" y="50.8" smashed="yes" rot="R90">
+<attribute name="VALUE" x="30.48" y="48.26" size="1.778" layer="96" rot="R90"/>
+<attribute name="NAME" x="19.558" y="48.26" size="1.778" layer="95" rot="R90"/>
+</instance>
+<instance part="JP3" gate="G$1" x="101.6" y="7.62" smashed="yes" rot="R90">
+<attribute name="VALUE" x="109.22" y="2.54" size="1.778" layer="96" rot="R90"/>
+<attribute name="NAME" x="93.218" y="2.54" size="1.778" layer="95" rot="R90"/>
 </instance>
 </instances>
@@
 <label x="38.1" y="-7.62" size="1.778" layer="95" rot="R90"/>
 </segment>
+<segment>
+<pinref part="STEPPERPOWER" gate="G$1" pin="2"/>
+<wire x1="22.86" y1="58.42" x2="22.86" y2="60.96" width="0.1524" layer="91"/>
+<label x="22.86" y="60.96" size="1.778" layer="95" rot="R90"/>
+</segment>
 </net>
 <net name="RST" class="0">
@@
 <label x="73.66" y="5.08" size="1.778" layer="95"/>
 </segment>
+<segment>
+<pinref part="STEPPERPOWER" gate="G$1" pin="1"/>
+<wire x1="25.4" y1="58.42" x2="25.4" y2="60.96" width="0.1524" layer="91"/>
+<label x="25.4" y="60.96" size="1.778" layer="95" rot="R90"/>
+</segment>
 </net>
 <net name="A7" class="0">
@@
 <junction x="-17.78" y="20.32"/>
 </segment>
+<segment>
+<pinref part="JP3" gate="G$1" pin="4"/>
+<wire x1="96.52" y1="12.7" x2="96.52" y2="15.24" width="0.1524" layer="91"/>
+<label x="96.52" y="15.24" size="1.778" layer="95"/>
+</segment>
 </net>
 <net name="A2" class="0">
@@
 <junction x="-17.78" y="22.86"/>
 </segment>
+<segment>
+<pinref part="JP3" gate="G$1" pin="3"/>
+<wire x1="99.06" y1="12.7" x2="99.06" y2="15.24" width="0.1524" layer="91"/>
+<label x="99.06" y="15.24" size="1.778" layer="95"/>
+</segment>
 </net>
 <net name="A1" class="0">
@@
 <pinref part="JP4" gate="G$1" pin="11"/>
 <wire x1="-17.78" y1="25.4" x2="-25.4" y2="25.4" width="0.1524" layer="91"/>
+</segment>
+<segment>
+<pinref part="JP3" gate="G$1" pin="2"/>
+<wire x1="101.6" y1="12.7" x2="101.6" y2="15.24" width="0.1524" layer="91"/>
+<label x="101.6" y="15.24" size="1.778" layer="95"/>
 </segment>
 </net>
@@
 <junction x="-17.78" y="27.94"/>
 </segment>
-</net>
+<segment>
+<pinref part="JP3" gate="G$1" pin="1"/>
+<wire x1="104.14" y1="12.7" x2="104.14" y2="15.24" width="0.1524" layer="91"/>
+<label x="104.14" y="15.24" size="1.778" layer="95"/>
+</segment>
+</net>
