File: projects/PCBmotors/v1/pcbmotor.brd (EAGLE design)
At the start: 25 x 32.5 mm, 3 parts

Commit message: sada
ds
Connections:
- removed net A: A.TP
- removed net B: B.TP
- removed net C: C.TP
- new net COILS: A.TP, B.TP, C.TP
Routing:
- net COILS: track 0.00 -> 836.2 mm, vias 0 -> 11
- net B: track 439.2 -> 0.00 mm, vias 4 -> 0
- net A: track 343.5 -> 100.8 mm, vias 4 -> 0
- net C: track 359.1 -> 204.8 mm, vias 5 -> 2
