File: projects/Soccerbot/V6/JetsonVersion/Jetsonboard.brd (EAGLE design)
At the start: 206.2 x 206.2 mm, 50 parts, among them J2 XT60-M

Commit message: sada
ds
Parts:
- moved MOTORCONNECTOR2 368.3 mm to (154.0, 88.5), turned to 45 degrees
- moved MOTORCONNECTOR3 349.3 mm to (153.3, 31.4), turned to 315 degrees
- moved U$6 262.1 mm to (134.6, 50.0)
- moved MOTORCONNECTOR4 259.7 mm to (47.0, 31.8), turned to 225 degrees
- moved MOTOR2 256.3 mm to (190.8, 61.4), turned to 90 degrees
- moved MOTOR3 255.6 mm to (190.6, 34.5), turned to 90 degrees
- moved MOTOR2PT2 250.4 mm to (155.1, 84.2), turned to 270 degrees
- moved MOTOR3PT2 234.9 mm to (155.0, 57.4), turned to 270 degrees
- moved MOTORCONNECTOR1 213.7 mm to (44.8, 89.0), turned to 135 degrees
- moved U$2 184.0 mm to (70.7, 50.0)
- moved MOTOR6PT2 182.1 mm to (-44.0, 185.9), turned to 270 degrees
- moved MOTOR5 177.4 mm to (111.6, 7.67), turned to 180 degrees
- moved MOTOR6 161.7 mm to (-31.2, 173.1), turned to 90 degrees
- moved MOTOR5PT2 157.9 mm to (91.2, -28.0)
- moved MOTOR1PT2 149.1 mm to (39.7, 61.2), turned to 90 degrees
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Other:
- board size 206.2 x 206.2 mm -> 417.6 x 217 mm
- board text added: "gnd"
- board text added: "pwm"
