File: projects/Princeton Led Controller/Led Controller.brd (EAGLE design)
At the start: 254 x 140 mm, 64 parts, among them J1 POWER_JACKPTH, J2 62000411121, J3 62000411121, J4 62000411121, J5 62000411121, J6 62000411121, J7 62000411121, J8 62000411121, J9 62000411121

Commit message: nlm
m.,
Routing:
- net GND: track 367.2 -> 367.9 mm
Changed lines of the file:
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@@
 <?xml version="1.0" encoding="utf-8"?>
 <!DOCTYPE eagle SYSTEM "eagle.dtd">
-<eagle version="9.3.2">
+<eagle version="9.4.2">
 <drawing>
 <settings>
@@
 <wire x1="92.3925" y1="108.42625" x2="92.3925" y2="109.5375" width="0.762" layer="1"/>
 <wire x1="92.3925" y1="109.5375" x2="92.423" y2="109.6" width="0.762" layer="1"/>
-<wire x1="155.41625" y1="110.8075" x2="155.41625" y2="109.69625" width="0.762" layer="1"/>
 <wire x1="155.41625" y1="109.69625" x2="155.423" y2="109.6" width="0.762" layer="1"/>
 <wire x1="218.44" y1="38.735" x2="218.44" y2="37.62375" width="0.762" layer="1"/>
@@
 <via x="155.41625" y="38.735" extent="1-16" drill="0.3937"/>
 <via x="92.3925" y="108.42625" extent="1-16" drill="0.3937"/>
-<via x="155.41625" y="110.8075" extent="1-16" drill="0.3937"/>
+<via x="155.16225" y="111.4425" extent="1-16" drill="0.3937"/>
 <via x="218.44" y="38.735" extent="1-16" drill="0.3937"/>
 <via x="218.44" y="110.8075" extent="1-16" drill="0.3937"/>
@@
 <wire x1="225.5012" y1="101.8987" x2="225.5012" y2="106.1212" width="0.762" layer="1"/>
 <wire x1="212.725" y1="96.901" x2="220.5035" y2="96.901" width="0.762" layer="1"/>
+<wire x1="155.16225" y1="111.4425" x2="155.16225" y2="109.95025" width="0.254" layer="1"/>
+<wire x1="155.16225" y1="109.95025" x2="155.41625" y2="109.69625" width="0.254" layer="1"/>
 </signal>
 <signal name="DIN">
@@
 <contactref element="J9" pad="4"/>
 <wire x1="154.9146" y1="106.6546" x2="153.4668" y2="105.2068" width="0.762" layer="16"/>
-<wire x1="154.9146" y1="109.4994" x2="154.9146" y2="106.6546" width="0.762" layer="16"/>
+<wire x1="154.9146" y1="109.4994" x2="154.9146" y2="107.442" width="0.762" layer="16"/>
+<wire x1="154.9146" y1="107.442" x2="154.9146" y2="106.6546" width="0.762" layer="16"/>
 <wire x1="157.9372" y1="112.522" x2="154.9146" y2="109.4994" width="0.762" layer="16"/>
 <wire x1="214.757" y1="110.998" x2="213.233" y2="112.522" width="0.762" layer="16"/>
