File: projects/Princeton Led Controller/Led ControllerV2.brd (EAGLE design)
At the start: 254 x 140 mm, 53 parts, among them J1 POWER_JACKPTH, J2 62000411121, J3 62000411121, J4 62000411121, J5 62000411121, J6 62000411121, J7 62000411121, J8 62000411121, J9 62000411121

Commit message: nlm
m.,
Parts:
- removed R2: 300, SparkFun-Resistors:0603
- added 1-8, 17-24, 25-32, 33-40, 41-48, 49-56, 57-64, 65-72, 73-80, 81-88, 89-96, 9-16: M09, SparkFun:1X09
- added D1, D2, D3, D4, D5, D6, D7, D8: (no value), SparkFun-LED:LED_5MM
- added JP12, JP13: INPUT, adafruit:1X06-CLEANBIG
- added NEOPASSTHROUGH: (no value), SparkFun:1X03
- added R1: 300, FaBo-Coil:AXL-REGULAR
- added SJ1, SJ2: (no value), BaseApp:SJW
Connections:
- removed net N$3: U$1.5V
- new net N$4: J9.1, NEOPASSTHROUGH.1
- new net VCCNANO: SJ1.2, U$1.5V
- net /OE: now also JP12.5, JP13.5
- net CLK: now also JP12.4, JP13.4
- net DATAIN: now also R1.2; no longer R2.2
- net DIN: now also JP13.3
- net DN4: now also JP12.3
- net GND: now also JP12.2, JP13.2, NEOPASSTHROUGH.3
- net LAT: now also JP12.6, JP13.6
- net LED+: now also 1-8.9, 17-24.9, 25-32.9, 33-40.9, 41-48.9, 49-56.9, 57-64.9, 65-72.9, 73-80.9, 81-88.9, 89-96.9, 9-16.9, D1.A, D2.A, D3.A, D4.A, D5.A, D6.A, D7.A, D8.A
- net LED1: now also 1-8.8, D1.K
- net LED10: now also 9-16.7
- net LED11: now also 9-16.6
- net LED12: now also 9-16.5
- net LED13: now also 9-16.4
- net LED14: now also 9-16.3
- net LED15: now also 9-16.2
- net LED16: now also 9-16.1
- net LED17: now also 17-24.8
- net LED18: now also 17-24.7
- net LED19: now also 17-24.6
- net LED2: now also 1-8.7, D2.K
- net LED20: now also 17-24.5
- net LED21: now also 17-24.4
- net LED22: now also 17-24.3
- net LED23: now also 17-24.2
- net LED24: now also 17-24.1
- net LED25: now also 25-32.8
- net LED26: now also 25-32.7
- net LED27: now also 25-32.6
- net LED28: now also 25-32.5
- net LED29: now also 25-32.4
- net LED3: now also 1-8.6, D3.K
- net LED30: now also 25-32.3
- net LED31: now also 25-32.2
- net LED32: now also 25-32.1
- net LED33: now also 33-40.8
- net LED34: now also 33-40.7
- net LED35: now also 33-40.6
- net LED36: now also 33-40.5
- net LED37: now also 33-40.4
- net LED38: now also 33-40.3
- net LED39: now also 33-40.2
- net LED4: now also 1-8.5, D4.K
- net LED40: now also 33-40.1
- net LED41: now also 41-48.8
- net LED42: now also 41-48.7
- net LED43: now also 41-48.6
- net LED44: now also 41-48.5
- net LED45: now also 41-48.4
- net LED46: now also 41-48.3
- net LED47: now also 41-48.2
- net LED48: now also 41-48.1
- net LED49: now also 49-56.8
- net LED5: now also 1-8.4, D5.K
- net LED50: now also 49-56.7
- net LED51: now also 49-56.6
- net LED52: now also 49-56.5
- net LED53: now also 49-56.4
- net LED54: now also 49-56.3
- net LED55: now also 49-56.2
- net LED56: now also 49-56.1
- net LED57: now also 57-64.8
- net LED58: now also 57-64.7
- net LED59: now also 57-64.6
- net LED6: now also 1-8.3, D6.K
- net LED60: now also 57-64.5
- net LED61: now also 57-64.4
- net LED62: now also 57-64.3
- net LED63: now also 57-64.2
- net LED64: now also 57-64.1
- net LED65: now also 65-72.8
- net LED66: now also 65-72.7
- net LED67: now also 65-72.6
- net LED68: now also 65-72.5
- net LED69: now also 65-72.4
- net LED7: now also 1-8.2, D7.K
- net LED70: now also 65-72.3
- net LED71: now also 65-72.2
- net LED72: now also 65-72.1
- net LED73: now also 73-80.8
- net LED74: now also 73-80.7
- net LED75: now also 73-80.6
- net LED76: now also 73-80.5
- net LED77: now also 73-80.4
- net LED78: now also 73-80.3
- net LED79: now also 73-80.2
- net LED8: now also 1-8.1, D8.K
- net LED80: now also 73-80.1
- net LED81: now also 81-88.8
- net LED82: now also 81-88.7
- net LED83: now also 81-88.6
- net LED84: now also 81-88.5
- net LED85: now also 81-88.4
- net LED86: now also 81-88.3
- net LED87: now also 81-88.2
- net LED88: now also 81-88.1
- net LED89: now also 89-96.8
- net LED9: now also 9-16.8
- net LED90: now also 89-96.7
- net LED91: now also 89-96.6
- net LED92: now also 89-96.5
- net LED93: now also 89-96.4
- net LED94: now also 89-96.3
- net LED95: now also 89-96.2
- net LED96: now also 89-96.1
- net N$1: now also SJ2.1
- net NEODATA1: now also R1.1; no longer R2.1
- net VCC: now also JP12.1, JP13.1, NEOPASSTHROUGH.2, SJ1.1, SJ2.2
Routing:
- net LED+: track 0.00 -> 852.2 mm, vias 0 -> 66
- net VCC: track 0.00 -> 729.8 mm, vias 0 -> 3
- net GND: track 0.00 -> 465.4 mm, vias 0 -> 12
- net LED8: track 0.00 -> 306.0 mm, vias 0 -> 3
- net LED6: track 0.00 -> 285.6 mm, vias 0 -> 1
- net LED13: track 0.00 -> 272.5 mm
- net N$34: track 0.00 -> 262.7 mm, vias 0 -> 1
- net LED12: track 0.00 -> 258.0 mm
- net LED34: track 0.00 -> 249.5 mm
- net LED15: track 0.00 -> 249.4 mm, vias 0 -> 1
- net LAT: track 0.00 -> 242.5 mm
- net LED11: track 0.00 -> 242.4 mm, vias 0 -> 1
- net LED16: track 0.00 -> 239.5 mm, vias 0 -> 2
- net LED9: track 0.00 -> 229.5 mm, vias 0 -> 1
- net CLK: track 0.00 -> 227.2 mm
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Other:
- board text added: "Designed By David Bershasky"
