File: projects/Princeton Led Controller/Led ControllerV2.brd (EAGLE design)
At the start: 254 x 140 mm, 78 parts, among them J1 POWER_JACKPTH, J2 62000411121, J3 62000411121, J4 62000411121, J5 62000411121, J6 62000411121, J7 62000411121, J8 62000411121, J9 62000411121

Commit message: sad
asd
Routing:
- net N$35: track 89.3 -> 86.4 mm
- net LED6: track 285.6 -> 283.2 mm
Changed lines of the file:
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@@
 <?xml version="1.0" encoding="utf-8"?>
 <!DOCTYPE eagle SYSTEM "eagle.dtd">
-<eagle version="9.4.2">
+<eagle version="9.5.0">
 <drawing>
 <settings>
@@
 <wire x1="102" y1="116" x2="100.5" y2="116" width="0.762" layer="1"/>
 <wire x1="100.5" y1="116" x2="93.5" y2="123" width="0.762" layer="1"/>
-<wire x1="23" y1="123" x2="93.5" y2="123" width="0.762" layer="1"/>
-<wire x1="23" y1="37.5" x2="23" y2="123" width="0.762" layer="1"/>
+<wire x1="27" y1="123" x2="93.5" y2="123" width="0.762" layer="1"/>
 <wire x1="38.5" y1="22" x2="23" y2="37.5" width="0.762" layer="1"/>
 <wire x1="75" y1="22" x2="38.5" y2="22" width="0.762" layer="1"/>
@@
 <wire x1="75" y1="20" x2="75.08" y2="20" width="0.762" layer="1"/>
 <via x="102" y="116" extent="1-16" drill="0.3937"/>
+<wire x1="23" y1="119" x2="27" y2="123" width="0.762" layer="1"/>
+<wire x1="23" y1="37.5" x2="23" y2="119" width="0.762" layer="1"/>
 </signal>
 <signal name="LED10">
@@
 <wire x1="43" y1="40" x2="43" y2="77" width="0.762" layer="16"/>
 <wire x1="70" y1="13" x2="43" y2="40" width="0.762" layer="16"/>
-<wire x1="248" y1="13" x2="70" y2="13" width="0.762" layer="16"/>
+<wire x1="70" y1="13" x2="248" y2="13" width="0.762" layer="16"/>
 <wire x1="248" y1="25" x2="248" y2="13" width="0.762" layer="16"/>
 <wire x1="245" y1="28" x2="248" y2="25" width="0.762" layer="16"/>
@@
 <contactref element="J7" pad="4"/>
 <wire x1="32.5" y1="106.5" x2="34" y2="105" width="0.762" layer="1"/>
-<wire x1="32.5" y1="122" x2="32.5" y2="106.5" width="0.762" layer="1"/>
-<wire x1="90.5" y1="122" x2="32.5" y2="122" width="0.762" layer="1"/>
-<wire x1="97" y1="115.5" x2="90.5" y2="122" width="0.762" layer="1"/>
+<wire x1="32.5" y1="106.5" x2="32.5" y2="117" width="0.762" layer="1"/>
+<wire x1="90.5" y1="122" x2="97" y2="115.5" width="0.762" layer="1"/>
 <wire x1="97" y1="111" x2="97" y2="115.5" width="0.762" layer="1"/>
+<wire x1="32.5" y1="117" x2="37.5" y2="122" width="0.762" layer="1"/>
+<wire x1="37.5" y1="122" x2="90.5" y2="122" width="0.762" layer="1"/>
 </signal>
 <signal name="N$36">
