File: projects/Soccerbot/V6/RaspiVersion/lowerboard.sch (EAGLE design)
At the start: 49 parts, among them J2 XT60-M

Commit message: asd
asd
Other:
- moved on the sheet: 5, 6, 7, 8, COLOR5, COLOR6, COLOR7, COLOR8
