File: projects/Soccerbot/V6/RaspiVersion/midboard.sch (EAGLE design)
At the start: 43 parts, among them J2 XT60-M

Commit message: asd
asd
Parts:
- added ENCODERSPI: M09, SparkFun:M09
- added F1: 72V/0.25A, SparkFun-Fuses:PPTC_PTH
- added J1: (no value), Wurth_Elektronik_Electromechanic_Board_to_Board_Connectors_rev17a:61304021021
- added MOTENCODER1, MOTENCODER2, MOTENCODER3, MOTENCODER4: (no value), SparkFun:M05PTH
- renumbered 1 to JP11, 2 to JP10, 3 to JP7, 4 to JP2, 5 to JP12, 6 to JP9, 7 to JP8, 8 to JP1
Connections:
- new net 1CS0: J1.29
- new net 1CS1: J1.28
- new net 1MISO: J1.11
- new net 1MOSI: J1.10
- new net 1SCK: J1.12
- new net 2CS0: J1.32
- new net 2CS1: J1.33
- new net 2CTS: J1.23
- new net 2MISO: J1.30
- new net 2MOSI: J1.19
- new net 2RTS: J1.6
- new net 2SCK: J1.7
- new net 4LRCK: J1.18
- new net 4SDIN: J1.22
- new net 4SDOUT: J1.21
- new net CAMAFEN: J1.15
- new net GPIOPE6: J1.17
- new net GPIOPZ0: J1.16
- new net LCDTE: J1.8
- new net LCD_BL_PWM: J1.25
- new net MCLK: J1.4
- new net RX2: J1.36
- new net SCL1: J1.27
- new net SCL2: J1.3
- new net SCLK4: J1.35
- new net SDA1: J1.14
- new net SDA2: J1.2
- new net TX2: J1.37
- net ENCCS1: now also ENCODERSPI.6
- net ENCCS2: now also ENCODERSPI.7
- net ENCCS3: now also ENCODERSPI.8
- net ENCCS4: now also ENCODERSPI.9
- net ENCGND: now also MOTENCODER1.1, MOTENCODER2.1, MOTENCODER3.1, MOTENCODER4.1
- net ENCMISO: now also ENCODERSPI.4
- net ENCMOSI: now also ENCODERSPI.5
- net ENCSCLK: now also ENCODERSPI.3
- net ENCVCC: now also MOTENCODER1.2, MOTENCODER2.2, MOTENCODER3.2, MOTENCODER4.2
- net GND: now also ENCODERSPI.1, J1.13, J1.20, J1.24, J1.26, J1.31, J1.34, J1.38, J1.5
- net M1ENCA: now also MOTENCODER1.3
- net M1ENCB: now also MOTENCODER1.4
- net M2ENCA: now also MOTENCODER2.3
- net M2ENCB: now also MOTENCODER2.4
- net M3ENCA: now also MOTENCODER3.3
- net M3ENCB: now also MOTENCODER3.4
- net M4ENCA: now also MOTENCODER4.3
- net M4ENCB: now also MOTENCODER4.4
- net VCC: now also ENCODERSPI.2, J1.39, J1.40
- net VCC3.3: now also J1.1, J1.9
