File: projects/Soccerbot/V6/RaspiVersion/lowerboard.brd (EAGLE design)
At the start: 218 x 218 mm, 49 parts, among them J2 XT60-M

Commit message: h
j
Parts:
- moved MOTOR1PT2 364.5 mm to (-29.3, -101.7)
- moved MOTOR2PT2 359.6 mm to (6.68, -101.7)
- moved MOTOR2 331.3 mm to (29.5, -66.1), turned to 180 degrees
- moved MOTOR5 322.0 mm to (62.6, -17.7), turned to 180 degrees
- moved MOTOR5PT2 319.0 mm to (39.7, 17.8)
- moved COLOR1 310.9 mm to (-30.3, -49.7), flipped to the bottom, turned to 225 degrees
- moved 1 309.3 mm to (-32.1, -51.5), flipped to the bottom, turned to 225 degrees
- moved VRM 306.7 mm to (7.53, -19.3), turned to 270 degrees
- moved MOTOR1 298.5 mm to (-6.47, -66.1), turned to 180 degrees
- moved MOTOR3 230.2 mm to (-6.47, 66.1), turned to 180 degrees
- moved MOTOR4PT2 224.1 mm to (6.68, 101.7)
- moved MOTOR4 221.3 mm to (29.5, 66.1), turned to 180 degrees
- moved MOTOR3PT2 179.7 mm to (-29.3, 101.7)

Commit message: asd
asd
Parts:
- moved COLOR7 413.6 mm to (-300.6, -132.9)
- moved COLOR6 409.2 mm to (-292.1, -127.9)
- moved COLOR8 406.8 mm to (-292.1, -132.9)
- moved COLOR5 380.1 mm to (-300.6, -127.9)
- moved 5 363.4 mm to (-300.6, -113.2)
- moved 7 363.1 mm to (-300.6, -120.5)
- moved 8 357.1 mm to (-292.5, -120.5)
- moved 6 356.6 mm to (-292.5, -113.2)
- moved COLOR2 351.5 mm to (23.5, -50.7), flipped to the bottom, turned to 135 degrees
- moved 2 305.9 mm to (25.3, -52.5), flipped to the bottom, turned to 315 degrees
- moved COLOR4 287.1 mm to (23.7, 50.8), flipped to the bottom, turned to 225 degrees
- moved COLOR3 248.0 mm to (-27.3, 47.1), flipped to the bottom, turned to 135 degrees
- moved 4 231.7 mm to (25.5, 52.6), flipped to the bottom, turned to 225 degrees
- moved 3 194.1 mm to (-25.5, 52.4), flipped to the bottom, turned to 135 degrees
- moved COLOR1 3.97 mm to (-27.3, -47.1)
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
Commit message: bnm
vbh
Parts:
- removed 1, 2, 3, 4, 5, 6, 7, 8: M01PTH, SparkFun:1X01
- removed COLOR1, COLOR2, COLOR3, COLOR4, COLOR5, COLOR6, COLOR7, COLOR8: (no value), SparkFun:1X03
- removed ENCODERSPI: M09, SparkFun:1X09
- removed MOTENCODER1, MOTENCODER2, MOTENCODER3, MOTENCODER4, VRM: (no value), SparkFun:1X05
- removed MOTOR1, MOTOR2, MOTOR3, MOTOR4, MOTOR5: M10", SparkFun:1X10
- removed MOTOR1PT2, MOTOR2PT2, MOTOR3PT2, MOTOR4PT2, MOTOR5PT2: (no value), SparkFun:1X08
- removed MOTOR6, MOTOR6PT2: (no value), SparkFun:1X06
- added JP1, JP2: (no value), SparkFun:1X04
- added JP10, JP20, JP22, JP26, JP28, JP30, JP32, JP36: (no value), SparkFun:1X03
- added JP11, JP24, JP3, JP5, JP7: M10", SparkFun:1X10
- added JP12, JP25, JP4, JP6, JP8: (no value), SparkFun:1X08
- added JP13, JP21, JP23, JP27, JP29, JP31, JP35, JP9: M01PTH, SparkFun:1X01
- added JP14, JP15, JP16, JP17, JP18: (no value), SparkFun:1X05
- added JP19: M09, SparkFun:1X09
- moved U$1 650.3 mm to (370.4, 122.8)
- moved MOTORCONNECTOR4 413.4 mm to (214.3, 87.7), turned to 315 degrees
- moved MOTORCONNECTOR1 359.1 mm to (163.5, 185.0), turned to 135 degrees
- moved MOTORCONNECTOR2 356.1 mm to (221.7, 194.5), turned to 225 degrees
- moved MOTORCONNECTOR3 339.6 mm to (152.8, 78.9), turned to 45 degrees
- moved U$6 315.5 mm to (82.9, 327.4)
- moved U$3 114.2 mm to (-49.4, 122.8)
- moved U$2 61.6 mm to (-163.2, 209.0)
Connections:
- removed net BAT+: J2.2, MOTOR1PT2.7, MOTOR1PT2.8, MOTOR2PT2.8, MOTOR3PT2.8, MOTOR4PT2.8, MOTOR5PT2.8, MOTOR6PT2.5, VRM.4
- removed net ENCGND: MOTENCODER1.1, MOTENCODER2.1, MOTENCODER3.1, MOTENCODER4.1, MOTORCONNECTOR1.4, MOTORCONNECTOR2.4, MOTORCONNECTOR3.4, MOTORCONNECTOR4.4
- removed net ENCVCC: MOTENCODER1.2, MOTENCODER2.2, MOTENCODER3.2, MOTENCODER4.2, MOTORCONNECTOR1.3, MOTORCONNECTOR2.3, MOTORCONNECTOR3.3, MOTORCONNECTOR4.3
- removed net M5OUTA: MOTOR5PT2.2
- removed net M5OUTB: MOTOR5PT2.4
- removed net M6OUTA: MOTOR6PT2.3
- removed net M6OUTB: MOTOR6PT2.4
- removed net N$1: MOTOR2PT2.5
- removed net N$10: MOTOR3PT2.7
- removed net N$11: MOTOR3PT2.1
- removed net N$12: MOTOR3PT2.3
- removed net N$13: MOTOR4PT2.5
- removed net N$14: MOTOR4PT2.7
- removed net N$15: MOTOR4PT2.1
- removed net N$16: MOTOR4PT2.3
- removed net N$17: MOTOR5PT2.5
- removed net N$18: MOTOR5PT2.7
- removed net N$19: MOTOR5PT2.1
- removed net N$2: MOTOR2PT2.7
- removed net N$20: MOTOR5PT2.3
- removed net N$3: MOTOR2PT2.1
- removed net N$4: MOTOR6.4
- removed net N$5: MOTOR6.5
- removed net N$6: MOTOR6.6
- removed net N$7: MOTOR2PT2.3
- removed net N$9: MOTOR3PT2.5
- removed net SO8: COLOR8.3
- new net 5V: JP1.4, JP10.2, JP11.7, JP14.1, JP19.8, JP2.4, JP20.2, JP22.2, JP24.7, JP26.2, JP28.2, JP3.7, JP30.2, JP32.2, JP36.2, JP5.7, JP7.7, MOTORCONNECTOR1.3, MOTORCONNECTOR2.3, MOTORCONNECTOR3.3, MOTORCONNECTOR4.3
- new net A0: JP15.3
- new net A1: JP16.3
- new net A2: JP17.3
- new net A3: JP18.3
- new net B0: JP15.2
- new net B1: JP16.2
- new net B2: JP17.2
- new net B3: JP18.2
- new net CS_DIS0: JP3.4
- new net CS_DIS1: JP7.4
- new net CS_DIS2: JP5.4
- new net CS_DIS3: JP11.4
- new net CS_DIS4: JP24.4
- new net EN: JP14.5
- new net ENA/DIAGA0: JP3.2
- new net ENA/DIAGA1: JP7.2
- new net ENA/DIAGA2: JP5.2
- new net ENA/DIAGA3: JP11.2
- new net ENA/DIAGA4: JP24.2
- new net ENB/DIAGB0: JP3.5
- new net ENB/DIAGB1: JP7.5
- new net ENB/DIAGB2: JP5.5
- new net ENB/DIAGB3: JP11.5
- new net ENB/DIAGB4: JP24.5
- new net G0: JP15.5
- new net G1: JP16.5
- new net G2: JP17.5
- new net G3: JP18.5
- new net I0: JP15.1
- new net I1: JP16.1
- new net I2: JP17.1
- new net I3: JP18.1
- new net OUTA0: JP4.1, JP4.2
- new net OUTA1: JP8.1, JP8.2
- new net OUTA2: JP6.1, JP6.2
- new net OUTA3: JP12.1, JP12.2
- new net OUTA4: JP25.1, JP25.2
- new net OUTB0: JP4.3, JP4.4
- new net OUTB1: JP8.3, JP8.4
- new net OUTB2: JP6.3, JP6.4
- new net OUTB3: JP12.3, JP12.4
- new net OUTB4: JP25.3, JP25.4
- new net PWM0: JP3.3
- new net PWM1: JP7.3
- new net PWM2: JP5.3
- new net PWM3: JP11.3
- new net PWM4: JP24.3
- new net SCLTOF: JP1.2, JP2.2, U$1.A5
- new net SDATOF: JP1.1, JP2.1, U$1.A4
- new net SO0: JP10.1
- new net V0: JP15.4
- new net V1: JP16.4
- new net V2: JP17.4
- new net V3: JP18.4
- new net VIN: J2.2, JP12.7, JP12.8, JP14.4, JP25.7, JP25.8, JP4.7, JP4.8, JP6.7, JP6.8, JP8.7, JP8.8
- new net VOUT0: JP3.9
- new net VOUT1: JP7.9
- new net VOUT2: JP5.9
- new net VOUT3: JP11.9
- new net VOUT4: JP24.9
- net CTRL: now also JP13.1, JP21.1, JP23.1, JP27.1, JP29.1, JP31.1, JP35.1, JP9.1; no longer 1.1, 2.1, 3.1, 4.1, 5.1, 6.1, 7.1, 8.1
- net ENCCS1: now also JP19.4; no longer ENCODERSPI.6
- net ENCCS2: now also JP19.3; no longer ENCODERSPI.7
- net ENCCS3: now also JP19.2; no longer ENCODERSPI.8
- net ENCCS4: now also JP19.1; no longer ENCODERSPI.9
- net ENCMISO: now also JP19.6; no longer ENCODERSPI.4
- net ENCMOSI: now also JP19.5; no longer ENCODERSPI.5
- net ENCSCLK: now also JP19.7; no longer ENCODERSPI.3
- net GND: now also JP1.3, JP10.3, JP11.10, JP11.8, JP12.5, JP12.6, JP14.2, JP14.3, JP19.9, JP2.3, JP20.3, JP22.3, JP24.10, JP24.8, JP25.5, JP25.6, JP26.3, JP28.3, JP3.10, JP3.8, JP30.3, JP32.3, JP36.3, JP4.5, JP4.6, JP5.10, JP5.8, JP6.5, JP6.6, JP7.10, JP7.8, JP8.5, JP8.6, MOTORCONNECTOR1.4, MOTORCONNECTOR2.4, MOTORCONNECTOR3.4, MOTORCONNECTOR4.4; no longer COLOR1.1, COLOR2.1, COLOR3.1, COLOR4.1, COLOR5.1, COLOR6.1, COLOR7.1, COLOR8.1, ENCODERSPI.1, MOTOR1.1, MOTOR1.3, MOTOR1PT2.5, MOTOR1PT2.6, MOTOR2.1, MOTOR2.3, MOTOR2PT2.6, MOTOR3.1, MOTOR3.3, MOTOR3PT2.6, MOTOR4.1, MOTOR4.3, MOTOR4PT2.6, MOTOR5.1, MOTOR5.3, MOTOR5PT2.6, MOTOR6PT2.2, MOTOR6PT2.6, VRM.2, VRM.3
- net INA0: now also JP3.1; no longer MOTOR1.10
- net INA1: now also JP7.1; no longer MOTOR2.10
- net INA2: now also JP5.1; no longer MOTOR3.10
- net INA3: now also JP11.1; no longer MOTOR4.10
- net INA4: now also JP24.1; no longer MOTOR5.10
- net INA5: no longer MOTOR6.3
- net INB0: now also JP3.6; no longer MOTOR1.5
- net INB1: now also JP7.6; no longer MOTOR2.5
- net INB2: now also JP5.6; no longer MOTOR3.5
- net INB3: now also JP11.6; no longer MOTOR4.5
- net INB4: now also JP24.6; no longer MOTOR5.5
- net INB5: no longer MOTOR6.2
- net M1ENCA: no longer MOTENCODER1.3
- net M1ENCB: no longer MOTENCODER1.4
- net M1OUTA: no longer MOTOR1PT2.1, MOTOR1PT2.2
- net M1OUTB: no longer MOTOR1PT2.3, MOTOR1PT2.4
- net M2ENCA: no longer MOTENCODER2.3
- net M2ENCB: no longer MOTENCODER2.4
- net M2OUTA: no longer MOTOR2PT2.2
- net M2OUTB: no longer MOTOR2PT2.4
- net M3ENCA: no longer MOTENCODER3.3
- net M3ENCB: no longer MOTENCODER3.4
- net M3OUTA: no longer MOTOR3PT2.2
- net M3OUTB: no longer MOTOR3PT2.4
- net M4ENCA: no longer MOTENCODER4.3
- net M4ENCB: no longer MOTENCODER4.4
- net M4OUTA: no longer MOTOR4PT2.2
- net M4OUTB: no longer MOTOR4PT2.4
- net MPWM0: no longer MOTOR1.8
- net MPWM1: no longer MOTOR2.8
- net MPWM2: no longer MOTOR3.8
- net MPWM3: no longer MOTOR4.8
- net MPWM4: no longer MOTOR5.8
- net MPWM5: no longer MOTOR6.1
- net SO1: now also JP30.1; no longer COLOR1.3
- net SO2: now also JP22.1; no longer COLOR2.3
- net SO3: now also JP36.1; no longer COLOR3.3
- net SO4: now also JP20.1; no longer COLOR4.3
- net SO5: now also JP32.1; no longer COLOR5.3
- net SO6: now also JP28.1; no longer COLOR6.3
- net SO7: now also JP26.1; no longer COLOR7.3
- net VCC: no longer COLOR1.2, COLOR2.2, COLOR3.2, COLOR4.2, COLOR5.2, COLOR6.2, COLOR7.2, COLOR8.2, ENCODERSPI.2, MOTOR1.4, MOTOR2.4, MOTOR3.4, MOTOR4.4, MOTOR5.4, MOTOR6PT2.1, VRM.1
Other:
- board text removed: "gnd"
- board text removed: "pwm"
