File: projects/RoomSteralizer/sterileplate.brd (EAGLE design)
At the start: 47 x 42 mm, 9 parts, among them J2 POWER_JACKPTH_LOCK, Q1 Transistor

Commit message: wqed
afs
Parts:
- added J1, J3: (no value), SparkFun-Connectors:1X01_2MM
- Q1: value Transistor -> Transistor >= 1.5Amp
- moved J2 22.0 mm to (22.1, 24.7)
- moved PIRSENSOR 17.0 mm to (27.8, 0.00)
- moved Q1 16.9 mm to (20.6, -16.2), turned to 180 degrees
- moved D3 10.4 mm to (14.0, -7.00)
- moved D4 10.2 mm to (14.0, 6.00)
- moved D1 7.62 mm to (3.00, -7.00)
- moved D2 7.28 mm to (3.00, 6.00)
Connections:
- net N$3: now also J3.1
- net N$4: now also J1.1
Routing:
- net GND: track 65.3 -> 92.1 mm
- net N$4: track 13.5 -> 34.2 mm
- net LEDTRIG: track 23.8 -> 38.8 mm
- net VIN: track 68.3 -> 83.1 mm
- net VCC: track 53.3 -> 65.9 mm
- net PIROUT: track 35.4 -> 45.2 mm
- net N$2: track 5.20 -> 8.20 mm, vias 0 -> 2
- net N$1: track 5.20 -> 8.20 mm, vias 0 -> 2
- net N$3: track 16.1 -> 17.6 mm
Other:
- board size 47 x 42 mm -> 64 x 42 mm
- board text added: "+"
- board text added: "-"

Commit message: asd
Parts:
- removed PIRSENSOR: 62000311121, Headers:62000311121
- added D5, D6: WP7113SGD, LED:RADIAL_5MM
- added J4: (no value), SparkFun-Connectors:1X01_2MM
- added JP1: (no value), SparkFun:1X03
Connections:
- removed net N$3: D1.1, D2.1, J3.1, R1.2
- new net N$6: D5.A, D6.A, J4.1
- new net N$7: D1.1, D2.1, D5.C, D6.C, J3.1, R1.2
- net GND: now also JP1.1; no longer PIRSENSOR.3
- net PIROUT: now also JP1.2; no longer PIRSENSOR.2
- net VCC: now also JP1.3; no longer PIRSENSOR.1
Routing:
- net N$7: track 0.00 -> 36.5 mm
- net VCC: track 65.9 -> 88.1 mm
- net N$3: track 17.6 -> 0.00 mm
- net N$6: track 0.00 -> 12.1 mm
- net GND: track 92.1 -> 85.4 mm
- net PIROUT: track 45.2 -> 51.4 mm
Other:
- board text added: "INCAND GND"
- board text added: "INDICATOR LED 1"
- board text added: "INDICATOR LED 2"
- board text added: "LED GND"
- board text removed: "-"
